File: proyecto/Microcontrolador.sch (KiCad schematic (older format))
At the start: 14 parts

Commit message: Add files via upload
Parts:
- added J?: Conn_ARM_JTAG_SWD_20, symbol Connector:Conn_ARM_JTAG_SWD_20
Connections:
- net labels added: +3.3V, SRST, TCK, TD0, TD1, TMS, TRST
- net labels removed: 3.3v
- wire segments 62 -> 77
Changed lines of the file:
@@
 $Descr A4 11693 8268
 encoding utf-8
-Sheet 2 5
+Sheet 2 7
 Title ""
 Date ""
@@
 Comment4 ""
 $EndDescr
-Text GLabel 5250 2500 2    50   Input ~ 0
-RST_M
-Wire Wire Line
-	4100 1700 4350 1700
-Connection ~ 4350 1700
 Wire Wire Line
 	4350 1700 4450 1700
@@
 	1    0    0    -1
 $EndComp
-Text GLabel 8000 3800 0    50   Input ~ 0
-RST_M
-Wire Wire Line
-	9250 3800 9100 3800
 Wire Wire Line
 	8800 3800 8600 3800
@@
 Wire Wire Line
 	3850 3900 3650 3900
-Wire Wire Line
-	5250 2500 5050 2500
 $Comp
 L MCU_ST_STM32L0:STM32L052C6Tx U?
@@
 Text HLabel 3650 4800 0    50   Input ~ 0
 PH_EN34
-Text HLabel 4100 1700 0    50   Input ~ 0
-3.3v
 Text HLabel 5200 4300 2    50   Input ~ 0
 MOSI
@@
 Wire Wire Line
 	5900 2900 5650 2900
-Text HLabel 9250 3800 2    50   Input ~ 0
-3.3v
+Text Label 5400 2500 2    50   ~ 0
+RST_M
+Text Label 8000 3800 0    50   ~ 0
+RST_M
+Wire Wire Line
+	5050 2500 5400 2500
+$Comp
+L Connector:Conn_ARM_JTAG_SWD_20 J?
+U 1 1 5E986004
+P 8750 2200
+F 0 "J?" H 8221 2246 50  0000 R CNN
+F 1 "Conn_ARM_JTAG_SWD_20" H 8221 2155 50  0000 R CNN
+F 2 "" H 9200 1150 50  0001 L TNN
+F 3 "http://infocenter.arm.com/help/topic/com.arm.doc.dui0499b/DUI0499B_system_design_reference.pdf" V 8400 950 50  0001 C CNN
+	1    8750 2200
+	1    0    0    -1
+$EndComp
+Text HLabel 9650 1700 2    50   Input ~ 0
+TRST
+Text HLabel 9650 1800 2    50   Input ~ 0
+SRST
+Text HLabel 9650 2100 2    50   Input ~ 0
+TCK
+Text HLabel 9650 2200 2    50   Input ~ 0
+TMS
+Text HLabel 9650 2300 2    50   Input ~ 0
+TD0
+Text HLabel 9650 2400 2    50   Input ~ 0
+TD1
+Wire Wire Line
+	9650 2400 9350 2400
+Wire Wire Line
+	9350 2300 9650 2300
+Wire Wire Line
+	9650 2200 9350 2200
+Wire Wire Line
+	9350 2100 9650 2100
+Wire Wire Line
+	9650 1800 9350 1800
+Wire Wire Line
+	9350 1700 9650 1700
+$Comp
+L power:GND #PWR?
+U 1 1 5E997632
+P 8650 3100
+F 0 "#PWR?" H 8650 2850 50  0001 C CNN
+F 1 "GND" H 8655 2927 50  0000 C CNN
+F 2 "" H 8650 3100 50  0001 C CNN
+F 3 "" H 8650 3100 50  0001 C CNN
+	1    8650 3100
+	1    0    0    -1
+$EndComp
+Wire Wire Line
+	8650 3100 8650 3000
+Text HLabel 5250 4800 2    50   Input ~ 0
+TRST
+Text HLabel 5250 4900 2    50   Input ~ 0
+SRST
+Text HLabel 5250 5000 2    50   Input ~ 0
+TCK
+Text HLabel 5250 5100 2    50   Input ~ 0
+TMS
+Text HLabel 5250 5200 2    50   Input ~ 0
+TD0
+Text HLabel 5250 5300 2    50   Input ~ 0
+TD1
+Wire Wire Line
+	5250 4800 5050 4800
+Wire Wire Line
+	5050 4900 5250 4900
+Wire Wire Line
+	5250 5000 5050 5000
+Wire Wire Line
+	5050 5100 5250 5100
+Wire Wire Line
+	5250 5200 5050 5200
+Wire Wire Line
+	5050 5300 5250 5300
+Wire Wire Line
+	8750 1400 8750 1100
+$Comp
+L power:+3.3V #PWR?
+U 1 1 5E9CE6D3
+P 8750 1100
+F 0 "#PWR?" H 8750 950 50  0001 C CNN
+F 1 "+3.3V" H 8765 1273 50  0000 C CNN
+F 2 "" H 8750 1100 50  0001 C CNN
+F 3 "" H 8750 1100 50  0001 C CNN
+	1    8750 1100
+	1    0    0    -1
+$EndComp
+$Comp
+L power:+3.3V #PWR?
+U 1 1 5E9CEFDA
+P 9300 3650
+F 0 "#PWR?" H 9300 3500 50  0001 C CNN
+F 1 "+3.3V" H 9315 3823 50  0000 C CNN
+F 2 "" H 9300 3650 50  0001 C CNN
+F 3 "" H 9300 3650 50  0001 C CNN
+	1    9300 3650
+	1    0    0    -1
+$EndComp
+Wire Wire Line
+	9100 3800 9300 3800
+Wire Wire Line
+	9300 3800 9300 3650
+$Comp
+L power:+3.3V #PWR?
+U 1 1 5E9D4164
+P 4350 1450
+F 0 "#PWR?" H 4350 1300 50  0001 C CNN
+F 1 "+3.3V" H 4365 1623 50  0000 C CNN
+F 2 "" H 4350 1450 50  0001 C CNN
+F 3 "" H 4350 1450 50  0001 C CNN
+	1    4350 1450
+	1    0    0    -1
+$EndComp
+Wire Wire Line
+	4350 1450 4350 1700
+Connection ~ 4350 1700
 $EndSCHEMATC

Commit message: Add files via upload
Parts:
- added R?: 510, symbol Device:R
Connections:
- net +3V3: now also J?.1 (VTREF)
- net GND: now also R?.1
- net at J?.11 (RTCK): now also R?.2
Changed lines of the file:
@@
 	9650 2200 9350 2200
-Wire Wire Line
-	9350 2100 9650 2100
-Wire Wire Line
-	9650 1800 9350 1800
 Wire Wire Line
 	9350 1700 9650 1700
@@
 	5050 5300 5250 5300
 Wire Wire Line
-	8750 1400 8750 1100
+	8750 1400 8750 1250
 $Comp
 L power:+3.3V #PWR?
@@
 	4350 1450 4350 1700
 Connection ~ 4350 1700
+Wire Wire Line
+	8650 1400 8650 1250
+Wire Wire Line
+	8650 1250 8750 1250
+Connection ~ 8750 1250
+Wire Wire Line
+	8750 1250 8750 1100
+$Comp
+L Device:R R?
+U 1 1 5EA45BC4
+P 9700 2000
+F 0 "R?" V 9493 2000 50  0001 C CNN
+F 1 "510" V 9585 2000 50  0000 C CNN
+F 2 "" V 9630 2000 50  0001 C CNN
+F 3 "~" H 9700 2000 50  0001 C CNN
+	1    9700 2000
+	0    1    1    0
+$EndComp
+Wire Wire Line
+	9350 2100 9650 2100
+Wire Wire Line
+	9350 1800 9650 1800
+$Comp
+L power:GND #PWR?
+U 1 1 5EA4A411
+P 10050 2000
+F 0 "#PWR?" H 10050 1750 50  0001 C CNN
+F 1 "GND" V 10055 1872 50  0000 R CNN
+F 2 "" H 10050 2000 50  0001 C CNN
+F 3 "" H 10050 2000 50  0001 C CNN
+	1    10050 2000
+	0    -1   -1   0
+$EndComp
+Wire Wire Line
+	9350 2000 9550 2000
+Wire Wire Line
+	10050 2000 9850 2000
 $EndSCHEMATC

Commit message: Add files via upload
Connections:
- net labels added: SRST1, TCK1, TD01, TD11, TMS1, TRST1
Changed lines of the file:
@@
 $Descr A4 11693 8268
 encoding utf-8
-Sheet 2 7
+Sheet 7 7
 Title ""
 Date ""
@@
 	1    0    0    -1
 $EndComp
-Text HLabel 9650 1700 2    50   Input ~ 0
-TRST
-Text HLabel 9650 1800 2    50   Input ~ 0
-SRST
-Text HLabel 9650 2100 2    50   Input ~ 0
-TCK
-Text HLabel 9650 2200 2    50   Input ~ 0
-TMS
-Text HLabel 9650 2300 2    50   Input ~ 0
-TD0
-Text HLabel 9650 2400 2    50   Input ~ 0
-TD1
 Wire Wire Line
 	9650 2400 9350 2400
@@
 Wire Wire Line
 	8650 3100 8650 3000
-Text HLabel 5250 4800 2    50   Input ~ 0
-TRST
-Text HLabel 5250 4900 2    50   Input ~ 0
-SRST
-Text HLabel 5250 5000 2    50   Input ~ 0
-TCK
-Text HLabel 5250 5100 2    50   Input ~ 0
-TMS
-Text HLabel 5250 5200 2    50   Input ~ 0
-TD0
-Text HLabel 5250 5300 2    50   Input ~ 0
-TD1
 Wire Wire Line
 	5250 4800 5050 4800
@@
 Wire Wire Line
 	8750 1250 8750 1100
+Wire Wire Line
+	9350 2100 9650 2100
+Wire Wire Line
+	9350 1800 9650 1800
+Text Label 9500 1700 0    50   ~ 0
+TRST1
+Text Label 9500 1800 0    50   ~ 0
+SRST1
+Text Label 9500 2100 0    50   ~ 0
+TCK1
+Text Label 9500 2200 0    50   ~ 0
+TMS1
+Text Label 9500 2300 0    50   ~ 0
+TD01
+Text Label 9500 2400 0    50   ~ 0
+TD11
+Wire Wire Line
+	9350 2000 9700 2000
+Wire Wire Line
+	10100 2000 10000 2000
+$Comp
+L power:GND #PWR?
+U 1 1 5EA4A411
+P 10100 2000
+F 0 "#PWR?" H 10100 1750 50  0001 C CNN
+F 1 "GND" V 10105 1872 50  0000 R CNN
+F 2 "" H 10100 2000 50  0001 C CNN
+F 3 "" H 10100 2000 50  0001 C CNN
+	1    10100 2000
+	0    -1   -1   0
+$EndComp
 $Comp
 L Device:R R?
 U 1 1 5EA45BC4
-P 9700 2000
-F 0 "R?" V 9493 2000 50  0001 C CNN
-F 1 "510" V 9585 2000 50  0000 C CNN
-F 2 "" V 9630 2000 50  0001 C CNN
-F 3 "~" H 9700 2000 50  0001 C CNN
-	1    9700 2000
+P 9850 2000
+F 0 "R?" V 9643 2000 50  0001 C CNN
+F 1 "510" V 9735 2000 50  0000 C CNN
+F 2 "" V 9780 2000 50  0001 C CNN
+F 3 "~" H 9850 2000 50  0001 C CNN
+	1    9850 2000
 	0    1    1    0
 $EndComp
-Wire Wire Line
-	9350 2100 9650 2100
-Wire Wire Line
-	9350 1800 9650 1800
-$Comp
-L power:GND #PWR?
-U 1 1 5EA4A411
-P 10050 2000
-F 0 "#PWR?" H 10050 1750 50  0001 C CNN
-F 1 "GND" V 10055 1872 50  0000 R CNN
-F 2 "" H 10050 2000 50  0001 C CNN
-F 3 "" H 10050 2000 50  0001 C CNN
-	1    10050 2000
-	0    -1   -1   0
-$EndComp
-Wire Wire Line
-	9350 2000 9550 2000
-Wire Wire Line
-	10050 2000 9850 2000
+Text Label 5250 4800 0    50   ~ 0
+TRST
+Text Label 5250 4900 0    50   ~ 0
+SRST
+Text Label 5250 5000 0    50   ~ 0
+TCK
+Text Label 5250 5100 0    50   ~ 0
+TMS
+Text Label 5250 5200 0    50   ~ 0
+TD0
+Text Label 5250 5300 0    50   ~ 0
+TD1
 $EndSCHEMATC

Commit message: Add files via upload
Other:
- note added: "JTAG"
- note added: "MICROPROCESADOR"
- note added: "RESET"
- moved on the sheet: C?, J?, R?, SW?, U?, Y?

Commit message: Add files via upload
Parts:
- gave numbers to parts that had none: 16
Changed lines of the file:
@@
 P 3700 2100
 AR Path="/5E9F4EED" Ref="C?"  Part="1"
-AR Path="/5E9DF408/5E9F4EED" Ref="C?"  Part="1"
-F 0 "C?" H 3815 2146 50  0000 L CNN
+AR Path="/5E9DF408/5E9F4EED" Ref="C28"  Part="1"
+F 0 "C28" H 3815 2146 50  0000 L CNN
 F 1 "0.1uM" H 3815 2055 50  0000 L CNN
 F 2 "" H 3738 1950 50  0001 C CNN
@@
 P 4000 2100
 AR Path="/5E9F4EF3" Ref="C?"  Part="1"
-AR Path="/5E9DF408/5E9F4EF3" Ref="C?"  Part="1"
-F 0 "C?" H 4115 2146 50  0000 L CNN
+AR Path="/5E9DF408/5E9F4EF3" Ref="C29"  Part="1"
+F 0 "C29" H 4115 2146 50  0000 L CNN
 F 1 "0.1uM" H 4115 2055 50  0000 L CNN
 F 2 "" H 4038 1950 50  0001 C CNN
@@
 P 4300 2100
 AR Path="/5E9F4EF9" Ref="C?"  Part="1"
-AR Path="/5E9DF408/5E9F4EF9" Ref="C?"  Part="1"
-F 0 "C?" H 4415 2146 50  0000 L CNN
+AR Path="/5E9DF408/5E9F4EF9" Ref="C30"  Part="1"
+F 0 "C30" H 4415 2146 50  0000 L CNN
 F 1 "0.1uM" H 4415 2055 50  0000 L CNN
 F 2 "" H 4338 1950 50  0001 C CNN
@@
 P 4650 2100
 AR Path="/5E9F4EFF" Ref="C?"  Part="1"
-AR Path="/5E9DF408/5E9F4EFF" Ref="C?"  Part="1"
-F 0 "C?" H 4765 2146 50  0000 L CNN
+AR Path="/5E9DF408/5E9F4EFF" Ref="C32"  Part="1"
+F 0 "C32" H 4765 2146 50  0000 L CNN
 F 1 "0.1uM" H 4765 2055 50  0000 L CNN
 F 2 "" H 4688 1950 50  0001 C CNN
@@
 P 5000 2100
 AR Path="/5E9F4F05" Ref="C?"  Part="1"
-AR Path="/5E9DF408/5E9F4F05" Ref="C?"  Part="1"
-F 0 "C?" H 5115 2146 50  0000 L CNN
+AR Path="/5E9DF408/5E9F4F05" Ref="C33"  Part="1"
+F 0 "C33" H 5115 2146 50  0000 L CNN
 F 1 "0.1uM" H 5115 2055 50  0000 L CNN
 F 2 "" H 5038 1950 50  0001 C CNN
@@
 P 5350 2100
 AR Path="/5E9F4F1D" Ref="C?"  Part="1"
-AR Path="/5E9DF408/5E9F4F1D" Ref="C?"  Part="1"
-F 0 "C?" H 5465 2146 50  0000 L CNN
+AR Path="/5E9DF408/5E9F4F1D" Ref="C35"  Part="1"
+F 0 "C35" H 5465 2146 50  0000 L CNN
 F 1 "0.1uM" H 5465 2055 50  0000 L CNN
 F 2 "" H 5388 1950 50  0001 C CNN
@@
 P 4450 2400
 AR Path="/5E9F4F26" Ref="#PWR?"  Part="1"
-AR Path="/5E9DF408/5E9F4F26" Ref="#PWR?"  Part="1"
-F 0 "#PWR?" H 4450 2150 50  0001 C CNN
+AR Path="/5E9DF408/5E9F4F26" Ref="#PWR0151"  Part="1"
+F 0 "#PWR0151" H 4450 2150 50  0001 C CNN
 F 1 "GND" H 4455 2227 50  0000 C CNN
 F 2 "" H 4450 2400 50  0001 C CNN
@@
 P 3400 5950
 AR Path="/5E9F4F3F" Ref="#PWR?"  Part="1"
-AR Path="/5E9DF408/5E9F4F3F" Ref="#PWR?"  Part="1"
-F 0 "#PWR?" H 3400 5700 50  0001 C CNN
+AR Path="/5E9DF408/5E9F4F3F" Ref="#PWR0152"  Part="1"
+F 0 "#PWR0152" H 3400 5700 50  0001 C CNN
 F 1 "GND" H 3405 5777 50  0000 C CNN
 F 2 "" H 3400 5950 50  0001 C CNN
@@
 P 9000 1600
 AR Path="/5EA16163" Ref="R?"  Part="1"
-AR Path="/5E9DF408/5EA16163" Ref="R?"  Part="1"
-F 0 "R?" V 8793 1600 50  0000 C CNN
+AR Path="/5E9DF408/5EA16163" Ref="R21"  Part="1"
+F 0 "R21" V 8793 1600 50  0000 C CNN
 F 1 "10k" V 8884 1600 50  0000 C CNN
 F 2 "" V 8930 1600 50  0001 C CNN
@@
 P 8650 1750
 AR Path="/5EA16169" Ref="C?"  Part="1"
-AR Path="/5E9DF408/5EA16169" Ref="C?"  Part="1"
-F 0 "C?" H 8765 1796 50  0000 L CNN
+AR Path="/5E9DF408/5EA16169" Ref="C36"  Part="1"
+F 0 "C36" H 8765 1796 50  0000 L CNN
 F 1 "0.1uF" H 8765 1705 50  0000 L CNN
 F 2 "" H 8688 1600 50  0001 C CNN
@@
 P 8650 2000
 AR Path="/5EA16173" Ref="#PWR?"  Part="1"
-AR Path="/5E9DF408/5EA16173" Ref="#PWR?"  Part="1"
-F 0 "#PWR?" H 8650 1750 50  0001 C CNN
+AR Path="/5E9DF408/5EA16173" Ref="#PWR0153"  Part="1"
+F 0 "#PWR0153" H 8650 1750 50  0001 C CNN
 F 1 "GND" H 8655 1827 50  0000 C CNN
 F 2 "" H 8650 2000 50  0001 C CNN
@@
 P 8300 1900
 AR Path="/5EA1617B" Ref="SW?"  Part="1"
-AR Path="/5E9DF408/5EA1617B" Ref="SW?"  Part="1"
-F 0 "SW?" V 8346 1852 50  0000 R CNN
+AR Path="/5E9DF408/5EA1617B" Ref="SW3"  Part="1"
+F 0 "SW3" V 8346 1852 50  0000 R CNN
 F 1 "SW_Push" V 8255 1852 50  0000 R CNN
 F 2 "" H 8300 2100 50  0001 C CNN
@@
 P 8300 2100
 AR Path="/5EA16181" Ref="#PWR?"  Part="1"
-AR Path="/5E9DF408/5EA16181" Ref="#PWR?"  Part="1"
-F 0 "#PWR?" H 8300 1850 50  0001 C CNN
+AR Path="/5E9DF408/5EA16181" Ref="#PWR0154"  Part="1"
+F 0 "#PWR0154" H 8300 1850 50  0001 C CNN
 F 1 "GND" H 8305 1927 50  0000 C CNN
 F 2 "" H 8300 2100 50  0001 C CNN
@@
 P 3450 4150
 AR Path="/5E9F4F50" Ref="U?"  Part="1"
-AR Path="/5E9DF408/5E9F4F50" Ref="U?"  Part="1"
-F 0 "U?" H 3450 5931 50  0000 C CNN
+AR Path="/5E9DF408/5E9F4F50" Ref="U10"  Part="1"
+F 0 "U10" H 3450 5931 50  0000 C CNN
 F 1 "STM32L052C6Tx" H 3927 5840 50  0000 C CNN
 F 2 "Package_QFP:LQFP-48_7x7mm_P0.5mm" H 2950 2650 50  0001 R CNN
@@
 	4850 4400 4850 4300
 $Comp
-L power:GND #PWR?
+L power:GND #PWR0155
 U 1 1 5EA4D9B8
 P 4850 4400
-F 0 "#PWR?" H 4850 4150 50  0001 C CNN
+F 0 "#PWR0155" H 4850 4150 50  0001 C CNN
 F 1 "GND" H 4855 4227 50  0000 C CNN
 F 2 "" H 4850 4400 50  0001 C CNN
@@
 	5150 3900 5150 3850
 $Comp
-L Device:Crystal Y?
+L Device:Crystal Y1
 U 1 1 5EA3D14C
 P 4850 3650
-F 0 "Y?" H 4850 3421 50  0000 C CNN
+F 0 "Y1" H 4850 3421 50  0000 C CNN
 F 1 "24M" H 4850 3473 50  0000 C CNN
 F 2 "" H 4850 3650 50  0001 C CNN
@@
 $EndComp
 $Comp
-L Device:C C?
+L Device:C C34
 U 1 1 5EA3BE5E
 P 5150 4000
-F 0 "C?" H 5035 3954 50  0000 R CNN
+F 0 "C34" H 5035 3954 50  0000 R CNN
 F 1 "2.2uF" H 5035 4045 50  0000 R CNN
 F 2 "" H 5188 3850 50  0001 C CNN
@@
 USART_1
 $Comp
-L Device:C C?
+L Device:C C31
 U 1 1 5EA3C6AF
 P 4500 4000
-F 0 "C?" H 4385 3954 50  0000 R CNN
+F 0 "C31" H 4385 3954 50  0000 R CNN
 F 1 "2.2uF" H 4385 4045 50  0000 R CNN
 F 2 "" H 4538 3850 50  0001 C CNN
@@
 Connection ~ 4500 3650
 $Comp
-L Device:R R?
+L Device:R R20
 U 1 1 5EA5A535
 P 4500 3150
-F 0 "R?" V 4293 3150 50  0000 C CNN
+F 0 "R20" V 4293 3150 50  0000 C CNN
 F 1 "10k" V 4384 3150 50  0000 C CNN
 F 2 "" V 4430 3150 50  0001 C CNN
@@
 P 4900 3150
 AR Path="/5E9F4F2F" Ref="#PWR?"  Part="1"
-AR Path="/5E9DF408/5E9F4F2F" Ref="#PWR?"  Part="1"
-F 0 "#PWR?" H 4900 2900 50  0001 C CNN
+AR Path="/5E9DF408/5E9F4F2F" Ref="#PWR0156"  Part="1"
+F 0 "#PWR0156" H 4900 2900 50  0001 C CNN
 F 1 "GND" H 4905 2977 50  0000 C CNN
 F 2 "" H 4900 3150 50  0001 C CNN
@@
 	4050 5550 4250 5550
 $Comp
-L power:+3.3V #PWR?
+L power:+3.3V #PWR0157
 U 1 1 5E9CEFDA
 P 9350 1450
-F 0 "#PWR?" H 9350 1300 50  0001 C CNN
+F 0 "#PWR0157" H 9350 1300 50  0001 C CNN
 F 1 "+3.3V" H 9365 1623 50  0000 C CNN
 F 2 "" H 9350 1450 50  0001 C CNN
@@
 	9350 1600 9350 1450
 $Comp
-L power:+3.3V #PWR?
+L power:+3.3V #PWR0158
 U 1 1 5E9D4164
 P 3350 1700
-F 0 "#PWR?" H 3350 1550 50  0001 C CNN
+F 0 "#PWR0158" H 3350 1550 50  0001 C CNN
 F 1 "+3.3V" H 3365 1873 50  0000 C CNN
 F 2 "" H 3350 1700 50  0001 C CNN
@@
 Connection ~ 3350 1950
 $Comp
-L power:GND #PWR?
+L power:GND #PWR0159
 U 1 1 5EA4A411
 P 10250 4750
-F 0 "#PWR?" H 10250 4500 50  0001 C CNN
+F 0 "#PWR0159" H 10250 4500 50  0001 C CNN
 F 1 "GND" V 10255 4622 50  0000 R CNN
 F 2 "" H 10250 4750 50  0001 C CNN
@@
 TD1
 $Comp
-L Device:R R?
+L Device:R R22
 U 1 1 5EA45BC4
 P 10000 4750
-F 0 "R?" V 9793 4750 50  0001 C CNN
+F 0 "R22" V 9793 4750 50  0001 C CNN
 F 1 "510" V 9885 4750 50  0000 C CNN
 F 2 "" V 9930 4750 50  0001 C CNN
@@
 	8800 4150 8800 4000
 $Comp
-L power:+3.3V #PWR?
+L power:+3.3V #PWR0160
 U 1 1 5E9CE6D3
 P 8900 3850
-F 0 "#PWR?" H 8900 3700 50  0001 C CNN
+F 0 "#PWR0160" H 8900 3700 50  0001 C CNN
 F 1 "+3.3V" H 8915 4023 50  0000 C CNN
 F 2 "" H 8900 3850 50  0001 C CNN
@@
 	8800 5850 8800 5750
 $Comp
-L power:GND #PWR?
+L power:GND #PWR0161
 U 1 1 5E997632
 P 8800 5850
-F 0 "#PWR?" H 8800 5600 50  0001 C CNN
+F 0 "#PWR0161" H 8800 5600 50  0001 C CNN
 F 1 "GND" H 8805 5677 50  0000 C CNN
 F 2 "" H 8800 5850 50  0001 C CNN
@@
 	9800 5150 9500 5150
 $Comp
-L Connector:Conn_ARM_JTAG_SWD_20 J?
+L Connector:Conn_ARM_JTAG_SWD_20 J9
 U 1 1 5E986004
 P 8900 4950
-F 0 "J?" H 8371 4996 50  0000 R CNN
+F 0 "J9" H 8371 4996 50  0000 R CNN
 F 1 "Conn_ARM_JTAG_SWD_20" H 8371 4905 50  0000 R CNN
 F 2 "" H 9350 3900 50  0001 L TNN

Commit message: Add files via upload
Parts:
- C28, C29, C30, C31, C32, C33, C34, C35, C36: footprint (none) -> Capacitor_SMD:C_0603_1608Metric_Pad1.05x0.95mm_HandSolder
- J9: footprint (none) -> Connector_PinSocket_1.27mm:PinSocket_2x10_P1.27mm_Vertical
- R20, R21, R22: footprint (none) -> Resistor_SMD:R_0201_0603Metric
- Y1: footprint (none) -> Crystal:Crystal_HC35-U
Changed lines of the file:
@@
 F 0 "C28" H 3815 2146 50  0000 L CNN
 F 1 "0.1uM" H 3815 2055 50  0000 L CNN
-F 2 "" H 3738 1950 50  0001 C CNN
+F 2 "Capacitor_SMD:C_0603_1608Metric_Pad1.05x0.95mm_HandSolder" H 3738 1950 50  0001 C CNN
 F 3 "~" H 3700 2100 50  0001 C CNN
 	1    3700 2100
@@
 F 0 "C29" H 4115 2146 50  0000 L CNN
 F 1 "0.1uM" H 4115 2055 50  0000 L CNN
-F 2 "" H 4038 1950 50  0001 C CNN
+F 2 "Capacitor_SMD:C_0603_1608Metric_Pad1.05x0.95mm_HandSolder" H 4038 1950 50  0001 C CNN
 F 3 "~" H 4000 2100 50  0001 C CNN
 	1    4000 2100
@@
 F 0 "C30" H 4415 2146 50  0000 L CNN
 F 1 "0.1uM" H 4415 2055 50  0000 L CNN
-F 2 "" H 4338 1950 50  0001 C CNN
+F 2 "Capacitor_SMD:C_0603_1608Metric_Pad1.05x0.95mm_HandSolder" H 4338 1950 50  0001 C CNN
 F 3 "~" H 4300 2100 50  0001 C CNN
 	1    4300 2100
@@
 F 0 "C32" H 4765 2146 50  0000 L CNN
 F 1 "0.1uM" H 4765 2055 50  0000 L CNN
-F 2 "" H 4688 1950 50  0001 C CNN
+F 2 "Capacitor_SMD:C_0603_1608Metric_Pad1.05x0.95mm_HandSolder" H 4688 1950 50  0001 C CNN
 F 3 "~" H 4650 2100 50  0001 C CNN
 	1    4650 2100
@@
 F 0 "C33" H 5115 2146 50  0000 L CNN
 F 1 "0.1uM" H 5115 2055 50  0000 L CNN
-F 2 "" H 5038 1950 50  0001 C CNN
+F 2 "Capacitor_SMD:C_0603_1608Metric_Pad1.05x0.95mm_HandSolder" H 5038 1950 50  0001 C CNN
 F 3 "~" H 5000 2100 50  0001 C CNN
 	1    5000 2100
@@
 F 0 "C35" H 5465 2146 50  0000 L CNN
 F 1 "0.1uM" H 5465 2055 50  0000 L CNN
-F 2 "" H 5388 1950 50  0001 C CNN
+F 2 "Capacitor_SMD:C_0603_1608Metric_Pad1.05x0.95mm_HandSolder" H 5388 1950 50  0001 C CNN
 F 3 "~" H 5350 2100 50  0001 C CNN
 	1    5350 2100
@@
 F 0 "R21" V 8793 1600 50  0000 C CNN
 F 1 "10k" V 8884 1600 50  0000 C CNN
-F 2 "" V 8930 1600 50  0001 C CNN
+F 2 "Resistor_SMD:R_0201_0603Metric" V 8930 1600 50  0001 C CNN
 F 3 "~" H 9000 1600 50  0001 C CNN
 	1    9000 1600
@@
 F 0 "C36" H 8765 1796 50  0000 L CNN
 F 1 "0.1uF" H 8765 1705 50  0000 L CNN
-F 2 "" H 8688 1600 50  0001 C CNN
+F 2 "Capacitor_SMD:C_0603_1608Metric_Pad1.05x0.95mm_HandSolder" H 8688 1600 50  0001 C CNN
 F 3 "~" H 8650 1750 50  0001 C CNN
 	1    8650 1750
@@
 F 0 "Y1" H 4850 3421 50  0000 C CNN
 F 1 "24M" H 4850 3473 50  0000 C CNN
-F 2 "" H 4850 3650 50  0001 C CNN
+F 2 "Crystal:Crystal_HC35-U" H 4850 3650 50  0001 C CNN
 F 3 "~" H 4850 3650 50  0001 C CNN
 	1    4850 3650
@@
 F 0 "C34" H 5035 3954 50  0000 R CNN
 F 1 "2.2uF" H 5035 4045 50  0000 R CNN
-F 2 "" H 5188 3850 50  0001 C CNN
+F 2 "Capacitor_SMD:C_0603_1608Metric_Pad1.05x0.95mm_HandSolder" H 5188 3850 50  0001 C CNN
 F 3 "~" H 5150 4000 50  0001 C CNN
 	1    5150 4000
@@
 F 0 "C31" H 4385 3954 50  0000 R CNN
 F 1 "2.2uF" H 4385 4045 50  0000 R CNN
-F 2 "" H 4538 3850 50  0001 C CNN
+F 2 "Capacitor_SMD:C_0603_1608Metric_Pad1.05x0.95mm_HandSolder" H 4538 3850 50  0001 C CNN
 F 3 "~" H 4500 4000 50  0001 C CNN
 	1    4500 4000
@@
 F 0 "R20" V 4293 3150 50  0000 C CNN
 F 1 "10k" V 4384 3150 50  0000 C CNN
-F 2 "" V 4430 3150 50  0001 C CNN
+F 2 "Resistor_SMD:R_0201_0603Metric" V 4430 3150 50  0001 C CNN
 F 3 "~" H 4500 3150 50  0001 C CNN
 	1    4500 3150
@@
 F 0 "R22" V 9793 4750 50  0001 C CNN
 F 1 "510" V 9885 4750 50  0000 C CNN
-F 2 "" V 9930 4750 50  0001 C CNN
+F 2 "Resistor_SMD:R_0201_0603Metric" V 9930 4750 50  0001 C CNN
 F 3 "~" H 10000 4750 50  0001 C CNN
 	1    10000 4750
@@
 F 0 "J9" H 8371 4996 50  0000 R CNN
 F 1 "Conn_ARM_JTAG_SWD_20" H 8371 4905 50  0000 R CNN
-F 2 "" H 9350 3900 50  0001 L TNN
+F 2 "Connector_PinSocket_1.27mm:PinSocket_2x10_P1.27mm_Vertical" H 9350 3900 50  0001 L TNN
 F 3 "http://infocenter.arm.com/help/topic/com.arm.doc.dui0499b/DUI0499B_system_design_reference.pdf" V 8550 3700 50  0001 C CNN
 	1    8900 4950

Commit message: Add files via upload
Parts:
- C31: footprint Capacitor_SMD:C_0603_1608Metric_Pad1.05x0.95mm_HandSolder -> Inductor_SMD:L_2010_5025Metric_Pad1.52x2.65mm_HandSolder
Changed lines of the file:
@@
 F 0 "C31" H 4385 3954 50  0000 R CNN
 F 1 "2.2uF" H 4385 4045 50  0000 R CNN
-F 2 "Capacitor_SMD:C_0603_1608Metric_Pad1.05x0.95mm_HandSolder" H 4538 3850 50  0001 C CNN
+F 2 "Inductor_SMD:L_2010_5025Metric_Pad1.52x2.65mm_HandSolder" H 4538 3850 50  0001 C CNN
 F 3 "~" H 4500 4000 50  0001 C CNN
 	1    4500 4000

Commit message: Add files via upload
Parts:
- SW3: footprint (none) -> Button_Switch_SMD:SW_DIP_SPSTx05_Slide_6.7x14.26mm_W6.73mm_P2.54mm_LowProfile_JPin
Changed lines of the file:
@@
 F 0 "SW3" V 8346 1852 50  0000 R CNN
 F 1 "SW_Push" V 8255 1852 50  0000 R CNN
-F 2 "" H 8300 2100 50  0001 C CNN
+F 2 "Button_Switch_SMD:SW_DIP_SPSTx05_Slide_6.7x14.26mm_W6.73mm_P2.54mm_LowProfile_JPin" H 8300 2100 50  0001 C CNN
 F 3 "~" H 8300 2100 50  0001 C CNN
 	1    8300 1900
