File: proyecto/Microcontrolador.sch (KiCad schematic (older format))
At the start: 16 parts, among them J9 Conn_ARM_JTAG_SWD_20, SW3 SW_Push, U10 STM32L052C6Tx, Y1 24M

Commit message: Add files via upload
Parts:
- SW3: footprint Button_Switch_SMD:SW_DIP_SPSTx05_Slide_6.7x14.26mm_W6.73mm_P2.54mm_LowProfile_JPin -> Button_Switch_SMD:SW_DIP_SPSTx01_Slide_6.7x4.1mm_W6.73mm_P2.54mm_LowProfile_JPin
Connections:
- net labels added: +3V8
- net labels removed: +3.3V, SRST, TCK, TD0, TD1, TMS, TRST
Changed lines of the file:
@@
 F 0 "SW3" V 8346 1852 50  0000 R CNN
 F 1 "SW_Push" V 8255 1852 50  0000 R CNN
-F 2 "Button_Switch_SMD:SW_DIP_SPSTx05_Slide_6.7x14.26mm_W6.73mm_P2.54mm_LowProfile_JPin" H 8300 2100 50  0001 C CNN
+F 2 "Button_Switch_SMD:SW_DIP_SPSTx01_Slide_6.7x4.1mm_W6.73mm_P2.54mm_LowProfile_JPin" H 8300 2100 50  0001 C CNN
 F 3 "~" H 8300 2100 50  0001 C CNN
 	1    8300 1900
@@
 Wire Wire Line
 	4050 5550 4250 5550
-$Comp
-L power:+3.3V #PWR0157
-U 1 1 5E9CEFDA
-P 9350 1450
-F 0 "#PWR0157" H 9350 1300 50  0001 C CNN
-F 1 "+3.3V" H 9365 1623 50  0000 C CNN
-F 2 "" H 9350 1450 50  0001 C CNN
-F 3 "" H 9350 1450 50  0001 C CNN
-	1    9350 1450
-	1    0    0    -1
-$EndComp
 Wire Wire Line
 	9150 1600 9350 1600
 Wire Wire Line
 	9350 1600 9350 1450
-$Comp
-L power:+3.3V #PWR0158
-U 1 1 5E9D4164
-P 3350 1700
-F 0 "#PWR0158" H 3350 1550 50  0001 C CNN
-F 1 "+3.3V" H 3365 1873 50  0000 C CNN
-F 2 "" H 3350 1700 50  0001 C CNN
-F 3 "" H 3350 1700 50  0001 C CNN
-	1    3350 1700
-	1    0    0    -1
-$EndComp
 Wire Wire Line
 	3350 1700 3350 1950
@@
 $EndComp
 Text Label 4250 5050 0    50   ~ 0
-TRST
+TRST1
 Text Label 4250 5150 0    50   ~ 0
-SRST
+SRST1
 Text Label 4250 5250 0    50   ~ 0
-TCK
+TCK1
 Text Label 4250 5350 0    50   ~ 0
-TMS
+TMS1
 Text Label 4250 5450 0    50   ~ 0
-TD0
+TD01
 Text Label 4250 5550 0    50   ~ 0
-TD1
+TD11
 $Comp
 L Device:R R22
@@
 Wire Wire Line
 	8800 4150 8800 4000
-$Comp
-L power:+3.3V #PWR0160
-U 1 1 5E9CE6D3
-P 8900 3850
-F 0 "#PWR0160" H 8900 3700 50  0001 C CNN
-F 1 "+3.3V" H 8915 4023 50  0000 C CNN
-F 2 "" H 8900 3850 50  0001 C CNN
-F 3 "" H 8900 3850 50  0001 C CNN
-	1    8900 3850
-	1    0    0    -1
-$EndComp
 Wire Wire Line
 	8900 4150 8900 4000
@@
 Text Notes 500  7750 0    50   ~ 0
 MICROPROCESADOR
+$Comp
+L power:+3V8 #PWR0157
+U 1 1 5EB6B814
+P 3350 1700
+F 0 "#PWR0157" H 3350 1550 50  0001 C CNN
+F 1 "+3V8" H 3365 1873 50  0000 C CNN
+F 2 "" H 3350 1700 50  0001 C CNN
+F 3 "" H 3350 1700 50  0001 C CNN
+	1    3350 1700
+	1    0    0    -1
+$EndComp
+$Comp
+L power:+3V8 #PWR0158
+U 1 1 5EB6BCC5
+P 8900 3850
+F 0 "#PWR0158" H 8900 3700 50  0001 C CNN
+F 1 "+3V8" H 8915 4023 50  0000 C CNN
+F 2 "" H 8900 3850 50  0001 C CNN
+F 3 "" H 8900 3850 50  0001 C CNN
+	1    8900 3850
+	1    0    0    -1
+$EndComp
+$Comp
+L power:+3V8 #PWR0160
+U 1 1 5EB6C42F
+P 9350 1450
+F 0 "#PWR0160" H 9350 1300 50  0001 C CNN
+F 1 "+3V8" H 9365 1623 50  0000 C CNN
+F 2 "" H 9350 1450 50  0001 C CNN
+F 3 "" H 9350 1450 50  0001 C CNN
+	1    9350 1450
+	1    0    0    -1
+$EndComp
 $EndSCHEMATC

Commit message: Add files via upload
Changed lines of the file:
@@
 	4050 5350 4250 5350
 Wire Wire Line
-	4250 5450 4050 5450
-Wire Wire Line
-	4050 5550 4250 5550
+	4250 5550 4050 5550
 Wire Wire Line
 	9150 1600 9350 1600
@@
 Text Label 4250 5150 0    50   ~ 0
 SRST1
-Text Label 4250 5250 0    50   ~ 0
+Text Label 4250 5450 0    50   ~ 0
 TCK1
-Text Label 4250 5350 0    50   ~ 0
-TMS1
-Text Label 4250 5450 0    50   ~ 0
-TD01
-Text Label 4250 5550 0    50   ~ 0
-TD11
 $Comp
 L Device:R R22
@@
 	1    0    0    -1
 $EndComp
+Wire Wire Line
+	4050 5450 4250 5450
+Text Label 4250 5250 0    50   ~ 0
+TD11
+Text Label 4250 5550 0    50   ~ 0
+TD01
+Text Label 4250 5350 0    50   ~ 0
+TMS1
 $EndSCHEMATC

Commit message: Add files via upload
Connections:
- net labels removed: PH_EN34
- wire segments 82 -> 81
Other:
- moved on the sheet: C31, C34, Y1
Changed lines of the file:
@@
 	4200 4550 4050 4550
 Wire Wire Line
-	2850 4950 2650 4950
-Wire Wire Line
-	2850 4850 2650 4850
+	2850 5550 2650 5550
+Wire Wire Line
+	2850 5450 2650 5450
 Wire Wire Line
 	2850 4650 2650 4650
@@
 	2850 4450 2650 4450
 Wire Wire Line
-	2850 4350 2650 4350
-Wire Wire Line
-	2850 4250 2650 4250
-Wire Wire Line
-	2650 5050 2850 5050
-Wire Wire Line
-	2850 4150 2650 4150
+	2850 5350 2650 5350
+Wire Wire Line
+	4050 4350 4250 4350
+Wire Wire Line
+	4050 4450 4250 4450
 $Comp
 L MCU_ST_STM32L0:STM32L052C6Tx U?
@@
 	-1   0    0    -1
 $EndComp
-Text HLabel 2650 4150 0    50   Input ~ 0
+Text HLabel 4250 4450 2    50   Input ~ 0
+PH_3A
+Text HLabel 4250 4350 2    50   Input ~ 0
+PH_4A
+Text HLabel 2650 5350 0    50   Input ~ 0
+PH_EN12
+Text HLabel 2650 5450 0    50   Input ~ 0
 PH_1A
-Text HLabel 2650 4250 0    50   Input ~ 0
+Text HLabel 2650 5550 0    50   Input ~ 0
 PH_2A
-Text HLabel 2650 4350 0    50   Input ~ 0
-PH_EN12
-Text HLabel 2650 4850 0    50   Input ~ 0
-PH_3A
-Text HLabel 2650 4950 0    50   Input ~ 0
-PH_4A
-Text HLabel 2650 5050 0    50   Input ~ 0
-PH_EN34
 Text HLabel 4200 4550 2    50   Input ~ 0
 MOSI
@@
 Text HLabel 4200 4750 2    50   Input ~ 0
 USART_2
-Wire Wire Line
-	4850 4300 5150 4300
-Connection ~ 4850 4300
-Wire Wire Line
-	4850 4400 4850 4300
-$Comp
-L power:GND #PWR0155
-U 1 1 5EA4D9B8
-P 4850 4400
-F 0 "#PWR0155" H 4850 4150 50  0001 C CNN
-F 1 "GND" H 4855 4227 50  0000 C CNN
-F 2 "" H 4850 4400 50  0001 C CNN
-F 3 "" H 4850 4400 50  0001 C CNN
-	1    4850 4400
-	1    0    0    -1
-$EndComp
-Wire Wire Line
-	5150 4300 5150 4150
-Wire Wire Line
-	4500 4300 4850 4300
-Wire Wire Line
-	4700 3650 4500 3650
-Wire Wire Line
-	5150 3850 5150 3650
-Connection ~ 5150 3850
-Wire Wire Line
-	5150 3900 5150 3850
-$Comp
-L Device:Crystal Y1
-U 1 1 5EA3D14C
-P 4850 3650
-F 0 "Y1" H 4850 3421 50  0000 C CNN
-F 1 "24M" H 4850 3473 50  0000 C CNN
-F 2 "Crystal:Crystal_HC35-U" H 4850 3650 50  0001 C CNN
-F 3 "~" H 4850 3650 50  0001 C CNN
-	1    4850 3650
-	-1   0    0    1
-$EndComp
-$Comp
-L Device:C C34
-U 1 1 5EA3BE5E
-P 5150 4000
-F 0 "C34" H 5035 3954 50  0000 R CNN
-F 1 "2.2uF" H 5035 4045 50  0000 R CNN
-F 2 "Capacitor_SMD:C_0603_1608Metric_Pad1.05x0.95mm_HandSolder" H 5188 3850 50  0001 C CNN
-F 3 "~" H 5150 4000 50  0001 C CNN
-	1    5150 4000
-	-1   0    0    1
-$EndComp
-Wire Wire Line
-	4500 3650 4500 3850
 Text HLabel 4200 4650 2    50   Input ~ 0
 USART_1
-$Comp
-L Device:C C31
-U 1 1 5EA3C6AF
-P 4500 4000
-F 0 "C31" H 4385 3954 50  0000 R CNN
-F 1 "2.2uF" H 4385 4045 50  0000 R CNN
-F 2 "Inductor_SMD:L_2010_5025Metric_Pad1.52x2.65mm_HandSolder" H 4538 3850 50  0001 C CNN
-F 3 "~" H 4500 4000 50  0001 C CNN
-	1    4500 4000
-	-1   0    0    1
-$EndComp
-Wire Wire Line
-	4500 4150 4500 4300
-Wire Wire Line
-	4500 3450 4050 3450
-Wire Wire Line
-	4500 3450 4500 3650
-Connection ~ 4500 3650
 $Comp
 L Device:R R20
@@
 	0    1    1    0
 $EndComp
-Connection ~ 5150 3650
-Wire Wire Line
-	5150 3650 5000 3650
-Wire Wire Line
-	5150 3350 5150 3650
-Wire Wire Line
-	4050 3350 5150 3350
 $Comp
 L power:GND #PWR?
@@
 Text Label 4250 5350 0    50   ~ 0
 TMS1
+Wire Wire Line
+	5650 4300 5950 4300
+Connection ~ 5650 4300
+Wire Wire Line
+	5650 4400 5650 4300
+$Comp
+L power:GND #PWR0155
+U 1 1 5EA4D9B8
+P 5650 4400
+F 0 "#PWR0155" H 5650 4150 50  0001 C CNN
+F 1 "GND" H 5655 4227 50  0000 C CNN
+F 2 "" H 5650 4400 50  0001 C CNN
+F 3 "" H 5650 4400 50  0001 C CNN
+	1    5650 4400
+	1    0    0    -1
+$EndComp
+Wire Wire Line
+	5300 4300 5650 4300
+$Comp
+L Device:C C31
+U 1 1 5EA3C6AF
+P 5300 4000
+F 0 "C31" H 5185 3954 50  0000 R CNN
+F 1 "2.2uF" H 5185 4045 50  0000 R CNN
+F 2 "Inductor_SMD:L_2010_5025Metric_Pad1.52x2.65mm_HandSolder" H 5338 3850 50  0001 C CNN
+F 3 "~" H 5300 4000 50  0001 C CNN
+	1    5300 4000
+	-1   0    0    1
+$EndComp
+Wire Wire Line
+	5950 3850 5950 3650
+Wire Wire Line
+	5950 3350 5950 3650
+Wire Wire Line
+	5300 3650 5300 3850
+Wire Wire Line
+	5300 3450 5300 3650
+Connection ~ 5300 3650
+Connection ~ 5950 3650
+Wire Wire Line
+	5300 4150 5300 4300
+$Comp
+L Device:C C34
+U 1 1 5EA3BE5E
+P 5950 4000
+F 0 "C34" H 5835 3954 50  0000 R CNN
+F 1 "2.2uF" H 5835 4045 50  0000 R CNN
+F 2 "Capacitor_SMD:C_0603_1608Metric_Pad1.05x0.95mm_HandSolder" H 5988 3850 50  0001 C CNN
+F 3 "~" H 5950 4000 50  0001 C CNN
+	1    5950 4000
+	-1   0    0    1
+$EndComp
+Wire Wire Line
+	5950 3900 5950 3850
+Connection ~ 5950 3850
+Wire Wire Line
+	5950 4300 5950 4150
+Wire Wire Line
+	4050 3350 5950 3350
+Wire Wire Line
+	4050 3450 5300 3450
+Wire Wire Line
+	5500 3650 5300 3650
+Wire Wire Line
+	5950 3650 5800 3650
+$Comp
+L Device:Crystal Y1
+U 1 1 5EA3D14C
+P 5650 3650
+F 0 "Y1" H 5650 3421 50  0000 C CNN
+F 1 "24M" H 5650 3473 50  0000 C CNN
+F 2 "Crystal:Crystal_HC35-U" H 5650 3650 50  0001 C CNN
+F 3 "~" H 5650 3650 50  0001 C CNN
+	1    5650 3650
+	-1   0    0    1
+$EndComp
 $EndSCHEMATC

Commit message: Add files via upload
Parts:
- removed C32, C33, C35: 0.1uM, Capacitor_SMD:C_0603_1608Metric_Pad1.05x0.95mm_HandSolder, symbol Device:C
- removed J9: Conn_ARM_JTAG_SWD_20, Connector_PinSocket_1.27mm:PinSocket_2x10_P1.27mm_Vertical, symbol Connector:Conn_ARM_JTAG_SWD_20
- removed R22: 510, Resistor_SMD:R_0201_0603Metric, symbol Device:R
- R20, R21: footprint Resistor_SMD:R_0201_0603Metric -> Resistor_SMD:R_0603_1608Metric_Pad1.05x0.95mm_HandSolder
- Y1: footprint Crystal:Crystal_HC35-U -> Crystal:Crystal_HC49-U_Horizontal
Connections:
- wire segments 81 -> 62
Other:
- note removed: "JTAG"

Commit message: Add files via upload
Parts:
- SW3: footprint Button_Switch_SMD:SW_DIP_SPSTx01_Slide_6.7x4.1mm_W6.73mm_P2.54mm_LowProfile_JPin -> Button_Switch_SMD:SW_Push_1P1T_NO_6x6mm_H9.5mm
- Y1: footprint Crystal:Crystal_HC49-U_Horizontal -> Crystal:Crystal_HC49-U_Vertical
Changed lines of the file:
@@
 F 0 "SW3" V 8346 1852 50  0000 R CNN
 F 1 "SW_Push" V 8255 1852 50  0000 R CNN
-F 2 "Button_Switch_SMD:SW_DIP_SPSTx01_Slide_6.7x4.1mm_W6.73mm_P2.54mm_LowProfile_JPin" H 8300 2100 50  0001 C CNN
+F 2 "Button_Switch_SMD:SW_Push_1P1T_NO_6x6mm_H9.5mm" H 8300 2100 50  0001 C CNN
 F 3 "~" H 8300 2100 50  0001 C CNN
 	1    8300 1900
@@
 F 0 "Y1" H 5650 3421 50  0000 C CNN
 F 1 "24M" H 5650 3473 50  0000 C CNN
-F 2 "Crystal:Crystal_HC49-U_Horizontal" H 5650 3650 50  0001 C CNN
+F 2 "Crystal:Crystal_HC49-U_Vertical" H 5650 3650 50  0001 C CNN
 F 3 "~" H 5650 3650 50  0001 C CNN
 	1    5650 3650

Commit message: Add files via upload
Parts:
- added D7: LED, Diode_SMD:D_0805_2012Metric_Pad1.15x1.40mm_HandSolder, symbol Device:LED
- added R7: R, Resistor_SMD:R_0603_1608Metric_Pad1.05x0.95mm_HandSolder, symbol Device:R
Connections:
- net GND: now also R7.2
- net at U10.12 (PA2): now also D7.2 (A)
- net TD11 renamed TDI1
- new net: D7.1 (K), R7.1
Changed lines of the file:
@@
 	4050 2750 4400 2750
 Wire Wire Line
-	4250 5050 4050 5050
-Wire Wire Line
-	4050 5150 4250 5150
-Wire Wire Line
-	4250 5250 4050 5250
-Wire Wire Line
-	4050 5350 4250 5350
-Wire Wire Line
-	4250 5550 4050 5550
-Wire Wire Line
 	9150 1600 9350 1600
 Wire Wire Line
 	9350 1600 9350 1450
-Text Label 4250 5050 0    50   ~ 0
-TRST1
-Text Label 4250 5150 0    50   ~ 0
-SRST1
-Text Label 4250 5450 0    50   ~ 0
-TCK1
 Wire Notes Line
 	6950 3050 11250 3050
@@
 	1    0    0    -1
 $EndComp
-Wire Wire Line
-	4050 5450 4250 5450
-Text Label 4250 5250 0    50   ~ 0
-TD11
-Text Label 4250 5550 0    50   ~ 0
-TD01
-Text Label 4250 5350 0    50   ~ 0
-TMS1
 Wire Wire Line
 	5650 4300 5950 4300
@@
 Wire Notes Line
 	6950 3050 6950 450
+$Comp
+L Device:LED D7
+U 1 1 5ECC6AF2
+P 2250 4250
+F 0 "D7" H 2243 4466 50  0000 C CNN
+F 1 "LED" H 2243 4375 50  0000 C CNN
+F 2 "Diode_SMD:D_0805_2012Metric_Pad1.15x1.40mm_HandSolder" H 2250 4250 50  0001 C CNN
+F 3 "~" H 2250 4250 50  0001 C CNN
+	1    2250 4250
+	1    0    0    -1
+$EndComp
+$Comp
+L Device:R R7
+U 1 1 5ECC7C9B
+P 1750 4250
+F 0 "R7" V 1543 4250 50  0000 C CNN
+F 1 "R" V 1634 4250 50  0000 C CNN
+F 2 "Resistor_SMD:R_0603_1608Metric_Pad1.05x0.95mm_HandSolder" V 1680 4250 50  0001 C CNN
+F 3 "~" H 1750 4250 50  0001 C CNN
+	1    1750 4250
+	0    1    1    0
+$EndComp
+$Comp
+L power:GND #PWR0111
+U 1 1 5ECCAB73
+P 1450 4250
+F 0 "#PWR0111" H 1450 4000 50  0001 C CNN
+F 1 "GND" V 1455 4122 50  0000 R CNN
+F 2 "" H 1450 4250 50  0001 C CNN
+F 3 "" H 1450 4250 50  0001 C CNN
+	1    1450 4250
+	0    1    1    0
+$EndComp
+Wire Wire Line
+	2850 4250 2400 4250
+Wire Wire Line
+	1450 4250 1600 4250
+Wire Wire Line
+	1900 4250 2100 4250
+Text HLabel 4350 5050 2    50   Input ~ 0
+TRST1
+Text HLabel 4350 5150 2    50   Input ~ 0
+SRST1
+Text HLabel 4350 5250 2    50   Input ~ 0
+TDI1
+Text HLabel 4350 5350 2    50   Input ~ 0
+TMS1
+Text HLabel 4350 5450 2    50   Input ~ 0
+TCK1
+Text HLabel 4350 5550 2    50   Input ~ 0
+TD01
+Wire Wire Line
+	4350 5550 4050 5550
+Wire Wire Line
+	4050 5450 4350 5450
+Wire Wire Line
+	4350 5350 4050 5350
+Wire Wire Line
+	4050 5250 4350 5250
+Wire Wire Line
+	4350 5150 4050 5150
+Wire Wire Line
+	4050 5050 4350 5050
 $EndSCHEMATC
