File: proyecto/Alimentacion.sch (KiCad schematic (older format))
At the start: 4 parts

Commit message: Add files via upload
Parts:
- added C?: 0.1uF, symbol Device:C
- added C? (x2): 10uF, symbol Device:C
- added J?: USB_B_Mini, symbol Connector:USB_B_Mini
- added U?: LM1117-5.0, symbol Regulator_Linear:LM1117-5.0
Connections:
- net +5V: now also C?.1, C?.1, U?.2 (VO)
- net GND: now also C?.2, C?.2, C?.2, J?.5 (GND), U?.1 (GND)
- new net: C?.1, J?.1 (VBUS), U?.3 (VI)
Other:
- moved on the sheet: C?, U?

Commit message: Add files via upload
Parts:
- removed C?: 0.1uF, symbol Device:C
- removed C? (x2): 10uF, symbol Device:C
- removed J?: USB_B_Mini, symbol Connector:USB_B_Mini
- removed U?: LM1117-5.0, symbol Regulator_Linear:LM1117-5.0
- added BT?: Battery_Cell_1, symbol Device:Battery_Cell
- added C? (x3): 4.7uF, symbol Device:C
- added C?: 1uF, symbol Device:C
- added C?: 22uF, symbol Device:C
- added D?: D_Schottky, symbol Device:D_Schottky
- added J?: USB_B_Mini, symbol Connector:USB_B_Mini
- added L?: 2.2uH, symbol Device:L
- added Q?: Q_PMOS_DSG, symbol Device:Q_PMOS_DSG
- added R? (x2): 10K, symbol Device:R
- added R?: 2M, symbol Device:R
- added R?: 180K, symbol Device:R
- added U?: MCP73811T-435I-OT, Package_TO_SOT_SMD:SOT-23-5, symbol Battery_Management:MCP73811T-435I-OT
- added U?: TPS61200DRC, Package_SON:Texas_S-PVSON-N10_ThermalVias, symbol Regulator_Switching:TPS61200DRC
Connections:
- net GND: now also BT?.2 (-), C?.2, C?.2, C?.2, C?.2, J?.4 (ID), J?.5 (GND), J?.6 (Shield), R?.2, U?.11 (PAD), U?.2 (VSS), U?.4 (PGND), U?.9 (GND)
- new net: C?.1, D?.2 (A), J?.1 (VBUS), Q?.3 (G), U?.4 (VDD)
- new net: C?.2, R?.2
- new net: R?.1, U?.5 (PROG)
- new net: BT?.1 (+), C?.1, Q?.2 (S), U?.3 (VBAT)
- new net: C?.1, L?.1, Q?.1 (D), R?.1, U?.5 (VIN), U?.6 (EN), U?.8 (PS)
- new net: C?.1, U?.1 (VAUX)
- new net: L?.2, U?.3 (L)
- new net: R?.1, R?.2, U?.7 (UVLO)
- new net +5VD: C?.1, D?.1 (K), R?.1, U?.10 (FB), U?.2 (VOUT)
- new net GNDA: R?.2
- no-connect marks 0 -> 1
Other:
- moved on the sheet: C?, U?

Commit message: Add files via upload
Connections:
- net +5VD is gone; now on net +5V: C?.1, D?.1 (K), R?.1, U?.10 (FB), U?.2 (VOUT)
Other:
- note added: "CARGADOR DE BATERIA"
- note added: "REGULADOR 3.3V"
- moved on the sheet: BT?, C?, D?, J?, L?, Q?, R?, U?

Commit message: Add files via upload
Parts:
- removed C?: 0.1uF, symbol Device:C
- removed C?: 10uF, symbol Device:C
- added C10, C?: 0.1uF, symbol Device:C
- added C11, C? (x2): 10uF, symbol Device:C
- added U?: LM1117-5.0, symbol Regulator_Linear:LM1117-5.0
- gave numbers to parts that had none: 18
Connections:
- net +3V3: now also C10.1, C11.1
- net +5V: now also C?.1, C?.1, U?.2 (VO); no longer C14.1, C8.1, D3.1 (K), R11.1, U4.3 (VI), U5.10 (FB), U5.2 (VOUT)
- net GND: now also C10.2, C11.2, C?.2, C?.2, C?.2, U?.1 (GND)
- net at J5.2 (D-): now also J5.3 (D+)
- new net +5VL: C14.1, C8.1, C?.1, D3.1 (K), R11.1, U4.3 (VI), U5.10 (FB), U5.2 (VOUT), U?.3 (VI)
Other:
- note added: "REGULADOR 5V"
- moved on the sheet: BT1, C12, C13, C14, C7, C8, C9, D3, J5, L4, Q1, R10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

Commit message: Add files via upload
Parts:
- BT1, U4: footprint (none) -> Package_TO_SOT_SMD:SOT-223
- C10, C11, C12, C13, C14, C7, C8, C9: footprint (none) -> Capacitor_SMD:C_0603_1608Metric_Pad1.05x0.95mm_HandSolder
- C37, C38, C39: renamed from C?; footprint (none) -> Capacitor_SMD:C_0603_1608Metric_Pad1.05x0.95mm_HandSolder
- D3: footprint (none) -> Diode_SMD:D_0603_1608Metric_Pad1.05x0.95mm_HandSolder
- J5: footprint (none) -> Connector_USB:USB_Mini-B_AdamTech_MUSB-B5-S-VT-TSMT-1_SMD_Vertical
- L4: footprint (none) -> Inductor_SMD:L_2010_5025Metric
- R10, R11, R8, R9: footprint (none) -> Resistor_SMD:R_0201_0603Metric
- U11: renamed from U?; footprint (none) -> Package_TO_SOT_SMD:SOT-223
Changed lines of the file:
@@
 F 0 "U4" H 2800 1792 50  0000 C CNN
 F 1 "LM1117-3.3" H 2800 1701 50  0000 C CNN
-F 2 "" H 2800 1550 50  0001 C CNN
+F 2 "Package_TO_SOT_SMD:SOT-223" H 2800 1550 50  0001 C CNN
 F 3 "http://www.ti.com/lit/ds/symlink/lm1117.pdf" H 2800 1550 50  0001 C CNN
 	1    2800 1550
@@
 F 0 "C8" H 2265 1846 50  0000 L CNN
 F 1 "10uF" H 2265 1755 50  0000 L CNN
-F 2 "" H 2188 1650 50  0001 C CNN
+F 2 "Capacitor_SMD:C_0603_1608Metric_Pad1.05x0.95mm_HandSolder" H 2188 1650 50  0001 C CNN
 F 3 "~" H 2150 1800 50  0001 C CNN
 	1    2150 1800
@@
 F 0 "C10" H 3515 1846 50  0000 L CNN
 F 1 "0.1uF" H 3515 1755 50  0000 L CNN
-F 2 "" H 3438 1650 50  0001 C CNN
+F 2 "Capacitor_SMD:C_0603_1608Metric_Pad1.05x0.95mm_HandSolder" H 3438 1650 50  0001 C CNN
 F 3 "~" H 3400 1800 50  0001 C CNN
 	1    3400 1800
@@
 F 0 "C11" H 3965 1846 50  0000 L CNN
 F 1 "10uF" H 3965 1755 50  0000 L CNN
-F 2 "" H 3888 1650 50  0001 C CNN
+F 2 "Capacitor_SMD:C_0603_1608Metric_Pad1.05x0.95mm_HandSolder" H 3888 1650 50  0001 C CNN
 F 3 "~" H 3850 1800 50  0001 C CNN
 	1    3850 1800
@@
 REGULADOR 3.3V
 $Comp
-L power:+5VL #PWR?
+L power:+5VL #PWR0143
 U 1 1 5EAA4BA0
 P 2150 1350
-F 0 "#PWR?" H 2150 1200 50  0001 C CNN
+F 0 "#PWR0143" H 2150 1200 50  0001 C CNN
 F 1 "+5VL" H 2165 1523 50  0000 C CNN
 F 2 "" H 2150 1350 50  0001 C CNN
@@
 REGULADOR 5V
 $Comp
-L power:+5V #PWR?
+L power:+5V #PWR0149
 U 1 1 5EAA5774
 P 9500 1300
-F 0 "#PWR?" H 9500 1150 50  0001 C CNN
+F 0 "#PWR0149" H 9500 1150 50  0001 C CNN
 F 1 "+5V" H 9515 1473 50  0000 C CNN
 F 2 "" H 9500 1300 50  0001 C CNN
@@
 $EndComp
 $Comp
-L power:+5VL #PWR?
+L power:+5VL #PWR0162
 U 1 1 5EAA51FD
 P 7800 1300
-F 0 "#PWR?" H 7800 1150 50  0001 C CNN
+F 0 "#PWR0162" H 7800 1150 50  0001 C CNN
 F 1 "+5VL" H 7815 1473 50  0000 C CNN
 F 2 "" H 7800 1300 50  0001 C CNN
@@
 $EndComp
 $Comp
-L Regulator_Linear:LM1117-5.0 U?
+L Regulator_Linear:LM1117-5.0 U11
 U 1 1 5EA96A0A
 P 8450 1500
-F 0 "U?" H 8450 1742 50  0000 C CNN
+F 0 "U11" H 8450 1742 50  0000 C CNN
 F 1 "LM1117-5.0" H 8450 1651 50  0000 C CNN
-F 2 "" H 8450 1500 50  0001 C CNN
+F 2 "Package_TO_SOT_SMD:SOT-223" H 8450 1500 50  0001 C CNN
 F 3 "http://www.ti.com/lit/ds/symlink/lm1117.pdf" H 8450 1500 50  0001 C CNN
 	1    8450 1500
@@
 P 8450 2100
 AR Path="/5EA93EF7" Ref="#PWR?"  Part="1"
-AR Path="/5E9BC166/5EA93EF7" Ref="#PWR?"  Part="1"
+AR Path="/5E9BC166/5EA93EF7" Ref="#PWR0163"  Part="1"
 AR Path="/5EA3D59C/5EA93EF7" Ref="#PWR?"  Part="1"
-F 0 "#PWR?" H 8450 1850 50  0001 C CNN
+F 0 "#PWR0163" H 8450 1850 50  0001 C CNN
 F 1 "GND" H 8455 1927 50  0000 C CNN
 F 2 "" H 8450 2100 50  0001 C CNN
@@
 P 9500 1750
 AR Path="/5EA93EEA" Ref="C?"  Part="1"
-AR Path="/5E9BC166/5EA93EEA" Ref="C?"  Part="1"
+AR Path="/5E9BC166/5EA93EEA" Ref="C39"  Part="1"
 AR Path="/5EA3D59C/5EA93EEA" Ref="C?"  Part="1"
-F 0 "C?" H 9615 1796 50  0000 L CNN
+F 0 "C39" H 9615 1796 50  0000 L CNN
 F 1 "10uF" H 9615 1705 50  0000 L CNN
-F 2 "" H 9538 1600 50  0001 C CNN
+F 2 "Capacitor_SMD:C_0603_1608Metric_Pad1.05x0.95mm_HandSolder" H 9538 1600 50  0001 C CNN
 F 3 "~" H 9500 1750 50  0001 C CNN
 	1    9500 1750
@@
 P 9050 1750
 AR Path="/5EA93EE4" Ref="C?"  Part="1"
-AR Path="/5E9BC166/5EA93EE4" Ref="C?"  Part="1"
+AR Path="/5E9BC166/5EA93EE4" Ref="C38"  Part="1"
 AR Path="/5EA3D59C/5EA93EE4" Ref="C?"  Part="1"
-F 0 "C?" H 9165 1796 50  0000 L CNN
+F 0 "C38" H 9165 1796 50  0000 L CNN
 F 1 "0.1uF" H 9165 1705 50  0000 L CNN
-F 2 "" H 9088 1600 50  0001 C CNN
+F 2 "Capacitor_SMD:C_0603_1608Metric_Pad1.05x0.95mm_HandSolder" H 9088 1600 50  0001 C CNN
 F 3 "~" H 9050 1750 50  0001 C CNN
 	1    9050 1750
@@
 P 7800 1750
 AR Path="/5EA93EDE" Ref="C?"  Part="1"
-AR Path="/5E9BC166/5EA93EDE" Ref="C?"  Part="1"
+AR Path="/5E9BC166/5EA93EDE" Ref="C37"  Part="1"
 AR Path="/5EA3D59C/5EA93EDE" Ref="C?"  Part="1"
-F 0 "C?" H 7915 1796 50  0000 L CNN
+F 0 "C37" H 7915 1796 50  0000 L CNN
 F 1 "10uF" H 7915 1705 50  0000 L CNN
-F 2 "" H 7838 1600 50  0001 C CNN
+F 2 "Capacitor_SMD:C_0603_1608Metric_Pad1.05x0.95mm_HandSolder" H 7838 1600 50  0001 C CNN
 F 3 "~" H 7800 1750 50  0001 C CNN
 	1    7800 1750
@@
 	8650 5900 7950 5900
 $Comp
-L power:+5VL #PWR?
+L power:+5VL #PWR0164
 U 1 1 5EAA434B
 P 9800 4950
-F 0 "#PWR?" H 9800 4800 50  0001 C CNN
+F 0 "#PWR0164" H 9800 4800 50  0001 C CNN
 F 1 "+5VL" H 9815 5123 50  0000 C CNN
 F 2 "" H 9800 4950 50  0001 C CNN
@@
 F 0 "D3" H 7350 3784 50  0000 C CNN
 F 1 "D_Schottky" H 7350 3875 50  0000 C CNN
-F 2 "" H 7350 4000 50  0001 C CNN
+F 2 "Diode_SMD:D_0603_1608Metric_Pad1.05x0.95mm_HandSolder" H 7350 4000 50  0001 C CNN
 F 3 "~" H 7350 4000 50  0001 C CNN
 	1    7350 4000
@@
 F 0 "R11" H 8870 4446 50  0000 L CNN
 F 1 "10K" H 8870 4355 50  0000 L CNN
-F 2 "" V 8730 4400 50  0001 C CNN
+F 2 "Resistor_SMD:R_0201_0603Metric" V 8730 4400 50  0001 C CNN
 F 3 "~" H 8800 4400 50  0001 C CNN
 	1    8800 4400
@@
 F 0 "C14" H 9315 5546 50  0000 L CNN
 F 1 "22uF" H 9315 5455 50  0000 L CNN
-F 2 "" H 9238 5350 50  0001 C CNN
+F 2 "Capacitor_SMD:C_0603_1608Metric_Pad1.05x0.95mm_HandSolder" H 9238 5350 50  0001 C CNN
 F 3 "~" H 9200 5500 50  0001 C CNN
 	1    9200 5500
@@
 F 0 "C13" H 8765 5546 50  0000 L CNN
 F 1 "1uF" H 8765 5455 50  0000 L CNN
-F 2 "" H 8688 5350 50  0001 C CNN
+F 2 "Capacitor_SMD:C_0603_1608Metric_Pad1.05x0.95mm_HandSolder" H 8688 5350 50  0001 C CNN
 F 3 "~" H 8650 5500 50  0001 C CNN
 	1    8650 5500
@@
 F 0 "L4" V 8050 4650 50  0000 C CNN
 F 1 "2.2uH" V 7950 4650 50  0000 C CNN
-F 2 "" H 7850 4650 50  0001 C CNN
+F 2 "Inductor_SMD:L_2010_5025Metric" H 7850 4650 50  0001 C CNN
 F 3 "~" H 7850 4650 50  0001 C CNN
 	1    7850 4650
@@
 F 0 "C12" H 6765 5196 50  0000 L CNN
 F 1 "4.7uF" H 6765 5105 50  0000 L CNN
-F 2 "" H 6688 5000 50  0001 C CNN
+F 2 "Capacitor_SMD:C_0603_1608Metric_Pad1.05x0.95mm_HandSolder" H 6688 5000 50  0001 C CNN
 F 3 "~" H 6650 5150 50  0001 C CNN
 	1    6650 5150
@@
 F 0 "R10" H 7070 5596 50  0000 L CNN
 F 1 "180K" H 7070 5505 50  0000 L CNN
-F 2 "" V 6930 5550 50  0001 C CNN
+F 2 "Resistor_SMD:R_0201_0603Metric" V 6930 5550 50  0001 C CNN
 F 3 "~" H 7000 5550 50  0001 C CNN
 	1    7000 5550
@@
 F 0 "R9" H 7070 5096 50  0000 L CNN
 F 1 "2M" H 7070 5005 50  0000 L CNN
-F 2 "" V 6930 5050 50  0001 C CNN
+F 2 "Resistor_SMD:R_0201_0603Metric" V 6930 5050 50  0001 C CNN
 F 3 "~" H 7000 5050 50  0001 C CNN
 	1    7000 5050
@@
 F 0 "BT1" H 5750 4900 50  0000 L CNN
 F 1 "Battery_Cell_1" H 5750 4800 50  0000 L CNN
-F 2 "" V 5700 5010 50  0001 C CNN
+F 2 "Package_TO_SOT_SMD:SOT-223" V 5700 5010 50  0001 C CNN
 F 3 "~" V 5700 5010 50  0001 C CNN
 	1    5700 4950
@@
 F 0 "C9" H 5365 4946 50  0000 L CNN
 F 1 "4.7uF" H 5365 4855 50  0000 L CNN
-F 2 "" H 5288 4750 50  0001 C CNN
+F 2 "Capacitor_SMD:C_0603_1608Metric_Pad1.05x0.95mm_HandSolder" H 5288 4750 50  0001 C CNN
 F 3 "~" H 5250 4900 50  0001 C CNN
 	1    5250 4900
@@
 F 0 "R8" V 3543 4850 50  0000 C CNN
 F 1 "10K" V 3634 4850 50  0000 C CNN
-F 2 "" V 3680 4850 50  0001 C CNN
+F 2 "Resistor_SMD:R_0201_0603Metric" V 3680 4850 50  0001 C CNN
 F 3 "~" H 3750 4850 50  0001 C CNN
 	1    3750 4850
@@
 F 0 "C7" H 3415 4646 50  0000 L CNN
 F 1 "4.7uF" H 3415 4555 50  0000 L CNN
-F 2 "" H 3338 4450 50  0001 C CNN
+F 2 "Capacitor_SMD:C_0603_1608Metric_Pad1.05x0.95mm_HandSolder" H 3338 4450 50  0001 C CNN
 F 3 "~" H 3300 4600 50  0001 C CNN
 	1    3300 4600
@@
 F 0 "J5" H 2557 4967 50  0000 C CNN
 F 1 "USB_B_Mini" H 2557 4876 50  0000 C CNN
-F 2 "" H 2650 4450 50  0001 C CNN
+F 2 "Connector_USB:USB_Mini-B_AdamTech_MUSB-B5-S-VT-TSMT-1_SMD_Vertical" H 2650 4450 50  0001 C CNN
 F 3 "~" H 2650 4450 50  0001 C CNN
 	1    2500 4500

Commit message: Add files via upload
Parts:
- added C44: 0.1uF, Capacitor_SMD:C_0603_1608Metric_Pad1.05x0.95mm_HandSolder, symbol Device:C
- Q1: footprint (none) -> Diode_SMD:D_0805_2012Metric
Connections:
- net GND: now also C44.2; no longer J5.6 (Shield)
- new net: C44.1, J5.6 (Shield)
Changed lines of the file:
@@
 F 0 "Q1" V 6499 4550 50  0000 C CNN
 F 1 "Q_PMOS_DSG" V 6590 4550 50  0000 C CNN
-F 2 "" H 6450 4650 50  0001 C CNN
+F 2 "Diode_SMD:D_0805_2012Metric" H 6450 4650 50  0001 C CNN
 F 3 "~" H 6250 4550 50  0001 C CNN
 	1    6250 4550
@@
 $EndComp
 Wire Wire Line
-	2400 4950 2500 4950
-Wire Wire Line
-	2400 4900 2400 4950
-Wire Wire Line
 	2500 4950 2500 4900
 Connection ~ 2500 4950
@@
 Wire Wire Line
 	2800 4600 2800 4500
+$Comp
+L Device:C C44
+U 1 1 5EB27D1F
+P 2250 5200
+F 0 "C44" H 2100 5300 50  0000 L CNN
+F 1 "0.1uF" H 2000 5100 50  0000 L CNN
+F 2 "Capacitor_SMD:C_0603_1608Metric_Pad1.05x0.95mm_HandSolder" H 2288 5050 50  0001 C CNN
+F 3 "~" H 2250 5200 50  0001 C CNN
+	1    2250 5200
+	1    0    0    -1
+$EndComp
+$Comp
+L power:GND #PWR0171
+U 1 1 5EB2C13C
+P 2250 5500
+F 0 "#PWR0171" H 2250 5250 50  0001 C CNN
+F 1 "GND" H 2255 5327 50  0000 C CNN
+F 2 "" H 2250 5500 50  0001 C CNN
+F 3 "" H 2250 5500 50  0001 C CNN
+	1    2250 5500
+	1    0    0    -1
+$EndComp
+Wire Wire Line
+	2250 5500 2250 5350
+Wire Wire Line
+	2250 5050 2250 5000
+Wire Wire Line
+	2250 5000 2400 5000
+Wire Wire Line
+	2400 5000 2400 4900
 $EndSCHEMATC

Commit message: Add files via upload
Parts:
- BT1: footprint Package_TO_SOT_SMD:SOT-223 -> (none)
Changed lines of the file:
@@
 F 0 "BT1" H 5750 4900 50  0000 L CNN
 F 1 "Battery_Cell_1" H 5750 4800 50  0000 L CNN
-F 2 "Package_TO_SOT_SMD:SOT-223" V 5700 5010 50  0001 C CNN
+F 2 "" V 5700 5010 50  0001 C CNN
 F 3 "~" V 5700 5010 50  0001 C CNN
 	1    5700 4950

Commit message: Add files via upload
Parts:
- removed D3: D_Schottky, Diode_SMD:D_0603_1608Metric_Pad1.05x0.95mm_HandSolder, symbol Device:D_Schottky
- added D3: 1N5817, Diode_THT:D_DO-41_SOD81_P10.16mm_Horizontal, symbol Diode:1N5817
- BT1: footprint (none) -> Battery:Battery_Panasonic_CR3032-VCN_Vertical_CircularHoles
Connections:
- net GNDA is gone; now on net GND: R11.2
- net +5VL: now also D3.1 (K)
- net at C7.1, J5.1 (VBUS), Q1.3 (G)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: now also D3.2 (A)
- net +3V3 renamed +3V8
Changed lines of the file:
@@
 Wire Wire Line
 	3850 1950 3850 2150
-$Comp
-L power:+3.3V #PWR0121
-U 1 1 5E9C6FA9
-P 3850 1350
-AR Path="/5E9BC166/5E9C6FA9" Ref="#PWR0121"  Part="1"
-AR Path="/5EA3D59C/5E9C6FA9" Ref="#PWR?"  Part="1"
-F 0 "#PWR0121" H 3850 1200 50  0001 C CNN
-F 1 "+3.3V" H 3865 1523 50  0000 C CNN
-F 2 "" H 3850 1350 50  0001 C CNN
-F 3 "" H 3850 1350 50  0001 C CNN
-	1    3850 1350
-	1    0    0    -1
-$EndComp
 Wire Wire Line
 	3850 1350 3850 1550
@@
 Wire Wire Line
 	8800 4550 8800 4650
-$Comp
-L power:GNDA #PWR?
-U 1 1 5EA974C2
-P 8800 4650
-AR Path="/5EA3D59C/5EA974C2" Ref="#PWR?"  Part="1"
-AR Path="/5E9BC166/5EA974C2" Ref="#PWR0123"  Part="1"
-F 0 "#PWR0123" H 8800 4400 50  0001 C CNN
-F 1 "GNDA" H 8805 4477 50  0000 C CNN
-F 2 "" H 8800 4650 50  0001 C CNN
-F 3 "" H 8800 4650 50  0001 C CNN
-	1    8800 4650
-	1    0    0    -1
-$EndComp
 Wire Wire Line
 	8800 4000 9200 4000
 Connection ~ 8800 4000
 Wire Wire Line
-	7500 4000 8800 4000
+	7550 4000 8800 4000
 Wire Wire Line
 	8800 4250 8800 4000
@@
 	4550 4000 4550 4300
 Wire Wire Line
-	7200 4000 6250 4000
+	7250 4000 6250 4000
 Wire Wire Line
 	9200 4000 9200 5150
@@
 Wire Wire Line
 	6450 4650 6650 4650
-$Comp
-L Device:D_Schottky D?
-U 1 1 5EA97495
-P 7350 4000
-AR Path="/5EA3D59C/5EA97495" Ref="D?"  Part="1"
-AR Path="/5E9BC166/5EA97495" Ref="D3"  Part="1"
-F 0 "D3" H 7350 3784 50  0000 C CNN
-F 1 "D_Schottky" H 7350 3875 50  0000 C CNN
-F 2 "Diode_SMD:D_0603_1608Metric_Pad1.05x0.95mm_HandSolder" H 7350 4000 50  0001 C CNN
-F 3 "~" H 7350 4000 50  0001 C CNN
-	1    7350 4000
-	-1   0    0    1
-$EndComp
 $Comp
 L Device:R R?
@@
 F 0 "BT1" H 5750 4900 50  0000 L CNN
 F 1 "Battery_Cell_1" H 5750 4800 50  0000 L CNN
-F 2 "" V 5700 5010 50  0001 C CNN
+F 2 "Battery:Battery_Panasonic_CR3032-VCN_Vertical_CircularHoles" V 5700 5010 50  0001 C CNN
 F 3 "~" V 5700 5010 50  0001 C CNN
 	1    5700 4950
@@
 Wire Wire Line
 	2400 5000 2400 4900
+$Comp
+L Diode:1N5817 D3
+U 1 1 5EB23B85
+P 7400 4000
+F 0 "D3" H 7400 3784 50  0000 C CNN
+F 1 "1N5817" H 7400 3875 50  0000 C CNN
+F 2 "Diode_THT:D_DO-41_SOD81_P10.16mm_Horizontal" H 7400 3825 50  0001 C CNN
+F 3 "http://www.vishay.com/docs/88525/1n5817.pdf" H 7400 4000 50  0001 C CNN
+	1    7400 4000
+	-1   0    0    1
+$EndComp
+$Comp
+L power:+3V8 #PWR0121
+U 1 1 5EB680DD
+P 3850 1350
+F 0 "#PWR0121" H 3850 1200 50  0001 C CNN
+F 1 "+3V8" H 3865 1523 50  0000 C CNN
+F 2 "" H 3850 1350 50  0001 C CNN
+F 3 "" H 3850 1350 50  0001 C CNN
+	1    3850 1350
+	1    0    0    -1
+$EndComp
+$Comp
+L power:GND #PWR?
+U 1 1 5EB6E88A
+P 8800 4650
+F 0 "#PWR?" H 8800 4400 50  0001 C CNN
+F 1 "GND" H 8805 4477 50  0000 C CNN
+F 2 "" H 8800 4650 50  0001 C CNN
+F 3 "" H 8800 4650 50  0001 C CNN
+	1    8800 4650
+	1    0    0    -1
+$EndComp
 $EndSCHEMATC
