File: proyecto/Alimentacion.sch (KiCad schematic (older format))
At the start: 25 parts, among them J5 USB_B_Mini, Q1 Q_PMOS_DSG, U11 LM1117-5.0, U3 MCP73811T-435I-OT, U4 LM1117-3.3, U5 TPS61200DRC

Commit message: Add files via upload
Parts:
- Q1: footprint Diode_SMD:D_0805_2012Metric -> Package_TO_SOT_SMD:SOT-23
Changed lines of the file:
@@
 F 0 "Q1" V 6499 4550 50  0000 C CNN
 F 1 "Q_PMOS_DSG" V 6590 4550 50  0000 C CNN
-F 2 "Diode_SMD:D_0805_2012Metric" H 6450 4650 50  0001 C CNN
+F 2 "Package_TO_SOT_SMD:SOT-23" H 6450 4650 50  0001 C CNN
 F 3 "~" H 6250 4550 50  0001 C CNN
 	1    6250 4550
@@
 $EndComp
 $Comp
-L power:GND #PWR?
+L power:GND #PWR0123
 U 1 1 5EB6E88A
 P 8800 4650
-F 0 "#PWR?" H 8800 4400 50  0001 C CNN
+F 0 "#PWR0123" H 8800 4400 50  0001 C CNN
 F 1 "GND" H 8805 4477 50  0000 C CNN
 F 2 "" H 8800 4650 50  0001 C CNN

Commit message: Add files via upload
Parts:
- removed BT1: Battery_Cell_1, Battery:Battery_Panasonic_CR3032-VCN_Vertical_CircularHoles, symbol Device:Battery_Cell
- added J9: Conn_01x02, Connector_PinHeader_1.00mm:PinHeader_1x02_P1.00mm_Horizontal, symbol Connector_Generic:Conn_01x02
- L4: footprint Inductor_SMD:L_2010_5025Metric -> Inductor_SMD:L_2010_5025Metric_Pad1.52x2.65mm_HandSolder
- R10, R11, R8, R9: footprint Resistor_SMD:R_0201_0603Metric -> Resistor_SMD:R_0603_1608Metric_Pad1.05x0.95mm_HandSolder
Connections:
- net GND: now also J9.2 (Pin_2)
- net at C9.1, Q1.2 (S), U3.3 (VBAT): now also J9.1 (Pin_1)
Changed lines of the file:
@@
 F 0 "R11" H 8870 4446 50  0000 L CNN
 F 1 "10K" H 8870 4355 50  0000 L CNN
-F 2 "Resistor_SMD:R_0201_0603Metric" V 8730 4400 50  0001 C CNN
+F 2 "Resistor_SMD:R_0603_1608Metric_Pad1.05x0.95mm_HandSolder" V 8730 4400 50  0001 C CNN
 F 3 "~" H 8800 4400 50  0001 C CNN
 	1    8800 4400
@@
 F 0 "L4" V 8050 4650 50  0000 C CNN
 F 1 "2.2uH" V 7950 4650 50  0000 C CNN
-F 2 "Inductor_SMD:L_2010_5025Metric" H 7850 4650 50  0001 C CNN
+F 2 "Inductor_SMD:L_2010_5025Metric_Pad1.52x2.65mm_HandSolder" H 7850 4650 50  0001 C CNN
 F 3 "~" H 7850 4650 50  0001 C CNN
 	1    7850 4650
@@
 F 0 "R10" H 7070 5596 50  0000 L CNN
 F 1 "180K" H 7070 5505 50  0000 L CNN
-F 2 "Resistor_SMD:R_0201_0603Metric" V 6930 5550 50  0001 C CNN
+F 2 "Resistor_SMD:R_0603_1608Metric_Pad1.05x0.95mm_HandSolder" V 6930 5550 50  0001 C CNN
 F 3 "~" H 7000 5550 50  0001 C CNN
 	1    7000 5550
@@
 F 0 "R9" H 7070 5096 50  0000 L CNN
 F 1 "2M" H 7070 5005 50  0000 L CNN
-F 2 "Resistor_SMD:R_0201_0603Metric" V 6930 5050 50  0001 C CNN
+F 2 "Resistor_SMD:R_0603_1608Metric_Pad1.05x0.95mm_HandSolder" V 6930 5050 50  0001 C CNN
 F 3 "~" H 7000 5050 50  0001 C CNN
 	1    7000 5050
@@
 	0    1    1    0
 $EndComp
-NoConn ~ 4550 4900
 Wire Wire Line
 	5250 5200 4550 5200
@@
 Wire Wire Line
 	4550 5200 4550 5300
-Connection ~ 4550 5200
 Wire Wire Line
 	5700 5200 5250 5200
-Wire Wire Line
-	5700 5050 5700 5200
 Wire Wire Line
 	5250 4650 5700 4650
@@
 Wire Wire Line
 	5250 4750 5250 4650
-Wire Wire Line
-	5700 4650 5700 4750
 Wire Wire Line
 	4950 4650 5250 4650
@@
 	4550 4450 4550 4300
 $Comp
-L Device:Battery_Cell BT?
-U 1 1 5EA9743D
-P 5700 4950
-AR Path="/5EA3D59C/5EA9743D" Ref="BT?"  Part="1"
-AR Path="/5E9BC166/5EA9743D" Ref="BT1"  Part="1"
-F 0 "BT1" H 5750 4900 50  0000 L CNN
-F 1 "Battery_Cell_1" H 5750 4800 50  0000 L CNN
-F 2 "Battery:Battery_Panasonic_CR3032-VCN_Vertical_CircularHoles" V 5700 5010 50  0001 C CNN
-F 3 "~" V 5700 5010 50  0001 C CNN
-	1    5700 4950
-	1    0    0    -1
-$EndComp
-$Comp
 L Device:C C?
 U 1 1 5EA97437
@@
 $EndComp
 Wire Wire Line
-	4550 5050 4550 5200
-Wire Wire Line
 	3300 4300 2800 4300
 Connection ~ 3300 4300
@@
 F 0 "R8" V 3543 4850 50  0000 C CNN
 F 1 "10K" V 3634 4850 50  0000 C CNN
-F 2 "Resistor_SMD:R_0201_0603Metric" V 3680 4850 50  0001 C CNN
+F 2 "Resistor_SMD:R_0603_1608Metric_Pad1.05x0.95mm_HandSolder" V 3680 4850 50  0001 C CNN
 F 3 "~" H 3750 4850 50  0001 C CNN
 	1    3750 4850
@@
 	1    0    0    -1
 $EndComp
+NoConn ~ 4550 4900
+Wire Wire Line
+	4550 5050 4550 5200
+Connection ~ 4550 5200
+$Comp
+L Connector_Generic:Conn_01x02 J9
+U 1 1 5ECEF3A0
+P 5900 5100
+F 0 "J9" H 5980 5092 50  0000 L CNN
+F 1 "Conn_01x02" H 5980 5001 50  0000 L CNN
+F 2 "Connector_PinHeader_1.00mm:PinHeader_1x02_P1.00mm_Horizontal" H 5900 5100 50  0001 C CNN
+F 3 "~" H 5900 5100 50  0001 C CNN
+	1    5900 5100
+	1    0    0    -1
+$EndComp
+Wire Wire Line
+	5700 4650 5700 5100
 $EndSCHEMATC

Commit message: Add files via upload
Parts:
- D3: footprint Diode_THT:D_DO-41_SOD81_P10.16mm_Horizontal -> Diode_THT:D_DO-41_SOD81_P5.08mm_Vertical_AnodeUp
Changed lines of the file:
@@
 F 0 "D3" H 7400 3784 50  0000 C CNN
 F 1 "1N5817" H 7400 3875 50  0000 C CNN
-F 2 "Diode_THT:D_DO-41_SOD81_P10.16mm_Horizontal" H 7400 3825 50  0001 C CNN
+F 2 "Diode_THT:D_DO-41_SOD81_P5.08mm_Vertical_AnodeUp" H 7400 3825 50  0001 C CNN
 F 3 "http://www.vishay.com/docs/88525/1n5817.pdf" H 7400 4000 50  0001 C CNN
 	1    7400 4000

Commit message: Add files via upload
Parts:
- added FL1, FL2, FL3, FL4: BLM18SG121TN1D, Resistor_SMD:R_0603_1608Metric_Pad1.05x0.95mm_HandSolder, symbol BLM18SG121TN1D:BLM18SG121TN1D
- added H1, H2, H3, H4: MountingHole_Pad, MountingHole:MountingHole_2.5mm_Pad, symbol Mechanical:MountingHole_Pad
Connections:
- net GND: now also FL1.2, FL2.2, FL3.2, FL4.2
- new net: FL1.1, H1.1
- new net: FL2.1, H2.1
- new net: FL3.1, H3.1
- new net: FL4.1, H4.1
Other:
- moved on the sheet: C10, C11, C12, C13, C14, C37, C38, C39, C44, C7, C8, C9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
