File: proyecto/Alimentacion_camara.sch (KiCad schematic (older format))
At the start: 4 parts

Commit message: Add files via upload
Other:
- moved on the sheet: C?, U?
Changed lines of the file:
@@
 $Descr A4 11693 8268
 encoding utf-8
-Sheet 5 7
+Sheet 7 7
 Title ""
 Date ""
@@
 L Regulator_Linear:LM1117-3.3 U?
 U 1 1 5E9D90F6
-P 4700 3450
+P 4250 3350
 AR Path="/5E9D90F6" Ref="U?"  Part="1"
 AR Path="/5E9BC166/5E9D90F6" Ref="U?"  Part="1"
 AR Path="/5EA3D59C/5E9D90F6" Ref="U?"  Part="1"
-F 0 "U?" H 4700 3692 50  0000 C CNN
-F 1 "LM1117-3.3" H 4700 3601 50  0000 C CNN
-F 2 "" H 4700 3450 50  0001 C CNN
-F 3 "http://www.ti.com/lit/ds/symlink/lm1117.pdf" H 4700 3450 50  0001 C CNN
-	1    4700 3450
+F 0 "U?" H 4250 3592 50  0000 C CNN
+F 1 "LM1117-3.3" H 4250 3501 50  0000 C CNN
+F 2 "" H 4250 3350 50  0001 C CNN
+F 3 "http://www.ti.com/lit/ds/symlink/lm1117.pdf" H 4250 3350 50  0001 C CNN
+	1    4250 3350
 	1    0    0    -1
 $EndComp
@@
 L Device:C C?
 U 1 1 5E9D90FC
-P 4050 3700
+P 3600 3600
 AR Path="/5E9D90FC" Ref="C?"  Part="1"
 AR Path="/5E9BC166/5E9D90FC" Ref="C?"  Part="1"
 AR Path="/5EA3D59C/5E9D90FC" Ref="C?"  Part="1"
-F 0 "C?" H 4165 3746 50  0000 L CNN
-F 1 "10uF" H 4165 3655 50  0000 L CNN
-F 2 "" H 4088 3550 50  0001 C CNN
-F 3 "~" H 4050 3700 50  0001 C CNN
-	1    4050 3700
+F 0 "C?" H 3715 3646 50  0000 L CNN
+F 1 "10uF" H 3715 3555 50  0000 L CNN
+F 2 "" H 3638 3450 50  0001 C CNN
+F 3 "~" H 3600 3600 50  0001 C CNN
+	1    3600 3600
 	1    0    0    -1
 $EndComp
@@
 L Device:C C?
 U 1 1 5E9D9102
-P 5300 3700
+P 4850 3600
 AR Path="/5E9D9102" Ref="C?"  Part="1"
 AR Path="/5E9BC166/5E9D9102" Ref="C?"  Part="1"
 AR Path="/5EA3D59C/5E9D9102" Ref="C?"  Part="1"
-F 0 "C?" H 5415 3746 50  0000 L CNN
-F 1 "0.1uF" H 5415 3655 50  0000 L CNN
-F 2 "" H 5338 3550 50  0001 C CNN
-F 3 "~" H 5300 3700 50  0001 C CNN
-	1    5300 3700
+F 0 "C?" H 4965 3646 50  0000 L CNN
+F 1 "0.1uF" H 4965 3555 50  0000 L CNN
+F 2 "" H 4888 3450 50  0001 C CNN
+F 3 "~" H 4850 3600 50  0001 C CNN
+	1    4850 3600
 	1    0    0    -1
 $EndComp
@@
 L Device:C C?
 U 1 1 5E9D9108
-P 5750 3700
+P 5300 3600
 AR Path="/5E9D9108" Ref="C?"  Part="1"
 AR Path="/5E9BC166/5E9D9108" Ref="C?"  Part="1"
 AR Path="/5EA3D59C/5E9D9108" Ref="C?"  Part="1"
-F 0 "C?" H 5865 3746 50  0000 L CNN
-F 1 "10uF" H 5865 3655 50  0000 L CNN
-F 2 "" H 5788 3550 50  0001 C CNN
-F 3 "~" H 5750 3700 50  0001 C CNN
-	1    5750 3700
+F 0 "C?" H 5415 3646 50  0000 L CNN
+F 1 "10uF" H 5415 3555 50  0000 L CNN
+F 2 "" H 5338 3450 50  0001 C CNN
+F 3 "~" H 5300 3600 50  0001 C CNN
+	1    5300 3600
 	1    0    0    -1
 $EndComp
 Wire Wire Line
-	4400 3450 4050 3450
+	3950 3350 3600 3350
 Wire Wire Line
-	4050 3550 4050 3450
+	3600 3450 3600 3350
 Wire Wire Line
-	5300 3550 5300 3450
-Connection ~ 5300 3450
+	4850 3450 4850 3350
+Connection ~ 4850 3350
 Wire Wire Line
-	5300 3450 5000 3450
+	4850 3350 4550 3350
 Wire Wire Line
-	5750 3550 5750 3450
+	5300 3450 5300 3350
 Wire Wire Line
-	5750 3450 5300 3450
+	5300 3350 4850 3350
 $Comp
 L power:GND #PWR?
 U 1 1 5E9D911B
-P 4700 4050
+P 4250 3950
 AR Path="/5E9D911B" Ref="#PWR?"  Part="1"
 AR Path="/5E9BC166/5E9D911B" Ref="#PWR?"  Part="1"
 AR Path="/5EA3D59C/5E9D911B" Ref="#PWR?"  Part="1"
-F 0 "#PWR?" H 4700 3800 50  0001 C CNN
-F 1 "GND" H 4705 3877 50  0000 C CNN
-F 2 "" H 4700 4050 50  0001 C CNN
-F 3 "" H 4700 4050 50  0001 C CNN
-	1    4700 4050
+F 0 "#PWR?" H 4250 3700 50  0001 C CNN
+F 1 "GND" H 4255 3777 50  0000 C CNN
+F 2 "" H 4250 3950 50  0001 C CNN
+F 3 "" H 4250 3950 50  0001 C CNN
+	1    4250 3950
 	1    0    0    -1
 $EndComp
 Wire Wire Line
-	5750 4050 5300 4050
-Connection ~ 4700 4050
+	5300 3950 4850 3950
+Connection ~ 4250 3950
 Wire Wire Line
-	4700 3750 4700 4050
+	4250 3650 4250 3950
 Wire Wire Line
-	5300 3850 5300 4050
-Connection ~ 5300 4050
+	4850 3750 4850 3950
+Connection ~ 4850 3950
 Wire Wire Line
-	5300 4050 4700 4050
+	4850 3950 4250 3950
 Wire Wire Line
-	4050 3850 4050 4050
+	3600 3750 3600 3950
 Wire Wire Line
-	4050 4050 4700 4050
+	3600 3950 4250 3950
 Wire Wire Line
-	5750 3850 5750 4050
+	5300 3750 5300 3950
 $Comp
 L power:+3.3V #PWR?
 U 1 1 5E9C6FA9
-P 5750 3250
+P 5300 3150
 AR Path="/5E9BC166/5E9C6FA9" Ref="#PWR?"  Part="1"
 AR Path="/5EA3D59C/5E9C6FA9" Ref="#PWR?"  Part="1"
-F 0 "#PWR?" H 5750 3100 50  0001 C CNN
-F 1 "+3.3V" H 5765 3423 50  0000 C CNN
-F 2 "" H 5750 3250 50  0001 C CNN
-F 3 "" H 5750 3250 50  0001 C CNN
-	1    5750 3250
+F 0 "#PWR?" H 5300 3000 50  0001 C CNN
+F 1 "+3.3V" H 5315 3323 50  0000 C CNN
+F 2 "" H 5300 3150 50  0001 C CNN
+F 3 "" H 5300 3150 50  0001 C CNN
+	1    5300 3150
 	1    0    0    -1
 $EndComp
@@
 L power:+5V #PWR?
 U 1 1 5E9C79B9
-P 4050 3250
+P 3600 3150
 AR Path="/5E9BC166/5E9C79B9" Ref="#PWR?"  Part="1"
 AR Path="/5EA3D59C/5E9C79B9" Ref="#PWR?"  Part="1"
-F 0 "#PWR?" H 4050 3100 50  0001 C CNN
-F 1 "+5V" H 4065 3423 50  0000 C CNN
-F 2 "" H 4050 3250 50  0001 C CNN
-F 3 "" H 4050 3250 50  0001 C CNN
-	1    4050 3250
+F 0 "#PWR?" H 3600 3000 50  0001 C CNN
+F 1 "+5V" H 3615 3323 50  0000 C CNN
+F 2 "" H 3600 3150 50  0001 C CNN
+F 3 "" H 3600 3150 50  0001 C CNN
+	1    3600 3150
 	1    0    0    -1
 $EndComp
 Wire Wire Line
-	5750 3250 5750 3450
-Connection ~ 5750 3450
+	5300 3150 5300 3350
+Connection ~ 5300 3350
 Wire Wire Line
-	4050 3450 4050 3250
-Connection ~ 4050 3450
+	3600 3350 3600 3150
+Connection ~ 3600 3350
 $EndSCHEMATC

Commit message: Add files via upload
Parts:
- added C?: 0.1uF, symbol Device:C
- added C? (x2): 10uF, symbol Device:C
- added J?: USB_B_Mini, symbol Connector:USB_B_Mini
- added U?: LM1117-5.0, symbol Regulator_Linear:LM1117-5.0
Connections:
- net +5V renamed +5VD
- net +5VD: now also C?.1, C?.1, U?.2 (VO)
- new net: C?.1, J?.1 (VBUS), U?.3 (VI)
- new net GNDA: C?.2, C?.2, C?.2, J?.5 (GND), U?.1 (GND)
Other:
- moved on the sheet: C?, U?

Commit message: Add files via upload
Parts:
- removed C?: 0.1uF, symbol Device:C
- removed C? (x2): 10uF, symbol Device:C
- removed U?: LM1117-5.0, symbol Regulator_Linear:LM1117-5.0
- added BT?: Battery_Cell_2, symbol Device:Battery_Cell
- added C? (x3): 4.7uF, symbol Device:C
- added C?: 1uF, symbol Device:C
- added C?: 22uF, symbol Device:C
- added D?: D_Schottky, symbol Device:D_Schottky
- added L?: 2.2uH, symbol Device:L
- added Q?: Q_PMOS_DSG, symbol Device:Q_PMOS_DSG
- added R? (x2): 10K, symbol Device:R
- added R?: 2M, symbol Device:R
- added R?: 180K, symbol Device:R
- added U?: MCP73811T-435I-OT, Package_TO_SOT_SMD:SOT-23-5, symbol Battery_Management:MCP73811T-435I-OT
- added U?: TPS61200DRC, Package_SON:Texas_S-PVSON-N10_ThermalVias, symbol Regulator_Switching:TPS61200DRC
Connections:
- net +5VD: now also C?.1, D?.1 (K), R?.1, U?.10 (FB), U?.2 (VOUT)
- net GNDA: now also J?.4 (ID), J?.6 (Shield), BT?.2 (-), C?.2, C?.2, C?.2, C?.2, R?.2, R?.2, U?.11 (PAD), U?.2 (VSS), U?.4 (PGND), U?.9 (GND)
- net at J?.1 (VBUS): now also C?.1, D?.2 (A), Q?.3 (G), U?.4 (VDD)
- new net: C?.2, R?.2
- new net: R?.1, U?.5 (PROG)
- new net: BT?.1 (+), C?.1, Q?.2 (S), U?.3 (VBAT)
- new net: C?.1, L?.1, Q?.1 (D), R?.1, U?.5 (VIN), U?.6 (EN), U?.8 (PS)
- new net: C?.1, U?.1 (VAUX)
- new net: L?.2, U?.3 (L)
- new net: R?.1, R?.2, U?.7 (UVLO)
- no-connect marks 0 -> 1
Other:
- moved on the sheet: C?, J?, U?

Commit message: Add files via upload
Other:
- note added: "CARGADOR DE BATERIA"
- note added: "REGULADOR 3.3V"
- moved on the sheet: C?, U?
Changed lines of the file:
@@
 Comment4 ""
 $EndDescr
-$Comp
-L Regulator_Linear:LM1117-3.3 U?
-U 1 1 5E9D90F6
-P 3600 4700
-AR Path="/5E9D90F6" Ref="U?"  Part="1"
-AR Path="/5E9BC166/5E9D90F6" Ref="U?"  Part="1"
-AR Path="/5EA3D59C/5E9D90F6" Ref="U?"  Part="1"
-F 0 "U?" H 3600 4942 50  0000 C CNN
-F 1 "LM1117-3.3" H 3600 4851 50  0000 C CNN
-F 2 "" H 3600 4700 50  0001 C CNN
-F 3 "http://www.ti.com/lit/ds/symlink/lm1117.pdf" H 3600 4700 50  0001 C CNN
-	1    3600 4700
-	1    0    0    -1
-$EndComp
-$Comp
-L Device:C C?
-U 1 1 5E9D90FC
-P 2950 4950
-AR Path="/5E9D90FC" Ref="C?"  Part="1"
-AR Path="/5E9BC166/5E9D90FC" Ref="C?"  Part="1"
-AR Path="/5EA3D59C/5E9D90FC" Ref="C?"  Part="1"
-F 0 "C?" H 3065 4996 50  0000 L CNN
-F 1 "10uF" H 3065 4905 50  0000 L CNN
-F 2 "" H 2988 4800 50  0001 C CNN
-F 3 "~" H 2950 4950 50  0001 C CNN
-	1    2950 4950
-	1    0    0    -1
-$EndComp
-$Comp
-L Device:C C?
-U 1 1 5E9D9102
-P 4200 4950
-AR Path="/5E9D9102" Ref="C?"  Part="1"
-AR Path="/5E9BC166/5E9D9102" Ref="C?"  Part="1"
-AR Path="/5EA3D59C/5E9D9102" Ref="C?"  Part="1"
-F 0 "C?" H 4315 4996 50  0000 L CNN
-F 1 "0.1uF" H 4315 4905 50  0000 L CNN
-F 2 "" H 4238 4800 50  0001 C CNN
-F 3 "~" H 4200 4950 50  0001 C CNN
-	1    4200 4950
-	1    0    0    -1
-$EndComp
-$Comp
-L Device:C C?
-U 1 1 5E9D9108
-P 4650 4950
-AR Path="/5E9D9108" Ref="C?"  Part="1"
-AR Path="/5E9BC166/5E9D9108" Ref="C?"  Part="1"
-AR Path="/5EA3D59C/5E9D9108" Ref="C?"  Part="1"
-F 0 "C?" H 4765 4996 50  0000 L CNN
-F 1 "10uF" H 4765 4905 50  0000 L CNN
-F 2 "" H 4688 4800 50  0001 C CNN
-F 3 "~" H 4650 4950 50  0001 C CNN
-	1    4650 4950
-	1    0    0    -1
-$EndComp
-Wire Wire Line
-	3300 4700 2950 4700
-Wire Wire Line
-	2950 4800 2950 4700
-Wire Wire Line
-	4200 4800 4200 4700
-Connection ~ 4200 4700
-Wire Wire Line
-	4200 4700 3900 4700
-Wire Wire Line
-	4650 4800 4650 4700
-Wire Wire Line
-	4650 4700 4200 4700
-$Comp
-L power:GND #PWR?
-U 1 1 5E9D911B
-P 3600 5300
-AR Path="/5E9D911B" Ref="#PWR?"  Part="1"
-AR Path="/5E9BC166/5E9D911B" Ref="#PWR?"  Part="1"
-AR Path="/5EA3D59C/5E9D911B" Ref="#PWR?"  Part="1"
-F 0 "#PWR?" H 3600 5050 50  0001 C CNN
-F 1 "GND" H 3605 5127 50  0000 C CNN
-F 2 "" H 3600 5300 50  0001 C CNN
-F 3 "" H 3600 5300 50  0001 C CNN
-	1    3600 5300
-	1    0    0    -1
-$EndComp
-Wire Wire Line
-	4650 5300 4200 5300
-Connection ~ 3600 5300
-Wire Wire Line
-	3600 5000 3600 5300
-Wire Wire Line
-	4200 5100 4200 5300
-Connection ~ 4200 5300
-Wire Wire Line
-	4200 5300 3600 5300
-Wire Wire Line
-	2950 5100 2950 5300
-Wire Wire Line
-	2950 5300 3600 5300
-Wire Wire Line
-	4650 5100 4650 5300
-Wire Wire Line
-	4650 4500 4650 4700
-Connection ~ 4650 4700
-Wire Wire Line
-	2950 4700 2950 4500
-Connection ~ 2950 4700
-$Comp
-L power:+5VD #PWR?
-U 1 1 5EA5E622
-P 2950 4500
-F 0 "#PWR?" H 2950 4350 50  0001 C CNN
-F 1 "+5VD" H 2965 4673 50  0000 C CNN
-F 2 "" H 2950 4500 50  0001 C CNN
-F 3 "" H 2950 4500 50  0001 C CNN
-	1    2950 4500
-	1    0    0    -1
-$EndComp
+Wire Wire Line
+	4750 6150 4750 6350
 $Comp
 L power:+3V3 #PWR?
 U 1 1 5EA5F12F
-P 4650 4500
-F 0 "#PWR?" H 4650 4350 50  0001 C CNN
-F 1 "+3V3" H 4665 4673 50  0000 C CNN
-F 2 "" H 4650 4500 50  0001 C CNN
-F 3 "" H 4650 4500 50  0001 C CNN
-	1    4650 4500
+P 4750 5550
+F 0 "#PWR?" H 4750 5400 50  0001 C CNN
+F 1 "+3V3" H 4765 5723 50  0000 C CNN
+F 2 "" H 4750 5550 50  0001 C CNN
+F 3 "" H 4750 5550 50  0001 C CNN
+	1    4750 5550
 	1    0    0    -1
 $EndComp
@@
 	1    0    0    -1
 $EndComp
+Connection ~ 4750 5750
+Wire Wire Line
+	4750 5550 4750 5750
+Wire Wire Line
+	4750 5850 4750 5750
+$Comp
+L power:+5VD #PWR?
+U 1 1 5EA5E622
+P 3050 5550
+F 0 "#PWR?" H 3050 5400 50  0001 C CNN
+F 1 "+5VD" H 3065 5723 50  0000 C CNN
+F 2 "" H 3050 5550 50  0001 C CNN
+F 3 "" H 3050 5550 50  0001 C CNN
+	1    3050 5550
+	1    0    0    -1
+$EndComp
+Connection ~ 3050 5750
+Wire Wire Line
+	3050 5750 3050 5550
+Wire Wire Line
+	3050 6350 3700 6350
+Wire Wire Line
+	3050 6150 3050 6350
+Wire Wire Line
+	4300 6350 3700 6350
+Connection ~ 4300 6350
+Wire Wire Line
+	4300 6150 4300 6350
+Wire Wire Line
+	3700 6050 3700 6350
+Connection ~ 3700 6350
+Wire Wire Line
+	4750 6350 4300 6350
+$Comp
+L power:GND #PWR?
+U 1 1 5E9D911B
+P 3700 6350
+AR Path="/5E9D911B" Ref="#PWR?"  Part="1"
+AR Path="/5E9BC166/5E9D911B" Ref="#PWR?"  Part="1"
+AR Path="/5EA3D59C/5E9D911B" Ref="#PWR?"  Part="1"
+F 0 "#PWR?" H 3700 6100 50  0001 C CNN
+F 1 "GND" H 3705 6177 50  0000 C CNN
+F 2 "" H 3700 6350 50  0001 C CNN
+F 3 "" H 3700 6350 50  0001 C CNN
+	1    3700 6350
+	1    0    0    -1
+$EndComp
+Wire Wire Line
+	4750 5750 4300 5750
+Wire Wire Line
+	4300 5750 4000 5750
+Connection ~ 4300 5750
+Wire Wire Line
+	4300 5850 4300 5750
+Wire Wire Line
+	3050 5850 3050 5750
+Wire Wire Line
+	3400 5750 3050 5750
+$Comp
+L Device:C C?
+U 1 1 5E9D9108
+P 4750 6000
+AR Path="/5E9D9108" Ref="C?"  Part="1"
+AR Path="/5E9BC166/5E9D9108" Ref="C?"  Part="1"
+AR Path="/5EA3D59C/5E9D9108" Ref="C?"  Part="1"
+F 0 "C?" H 4865 6046 50  0000 L CNN
+F 1 "10uF" H 4865 5955 50  0000 L CNN
+F 2 "" H 4788 5850 50  0001 C CNN
+F 3 "~" H 4750 6000 50  0001 C CNN
+	1    4750 6000
+	1    0    0    -1
+$EndComp
+$Comp
+L Device:C C?
+U 1 1 5E9D9102
+P 4300 6000
+AR Path="/5E9D9102" Ref="C?"  Part="1"
+AR Path="/5E9BC166/5E9D9102" Ref="C?"  Part="1"
+AR Path="/5EA3D59C/5E9D9102" Ref="C?"  Part="1"
+F 0 "C?" H 4415 6046 50  0000 L CNN
+F 1 "0.1uF" H 4415 5955 50  0000 L CNN
+F 2 "" H 4338 5850 50  0001 C CNN
+F 3 "~" H 4300 6000 50  0001 C CNN
+	1    4300 6000
+	1    0    0    -1
+$EndComp
+$Comp
+L Device:C C?
+U 1 1 5E9D90FC
+P 3050 6000
+AR Path="/5E9D90FC" Ref="C?"  Part="1"
+AR Path="/5E9BC166/5E9D90FC" Ref="C?"  Part="1"
+AR Path="/5EA3D59C/5E9D90FC" Ref="C?"  Part="1"
+F 0 "C?" H 3165 6046 50  0000 L CNN
+F 1 "10uF" H 3165 5955 50  0000 L CNN
+F 2 "" H 3088 5850 50  0001 C CNN
+F 3 "~" H 3050 6000 50  0001 C CNN
+	1    3050 6000
+	1    0    0    -1
+$EndComp
+$Comp
+L Regulator_Linear:LM1117-3.3 U?
+U 1 1 5E9D90F6
+P 3700 5750
+AR Path="/5E9D90F6" Ref="U?"  Part="1"
+AR Path="/5E9BC166/5E9D90F6" Ref="U?"  Part="1"
+AR Path="/5EA3D59C/5E9D90F6" Ref="U?"  Part="1"
+F 0 "U?" H 3700 5992 50  0000 C CNN
+F 1 "LM1117-3.3" H 3700 5901 50  0000 C CNN
+F 2 "" H 3700 5750 50  0001 C CNN
+F 3 "http://www.ti.com/lit/ds/symlink/lm1117.pdf" H 3700 5750 50  0001 C CNN
+	1    3700 5750
+	1    0    0    -1
+$EndComp
+Wire Notes Line
+	11250 4350 450  4350
+Text Notes 500  4300 0    50   ~ 0
+CARGADOR DE BATERIA
+Text Notes 500  7750 0    50   ~ 0
+REGULADOR 3.3V
 $EndSCHEMATC

Commit message: Add files via upload
Parts:
- removed C?: 10uF, symbol Device:C
- removed U?: LM1117-3.3, symbol Regulator_Linear:LM1117-3.3
- added C21, C? (x2): 10uF, symbol Device:C
- added C?: 0.1uF, symbol Device:C
- added U7: LM1117-3.3, symbol Regulator_Linear:LM1117-3.3
- added U?: LM1117-5.0, symbol Regulator_Linear:LM1117-5.0
- gave numbers to parts that had none: 18
Connections:
- net +3V3: now also U7.2 (VO)
- net +5VD: now also C?.1, C?.1, U?.2 (VO); no longer C27.1, D6.1 (K), R19.1, U9.10 (FB), U9.2 (VOUT)
- net GND: now also C21.2, C?.2, C?.2, C?.2, U7.1 (GND), U?.1 (GND)
- net at J8.2 (D-): now also J8.3 (D+)
- new net +5VP: C21.1, C27.1, C?.1, D6.1 (K), R19.1, U7.3 (VI), U9.10 (FB), U9.2 (VOUT), U?.3 (VI)
Other:
- note added: "REGULADOR 5V"
- moved on the sheet: BT2, C20, C22, C23, C24, C25, C26, C27, D6, J8, L8, Q2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

Commit message: Add files via upload
Parts:
- C20, C21, C22, C23, C24, C25, C26, C27: footprint (none) -> Capacitor_SMD:C_0603_1608Metric_Pad1.05x0.95mm_HandSolder
- C40, C41, C42: renamed from C?; footprint (none) -> Capacitor_SMD:C_0603_1608Metric_Pad1.05x0.95mm_HandSolder
- D6: footprint (none) -> Diode_SMD:D_0603_1608Metric_Pad1.05x0.95mm_HandSolder
- J8: footprint (none) -> Connector_USB:USB_Mini-B_AdamTech_MUSB-B5-S-VT-TSMT-1_SMD_Vertical
- L8: footprint (none) -> Inductor_SMD:L_2010_5025Metric
- R16, R18, R19: footprint (none) -> Resistor_SMD:R_0201_0603Metric
- U12: renamed from U?; footprint (none) -> Package_TO_SOT_SMD:SOT-223
- U7: footprint (none) -> Package_TO_SOT_SMD:SOT-223
Changed lines of the file:
@@
 F 0 "D6" H 7950 3834 50  0000 C CNN
 F 1 "D_Schottky" H 7950 3925 50  0000 C CNN
-F 2 "" H 7950 4050 50  0001 C CNN
+F 2 "Diode_SMD:D_0603_1608Metric_Pad1.05x0.95mm_HandSolder" H 7950 4050 50  0001 C CNN
 F 3 "~" H 7950 4050 50  0001 C CNN
 	1    7950 4050
@@
 F 0 "R19" H 9470 4496 50  0000 L CNN
 F 1 "10K" H 9470 4405 50  0000 L CNN
-F 2 "" V 9330 4450 50  0001 C CNN
+F 2 "Resistor_SMD:R_0201_0603Metric" V 9330 4450 50  0001 C CNN
 F 3 "~" H 9400 4450 50  0001 C CNN
 	1    9400 4450
@@
 F 0 "C27" H 9915 5596 50  0000 L CNN
 F 1 "22uF" H 9915 5505 50  0000 L CNN
-F 2 "" H 9838 5400 50  0001 C CNN
+F 2 "Capacitor_SMD:C_0603_1608Metric_Pad1.05x0.95mm_HandSolder" H 9838 5400 50  0001 C CNN
 F 3 "~" H 9800 5550 50  0001 C CNN
 	1    9800 5550
@@
 F 0 "C26" H 9365 5596 50  0000 L CNN
 F 1 "1uF" H 9365 5505 50  0000 L CNN
-F 2 "" H 9288 5400 50  0001 C CNN
+F 2 "Capacitor_SMD:C_0603_1608Metric_Pad1.05x0.95mm_HandSolder" H 9288 5400 50  0001 C CNN
 F 3 "~" H 9250 5550 50  0001 C CNN
 	1    9250 5550
@@
 F 0 "L8" V 8650 4700 50  0000 C CNN
 F 1 "2.2uH" V 8550 4700 50  0000 C CNN
-F 2 "" H 8450 4700 50  0001 C CNN
+F 2 "Inductor_SMD:L_2010_5025Metric" H 8450 4700 50  0001 C CNN
 F 3 "~" H 8450 4700 50  0001 C CNN
 	1    8450 4700
@@
 F 0 "C25" H 7365 5246 50  0000 L CNN
 F 1 "4.7uF" H 7365 5155 50  0000 L CNN
-F 2 "" H 7288 5050 50  0001 C CNN
+F 2 "Capacitor_SMD:C_0603_1608Metric_Pad1.05x0.95mm_HandSolder" H 7288 5050 50  0001 C CNN
 F 3 "~" H 7250 5200 50  0001 C CNN
 	1    7250 5200
@@
 F 0 "R18" H 7670 5646 50  0000 L CNN
 F 1 "180K" H 7670 5555 50  0000 L CNN
-F 2 "" V 7530 5600 50  0001 C CNN
+F 2 "Resistor_SMD:R_0201_0603Metric" V 7530 5600 50  0001 C CNN
 F 3 "~" H 7600 5600 50  0001 C CNN
 	1    7600 5600
@@
 F 0 "C24" H 5965 4996 50  0000 L CNN
 F 1 "4.7uF" H 5965 4905 50  0000 L CNN
-F 2 "" H 5888 4800 50  0001 C CNN
+F 2 "Capacitor_SMD:C_0603_1608Metric_Pad1.05x0.95mm_HandSolder" H 5888 4800 50  0001 C CNN
 F 3 "~" H 5850 4950 50  0001 C CNN
 	1    5850 4950
@@
 F 0 "R16" V 4143 4900 50  0000 C CNN
 F 1 "10K" V 4234 4900 50  0000 C CNN
-F 2 "" V 4280 4900 50  0001 C CNN
+F 2 "Resistor_SMD:R_0201_0603Metric" V 4280 4900 50  0001 C CNN
 F 3 "~" H 4350 4900 50  0001 C CNN
 	1    4350 4900
@@
 F 0 "C20" H 4015 4696 50  0000 L CNN
 F 1 "4.7uF" H 4015 4605 50  0000 L CNN
-F 2 "" H 3938 4500 50  0001 C CNN
+F 2 "Capacitor_SMD:C_0603_1608Metric_Pad1.05x0.95mm_HandSolder" H 3938 4500 50  0001 C CNN
 F 3 "~" H 3900 4650 50  0001 C CNN
 	1    3900 4650
@@
 F 0 "J8" H 3157 5017 50  0000 C CNN
 F 1 "USB_B_Mini" H 3157 4926 50  0000 C CNN
-F 2 "" H 3250 4500 50  0001 C CNN
+F 2 "Connector_USB:USB_Mini-B_AdamTech_MUSB-B5-S-VT-TSMT-1_SMD_Vertical" H 3250 4500 50  0001 C CNN
 F 3 "~" H 3250 4500 50  0001 C CNN
 	1    3100 4550
@@
 F 0 "C23" H 3965 1896 50  0000 L CNN
 F 1 "10uF" H 3965 1805 50  0000 L CNN
-F 2 "" H 3888 1700 50  0001 C CNN
+F 2 "Capacitor_SMD:C_0603_1608Metric_Pad1.05x0.95mm_HandSolder" H 3888 1700 50  0001 C CNN
 F 3 "~" H 3850 1850 50  0001 C CNN
 	1    3850 1850
@@
 F 0 "C22" H 3515 1896 50  0000 L CNN
 F 1 "0.1uF" H 3515 1805 50  0000 L CNN
-F 2 "" H 3438 1700 50  0001 C CNN
+F 2 "Capacitor_SMD:C_0603_1608Metric_Pad1.05x0.95mm_HandSolder" H 3438 1700 50  0001 C CNN
 F 3 "~" H 3400 1850 50  0001 C CNN
 	1    3400 1850
@@
 F 0 "C21" H 2265 1896 50  0000 L CNN
 F 1 "10uF" H 2265 1805 50  0000 L CNN
-F 2 "" H 2188 1700 50  0001 C CNN
+F 2 "Capacitor_SMD:C_0603_1608Metric_Pad1.05x0.95mm_HandSolder" H 2188 1700 50  0001 C CNN
 F 3 "~" H 2150 1850 50  0001 C CNN
 	1    2150 1850
@@
 F 0 "U7" H 2800 1842 50  0000 C CNN
 F 1 "LM1117-3.3" H 2800 1751 50  0000 C CNN
-F 2 "" H 2800 1600 50  0001 C CNN
+F 2 "Package_TO_SOT_SMD:SOT-223" H 2800 1600 50  0001 C CNN
 F 3 "http://www.ti.com/lit/ds/symlink/lm1117.pdf" H 2800 1600 50  0001 C CNN
 	1    2800 1600
@@
 AR Path="/5EAC03C0" Ref="C?"  Part="1"
 AR Path="/5E9BC166/5EAC03C0" Ref="C?"  Part="1"
-AR Path="/5EA3D59C/5EAC03C0" Ref="C?"  Part="1"
-F 0 "C?" H 7765 1896 50  0000 L CNN
+AR Path="/5EA3D59C/5EAC03C0" Ref="C40"  Part="1"
+F 0 "C40" H 7765 1896 50  0000 L CNN
 F 1 "10uF" H 7765 1805 50  0000 L CNN
-F 2 "" H 7688 1700 50  0001 C CNN
+F 2 "Capacitor_SMD:C_0603_1608Metric_Pad1.05x0.95mm_HandSolder" H 7688 1700 50  0001 C CNN
 F 3 "~" H 7650 1850 50  0001 C CNN
 	1    7650 1850
@@
 $EndComp
 $Comp
-L power:+5VP #PWR?
+L power:+5VP #PWR0165
 U 1 1 5EAC405A
 P 10400 5000
-F 0 "#PWR?" H 10400 4850 50  0001 C CNN
+F 0 "#PWR0165" H 10400 4850 50  0001 C CNN
 F 1 "+5VP" H 10415 5173 50  0000 C CNN
 F 2 "" H 10400 5000 50  0001 C CNN
@@
 $EndComp
 $Comp
-L power:+5VP #PWR?
+L power:+5VP #PWR0166
 U 1 1 5EAC488F
 P 2150 1400
-F 0 "#PWR?" H 2150 1250 50  0001 C CNN
+F 0 "#PWR0166" H 2150 1250 50  0001 C CNN
 F 1 "+5VP" H 2165 1573 50  0000 C CNN
 F 2 "" H 2150 1400 50  0001 C CNN
@@
 $EndComp
 $Comp
-L power:+5VP #PWR?
+L power:+5VP #PWR0167
 U 1 1 5EAC54AC
 P 7650 1400
-F 0 "#PWR?" H 7650 1250 50  0001 C CNN
+F 0 "#PWR0167" H 7650 1250 50  0001 C CNN
 F 1 "+5VP" H 7665 1573 50  0000 C CNN
 F 2 "" H 7650 1400 50  0001 C CNN
@@
 Connection ~ 8300 2200
 $Comp
-L power:+5VD #PWR?
+L power:+5VD #PWR0168
 U 1 1 5EAC3757
 P 9350 1400
-F 0 "#PWR?" H 9350 1250 50  0001 C CNN
+F 0 "#PWR0168" H 9350 1250 50  0001 C CNN
 F 1 "+5VD" H 9365 1573 50  0000 C CNN
 F 2 "" H 9350 1400 50  0001 C CNN
@@
 AR Path="/5EAC03BA" Ref="C?"  Part="1"
 AR Path="/5E9BC166/5EAC03BA" Ref="C?"  Part="1"
-AR Path="/5EA3D59C/5EAC03BA" Ref="C?"  Part="1"
-F 0 "C?" H 9015 1896 50  0000 L CNN
+AR Path="/5EA3D59C/5EAC03BA" Ref="C41"  Part="1"
+F 0 "C41" H 9015 1896 50  0000 L CNN
 F 1 "0.1uF" H 9015 1805 50  0000 L CNN
-F 2 "" H 8938 1700 50  0001 C CNN
+F 2 "Capacitor_SMD:C_0603_1608Metric_Pad1.05x0.95mm_HandSolder" H 8938 1700 50  0001 C CNN
 F 3 "~" H 8900 1850 50  0001 C CNN
 	1    8900 1850
@@
 AR Path="/5EAC03B4" Ref="C?"  Part="1"
 AR Path="/5E9BC166/5EAC03B4" Ref="C?"  Part="1"
-AR Path="/5EA3D59C/5EAC03B4" Ref="C?"  Part="1"
-F 0 "C?" H 9465 1896 50  0000 L CNN
+AR Path="/5EA3D59C/5EAC03B4" Ref="C42"  Part="1"
+F 0 "C42" H 9465 1896 50  0000 L CNN
 F 1 "10uF" H 9465 1805 50  0000 L CNN
-F 2 "" H 9388 1700 50  0001 C CNN
+F 2 "Capacitor_SMD:C_0603_1608Metric_Pad1.05x0.95mm_HandSolder" H 9388 1700 50  0001 C CNN
 F 3 "~" H 9350 1850 50  0001 C CNN
 	1    9350 1850
@@
 AR Path="/5EAC03A4" Ref="#PWR?"  Part="1"
 AR Path="/5E9BC166/5EAC03A4" Ref="#PWR?"  Part="1"
-AR Path="/5EA3D59C/5EAC03A4" Ref="#PWR?"  Part="1"
-F 0 "#PWR?" H 8300 1950 50  0001 C CNN
+AR Path="/5EA3D59C/5EAC03A4" Ref="#PWR0169"  Part="1"
+F 0 "#PWR0169" H 8300 1950 50  0001 C CNN
 F 1 "GND" H 8305 2027 50  0000 C CNN
 F 2 "" H 8300 2200 50  0001 C CNN
@@
 P 8300 1600
 AR Path="/5E9BC166/5EAC0394" Ref="U?"  Part="1"
-AR Path="/5EA3D59C/5EAC0394" Ref="U?"  Part="1"
-F 0 "U?" H 8300 1842 50  0000 C CNN
+AR Path="/5EA3D59C/5EAC0394" Ref="U12"  Part="1"
+F 0 "U12" H 8300 1842 50  0000 C CNN
 F 1 "LM1117-5.0" H 8300 1751 50  0000 C CNN
-F 2 "" H 8300 1600 50  0001 C CNN
+F 2 "Package_TO_SOT_SMD:SOT-223" H 8300 1600 50  0001 C CNN
 F 3 "http://www.ti.com/lit/ds/symlink/lm1117.pdf" H 8300 1600 50  0001 C CNN
 	1    8300 1600

Commit message: Add files via upload
Parts:
- Q2: footprint (none) -> Diode_SMD:D_0805_2012Metric
- R17: footprint (none) -> Resistor_SMD:R_0201_0603Metric
Changed lines of the file:
@@
 F 0 "R17" H 7670 5146 50  0000 L CNN
 F 1 "2M" H 7670 5055 50  0000 L CNN
-F 2 "" V 7530 5100 50  0001 C CNN
+F 2 "Resistor_SMD:R_0201_0603Metric" V 7530 5100 50  0001 C CNN
 F 3 "~" H 7600 5100 50  0001 C CNN
 	1    7600 5100
@@
 F 0 "Q2" V 7099 4600 50  0000 C CNN
 F 1 "Q_PMOS_DSG" V 7190 4600 50  0000 C CNN
-F 2 "" H 7050 4700 50  0001 C CNN
+F 2 "Diode_SMD:D_0805_2012Metric" H 7050 4700 50  0001 C CNN
 F 3 "~" H 6850 4600 50  0001 C CNN
 	1    6850 4600
