File: proyecto/Alimentacion_camara.sch (KiCad schematic (older format))
At the start: 24 parts, among them J8 USB_B_Mini, Q2 Q_PMOS_DSG, U12 LM1117-5.0, U7 LM1117-3.3, U8 MCP73811T-435I-OT, U9 TPS61200DRC

Commit message: Add files via upload
Parts:
- Q2: footprint Diode_SMD:D_0805_2012Metric -> Package_TO_SOT_SMD:SOT-23
Changed lines of the file:
@@
 F 0 "Q2" V 7099 4600 50  0000 C CNN
 F 1 "Q_PMOS_DSG" V 7190 4600 50  0000 C CNN
-F 2 "Diode_SMD:D_0805_2012Metric" H 7050 4700 50  0001 C CNN
+F 2 "Package_TO_SOT_SMD:SOT-23" H 7050 4700 50  0001 C CNN
 F 3 "~" H 6850 4600 50  0001 C CNN
 	1    6850 4600

Commit message: Add files via upload
Parts:
- removed BT2: Battery_Cell_2, Battery:Battery_Panasonic_CR3032-VCN_Vertical_CircularHoles, symbol Device:Battery_Cell
- added J10: Conn_01x02, Connector_PinHeader_1.00mm:PinHeader_1x02_P1.00mm_Horizontal, symbol Connector_Generic:Conn_01x02
- L8: footprint Inductor_SMD:L_2010_5025Metric -> Inductor_SMD:L_2010_5025Metric_Pad1.52x2.65mm_HandSolder
- R16, R17, R18, R19: footprint Resistor_SMD:R_0201_0603Metric -> Resistor_SMD:R_0603_1608Metric_Pad1.05x0.95mm_HandSolder
Connections:
- net GNDA: now also J10.2 (Pin_2)
- net at C24.1, Q2.2 (S), U8.3 (VBAT): now also J10.1 (Pin_1)
Changed lines of the file:
@@
 F 0 "R19" H 9470 4496 50  0000 L CNN
 F 1 "10K" H 9470 4405 50  0000 L CNN
-F 2 "Resistor_SMD:R_0201_0603Metric" V 9330 4450 50  0001 C CNN
+F 2 "Resistor_SMD:R_0603_1608Metric_Pad1.05x0.95mm_HandSolder" V 9330 4450 50  0001 C CNN
 F 3 "~" H 9400 4450 50  0001 C CNN
 	1    9400 4450
@@
 F 0 "L8" V 8650 4700 50  0000 C CNN
 F 1 "2.2uH" V 8550 4700 50  0000 C CNN
-F 2 "Inductor_SMD:L_2010_5025Metric" H 8450 4700 50  0001 C CNN
+F 2 "Inductor_SMD:L_2010_5025Metric_Pad1.52x2.65mm_HandSolder" H 8450 4700 50  0001 C CNN
 F 3 "~" H 8450 4700 50  0001 C CNN
 	1    8450 4700
@@
 F 0 "R18" H 7670 5646 50  0000 L CNN
 F 1 "180K" H 7670 5555 50  0000 L CNN
-F 2 "Resistor_SMD:R_0201_0603Metric" V 7530 5600 50  0001 C CNN
+F 2 "Resistor_SMD:R_0603_1608Metric_Pad1.05x0.95mm_HandSolder" V 7530 5600 50  0001 C CNN
 F 3 "~" H 7600 5600 50  0001 C CNN
 	1    7600 5600
@@
 F 0 "R17" H 7670 5146 50  0000 L CNN
 F 1 "2M" H 7670 5055 50  0000 L CNN
-F 2 "Resistor_SMD:R_0201_0603Metric" V 7530 5100 50  0001 C CNN
+F 2 "Resistor_SMD:R_0603_1608Metric_Pad1.05x0.95mm_HandSolder" V 7530 5100 50  0001 C CNN
 F 3 "~" H 7600 5100 50  0001 C CNN
 	1    7600 5100
@@
 	1    0    0    -1
 $EndComp
-Connection ~ 6300 4700
-Wire Wire Line
-	6650 4700 6300 4700
+Connection ~ 6200 4700
+Wire Wire Line
+	6650 4700 6200 4700
 $Comp
 L Device:Q_PMOS_DSG Q2
@@
 Connection ~ 5150 5250
 Wire Wire Line
-	6300 5250 5850 5250
-Wire Wire Line
-	6300 5100 6300 5250
-Wire Wire Line
-	5850 4700 6300 4700
+	6200 5250 5850 5250
+Wire Wire Line
+	5850 4700 6200 4700
 Connection ~ 5850 4700
 Wire Wire Line
 	5850 4800 5850 4700
-Wire Wire Line
-	6300 4700 6300 4800
 Wire Wire Line
 	5550 4700 5850 4700
@@
 	5150 4500 5150 4350
 $Comp
-L Device:Battery_Cell BT2
-U 1 1 5EA3E896
-P 6300 5000
-F 0 "BT2" H 6350 4950 50  0000 L CNN
-F 1 "Battery_Cell_2" H 6350 4850 50  0000 L CNN
-F 2 "Battery:Battery_Panasonic_CR3032-VCN_Vertical_CircularHoles" V 6300 5060 50  0001 C CNN
-F 3 "~" V 6300 5060 50  0001 C CNN
-	1    6300 5000
-	1    0    0    -1
-$EndComp
-$Comp
 L Device:C C24
 U 1 1 5EA3CD6D
@@
 F 0 "R16" V 4143 4900 50  0000 C CNN
 F 1 "10K" V 4234 4900 50  0000 C CNN
-F 2 "Resistor_SMD:R_0201_0603Metric" V 4280 4900 50  0001 C CNN
+F 2 "Resistor_SMD:R_0603_1608Metric_Pad1.05x0.95mm_HandSolder" V 4280 4900 50  0001 C CNN
 F 3 "~" H 4350 4900 50  0001 C CNN
 	1    4350 4900
@@
 	3400 2200 2800 2200
 Connection ~ 3400 2200
+$Comp
+L Connector_Generic:Conn_01x02 J10
+U 1 1 5ECF7F80
+P 6400 5150
+F 0 "J10" H 6480 5142 50  0000 L CNN
+F 1 "Conn_01x02" H 6480 5051 50  0000 L CNN
+F 2 "Connector_PinHeader_1.00mm:PinHeader_1x02_P1.00mm_Horizontal" H 6400 5150 50  0001 C CNN
+F 3 "~" H 6400 5150 50  0001 C CNN
+	1    6400 5150
+	1    0    0    -1
+$EndComp
+Wire Wire Line
+	6200 4700 6200 5150
 $EndSCHEMATC

Commit message: Add files via upload
Parts:
- added FL5, FL6, FL7, FL8: BLM18SG121TN1D, Resistor_SMD:R_0603_1608Metric_Pad1.05x0.95mm_HandSolder, symbol BLM18SG121TN1D:BLM18SG121TN1D
- added H5, H6, H7, H8: MountingHole_Pad, MountingHole:MountingHole_2.5mm_Pad, symbol Mechanical:MountingHole_Pad
Connections:
- net GNDA: now also FL5.2, FL6.2, FL7.2, FL8.2
- new net: FL5.1, H5.1
- new net: FL6.1, H6.1
- new net: FL7.1, H7.1
- new net: FL8.1, H8.1
Other:
- moved on the sheet: C21, C22, C23, C40, C41, C42, U12, U7
