File: proyecto/Procesador.sch (KiCad schematic (older format))
At the start: 16 parts

Commit message: Add files via upload
Connections:
- net TD0: now reaches U?.19
- net TRST: now reaches U?.2 (11)
- net TD1: now reaches U?.20 (18)
- net SRST: now reaches U?.5 (17)
- net TCK: now reaches U?.6 (16)
- net TMS: now reaches U?.7 (15)
- net 3.3v renamed +3V3
- net 5v renamed +5V
Other:
- moved on the sheet: C?, D?, J?, L?, R?, SW?

Commit message: Add files via upload
Parts:
- added J?: Conn_ARM_JTAG_SWD_20, symbol Connector:Conn_ARM_JTAG_SWD_20
- added R?: 510, symbol Device:R
Connections:
- net +3V3: now also J?.1 (VTREF), J?.2 (VCC/NC)
- net GND: now also J?.10 (GND), J?.12 (GND), J?.14 (GND), J?.16 (GND), J?.18 (GND), J?.20 (GND), J?.4 (GND), J?.6 (GND), J?.8 (GND), R?.1
- net SRST renamed SRST2
- net SRST2: now also J?.15 (~SRST~)
- net TCK renamed TCK2
- net TCK2: now also J?.9 (TCK/SWDCLK)
- net TD0 renamed TD02
- net TD02: now also J?.13 (TDO/SWO)
- net TD1 renamed TD12
- net TD12: now also J?.5 (TDI)
- net TMS renamed TMS2
- net TMS2: now also J?.7 (TMS/SWDIO)
- net TRST renamed TRST2
- net TRST2: now also J?.3 (~TRST~)
- new net: J?.11 (RTCK), R?.2
Other:
- moved on the sheet: C?, R?, SW?, U?

Commit message: Add files via upload
Other:
- note added: "JTAG"
- note added: "PROCESADOR"
- note added: "RESET"
- note added: "USB"
- moved on the sheet: C?, D?, J?, L?, R?, SW?, U?

Commit message: Add files via upload
Parts:
- gave numbers to parts that had none: 18
Changed lines of the file:
@@
 P 2650 2250
 AR Path="/5EA0EFB0" Ref="D?"  Part="1"
-AR Path="/5E9F954D/5EA0EFB0" Ref="D?"  Part="1"
-F 0 "D?" H 2855 2296 50  0000 L CNN
+AR Path="/5E9F954D/5EA0EFB0" Ref="D2"  Part="1"
+F 0 "D2" H 2855 2296 50  0000 L CNN
 F 1 "SP0502BAHT" H 2855 2205 50  0000 L CNN
 F 2 "Package_TO_SOT_SMD:SOT-23" H 2875 2200 50  0001 L CNN
@@
 P 1900 1850
 AR Path="/5EA0EFB6" Ref="J?"  Part="1"
-AR Path="/5E9F954D/5EA0EFB6" Ref="J?"  Part="1"
-F 0 "J?" H 1957 2317 50  0000 C CNN
+AR Path="/5E9F954D/5EA0EFB6" Ref="J3"  Part="1"
+F 0 "J3" H 1957 2317 50  0000 C CNN
 F 1 "USB_A" H 1957 2226 50  0000 C CNN
 F 2 "" H 2050 1800 50  0001 C CNN
@@
 P 2650 2600
 AR Path="/5EA0EFC1" Ref="#PWR?"  Part="1"
-AR Path="/5E9F954D/5EA0EFC1" Ref="#PWR?"  Part="1"
-F 0 "#PWR?" H 2650 2350 50  0001 C CNN
+AR Path="/5E9F954D/5EA0EFC1" Ref="#PWR0107"  Part="1"
+F 0 "#PWR0107" H 2650 2350 50  0001 C CNN
 F 1 "GND" H 2655 2427 50  0000 C CNN
 F 2 "" H 2650 2600 50  0001 C CNN
@@
 P 3000 1950
 AR Path="/5EA0EFC8" Ref="L?"  Part="1"
-AR Path="/5E9F954D/5EA0EFC8" Ref="L?"  Part="1"
-F 0 "L?" V 3190 1950 50  0000 C CNN
+AR Path="/5E9F954D/5EA0EFC8" Ref="L1"  Part="1"
+F 0 "L1" V 3190 1950 50  0000 C CNN
 F 1 "L" V 3099 1950 50  0000 C CNN
 F 2 "" H 3000 1950 50  0001 C CNN
@@
 P 3100 1850
 AR Path="/5EA0EFCE" Ref="L?"  Part="1"
-AR Path="/5E9F954D/5EA0EFCE" Ref="L?"  Part="1"
-F 0 "L?" V 3290 1850 50  0000 C CNN
+AR Path="/5E9F954D/5EA0EFCE" Ref="L2"  Part="1"
+F 0 "L2" V 3290 1850 50  0000 C CNN
 F 1 "L" V 3199 1850 50  0000 C CNN
 F 2 "" H 3100 1850 50  0001 C CNN
@@
 P 3600 1850
 AR Path="/5EA0EFD4" Ref="R?"  Part="1"
-AR Path="/5E9F954D/5EA0EFD4" Ref="R?"  Part="1"
-F 0 "R?" V 3393 1850 50  0000 C CNN
+AR Path="/5E9F954D/5EA0EFD4" Ref="R5"  Part="1"
+F 0 "R5" V 3393 1850 50  0000 C CNN
 F 1 "R" V 3484 1850 50  0000 C CNN
 F 2 "" V 3530 1850 50  0001 C CNN
@@
 P 3450 1950
 AR Path="/5EA0EFDA" Ref="R?"  Part="1"
-AR Path="/5E9F954D/5EA0EFDA" Ref="R?"  Part="1"
-F 0 "R?" V 3243 1950 50  0000 C CNN
+AR Path="/5E9F954D/5EA0EFDA" Ref="R4"  Part="1"
+F 0 "R4" V 3243 1950 50  0000 C CNN
 F 1 "R" V 3334 1950 50  0000 C CNN
 F 2 "" V 3380 1950 50  0001 C CNN
@@
 P 2500 1200
 AR Path="/5EA0EFF0" Ref="D?"  Part="1"
-AR Path="/5E9F954D/5EA0EFF0" Ref="D?"  Part="1"
-F 0 "D?" V 2454 1279 50  0000 L CNN
+AR Path="/5E9F954D/5EA0EFF0" Ref="D1"  Part="1"
+F 0 "D1" V 2454 1279 50  0000 L CNN
 F 1 "1N47xxA" V 2545 1279 50  0000 L CNN
 F 2 "Diode_THT:D_DO-41_SOD81_P10.16mm_Horizontal" H 2500 1025 50  0001 C CNN
@@
 P 2900 1200
 AR Path="/5EA0EFF6" Ref="C?"  Part="1"
-AR Path="/5E9F954D/5EA0EFF6" Ref="C?"  Part="1"
-F 0 "C?" H 3015 1246 50  0000 L CNN
+AR Path="/5E9F954D/5EA0EFF6" Ref="C2"  Part="1"
+F 0 "C2" H 3015 1246 50  0000 L CNN
 F 1 "C" H 3015 1155 50  0000 L CNN
 F 2 "" H 2938 1050 50  0001 C CNN
@@
 P 3250 1200
 AR Path="/5EA0EFFC" Ref="C?"  Part="1"
-AR Path="/5E9F954D/5EA0EFFC" Ref="C?"  Part="1"
-F 0 "C?" H 3365 1246 50  0000 L CNN
+AR Path="/5E9F954D/5EA0EFFC" Ref="C3"  Part="1"
+F 0 "C3" H 3365 1246 50  0000 L CNN
 F 1 "C" H 3365 1155 50  0000 L CNN
 F 2 "" H 3288 1050 50  0001 C CNN
@@
 P 2750 1550
 AR Path="/5EA0F002" Ref="#PWR?"  Part="1"
-AR Path="/5E9F954D/5EA0F002" Ref="#PWR?"  Part="1"
-F 0 "#PWR?" H 2750 1300 50  0001 C CNN
+AR Path="/5E9F954D/5EA0F002" Ref="#PWR0108"  Part="1"
+F 0 "#PWR0108" H 2750 1300 50  0001 C CNN
 F 1 "GND" H 2755 1377 50  0000 C CNN
 F 2 "" H 2750 1550 50  0001 C CNN
@@
 P 3650 950
 AR Path="/5EA0F00D" Ref="L?"  Part="1"
-AR Path="/5E9F954D/5EA0F00D" Ref="L?"  Part="1"
-F 0 "L?" V 3840 950 50  0000 C CNN
+AR Path="/5E9F954D/5EA0F00D" Ref="L3"  Part="1"
+F 0 "L3" V 3840 950 50  0000 C CNN
 F 1 "L" V 3749 950 50  0000 C CNN
 F 2 "" H 3650 950 50  0001 C CNN
@@
 P 1900 2450
 AR Path="/5EA0F02B" Ref="#PWR?"  Part="1"
-AR Path="/5E9F954D/5EA0F02B" Ref="#PWR?"  Part="1"
-F 0 "#PWR?" H 1900 2200 50  0001 C CNN
+AR Path="/5E9F954D/5EA0F02B" Ref="#PWR0109"  Part="1"
+F 0 "#PWR0109" H 1900 2200 50  0001 C CNN
 F 1 "GND" H 1905 2277 50  0000 C CNN
 F 2 "" H 1900 2450 50  0001 C CNN
@@
 USB_D-
 $Comp
-L power:+5V #PWR?
+L power:+5V #PWR0110
 U 1 1 5E9CC544
 P 4000 800
-F 0 "#PWR?" H 4000 650 50  0001 C CNN
+F 0 "#PWR0110" H 4000 650 50  0001 C CNN
 F 1 "+5V" H 4015 973 50  0000 C CNN
 F 2 "" H 4000 800 50  0001 C CNN
@@
 P 8500 5700
 AR Path="/5E9DF408/5EA20F46" Ref="#PWR?"  Part="1"
-AR Path="/5E9F954D/5EA20F46" Ref="#PWR?"  Part="1"
-F 0 "#PWR?" H 8500 5450 50  0001 C CNN
+AR Path="/5E9F954D/5EA20F46" Ref="#PWR0111"  Part="1"
+F 0 "#PWR0111" H 8500 5450 50  0001 C CNN
 F 1 "GND" H 8505 5527 50  0000 C CNN
 F 2 "" H 8500 5700 50  0001 C CNN
@@
 P 10000 4600
 AR Path="/5E9DF408/5EA20F58" Ref="R?"  Part="1"
-AR Path="/5E9F954D/5EA20F58" Ref="R?"  Part="1"
-F 0 "R?" V 9793 4600 50  0001 C CNN
+AR Path="/5E9F954D/5EA20F58" Ref="R7"  Part="1"
+F 0 "R7" V 9793 4600 50  0001 C CNN
 F 1 "510" V 9885 4600 50  0000 C CNN
 F 2 "" V 9930 4600 50  0001 C CNN
@@
 P 10400 4600
 AR Path="/5E9DF408/5EA20F60" Ref="#PWR?"  Part="1"
-AR Path="/5E9F954D/5EA20F60" Ref="#PWR?"  Part="1"
-F 0 "#PWR?" H 10400 4350 50  0001 C CNN
+AR Path="/5E9F954D/5EA20F60" Ref="#PWR0112"  Part="1"
+F 0 "#PWR0112" H 10400 4350 50  0001 C CNN
 F 1 "GND" V 10405 4472 50  0000 R CNN
 F 2 "" H 10400 4600 50  0001 C CNN
@@
 	3800 3600 3800 3800
 $Comp
-L power:+3.3V #PWR?
+L power:+3.3V #PWR0113
 U 1 1 5E9C8B2C
 P 3800 3600
-F 0 "#PWR?" H 3800 3450 50  0001 C CNN
+F 0 "#PWR0113" H 3800 3450 50  0001 C CNN
 F 1 "+3.3V" H 3815 3773 50  0000 C CNN
 F 2 "" H 3800 3600 50  0001 C CNN
@@
 P 3550 4200
 AR Path="/5EA0F057" Ref="#PWR?"  Part="1"
-AR Path="/5E9F954D/5EA0F057" Ref="#PWR?"  Part="1"
-F 0 "#PWR?" H 3550 3950 50  0001 C CNN
+AR Path="/5E9F954D/5EA0F057" Ref="#PWR0114"  Part="1"
+F 0 "#PWR0114" H 3550 3950 50  0001 C CNN
 F 1 "GND" H 3555 4027 50  0000 C CNN
 F 2 "" H 3550 4200 50  0001 C CNN
@@
 P 3400 4000
 AR Path="/5EA0F048" Ref="C?"  Part="1"
-AR Path="/5E9F954D/5EA0F048" Ref="C?"  Part="1"
-F 0 "C?" H 3515 4046 50  0000 L CNN
+AR Path="/5E9F954D/5EA0F048" Ref="C4"  Part="1"
+F 0 "C4" H 3515 4046 50  0000 L CNN
 F 1 "0.1uF" H 3515 3955 50  0000 L CNN
 F 2 "" H 3438 3850 50  0001 C CNN
@@
 P 3800 4000
 AR Path="/5EA0F042" Ref="C?"  Part="1"
-AR Path="/5E9F954D/5EA0F042" Ref="C?"  Part="1"
-F 0 "C?" H 3915 4046 50  0000 L CNN
+AR Path="/5E9F954D/5EA0F042" Ref="C5"  Part="1"
+F 0 "C5" H 3915 4046 50  0000 L CNN
 F 1 "0.1uF" H 3915 3955 50  0000 L CNN
 F 2 "" H 3838 3850 50  0001 C CNN
@@
 P 3100 5550
 AR Path="/5EA0F03C" Ref="U?"  Part="1"
-AR Path="/5E9F954D/5EA0F03C" Ref="U?"  Part="1"
-F 0 "U?" H 3100 4261 50  0000 C CNN
+AR Path="/5E9F954D/5EA0F03C" Ref="U2"  Part="1"
+F 0 "U2" H 3100 4261 50  0000 C CNN
 F 1 "Omega2+" H 3100 4170 50  0000 C CNN
 F 2 "Module:Onion_Omega2+" H 3100 4050 50  0001 C CNN
@@
 P 3100 6950
 AR Path="/5EA0EFAA" Ref="#PWR?"  Part="1"
-AR Path="/5E9F954D/5EA0EFAA" Ref="#PWR?"  Part="1"
-F 0 "#PWR?" H 3100 6700 50  0001 C CNN
+AR Path="/5E9F954D/5EA0EFAA" Ref="#PWR0115"  Part="1"
+F 0 "#PWR0115" H 3100 6700 50  0001 C CNN
 F 1 "GND" H 3105 6777 50  0000 C CNN
 F 2 "" H 3100 6950 50  0001 C CNN
@@
 P 8600 4800
 AR Path="/5E9DF408/5EA20F36" Ref="J?"  Part="1"
-AR Path="/5E9F954D/5EA20F36" Ref="J?"  Part="1"
-F 0 "J?" H 8071 4846 50  0000 R CNN
+AR Path="/5E9F954D/5EA20F36" Ref="J4"  Part="1"
+F 0 "J4" H 8071 4846 50  0000 R CNN
 F 1 "Conn_ARM_JTAG_SWD_20" H 8071 4755 50  0000 R CNN
 F 2 "" H 9050 3750 50  0001 L TNN
@@
 P 8600 3700
 AR Path="/5E9DF408/5EA20F4E" Ref="#PWR?"  Part="1"
-AR Path="/5E9F954D/5EA20F4E" Ref="#PWR?"  Part="1"
-F 0 "#PWR?" H 8600 3550 50  0001 C CNN
+AR Path="/5E9F954D/5EA20F4E" Ref="#PWR0116"  Part="1"
+F 0 "#PWR0116" H 8600 3550 50  0001 C CNN
 F 1 "+3.3V" H 8615 3873 50  0000 C CNN
 F 2 "" H 8600 3700 50  0001 C CNN
@@
 	9400 1450 9400 1600
 $Comp
-L power:+3.3V #PWR?
+L power:+3.3V #PWR0117
 U 1 1 5E9CA689
 P 9400 1450
-F 0 "#PWR?" H 9400 1300 50  0001 C CNN
+F 0 "#PWR0117" H 9400 1300 50  0001 C CNN
 F 1 "+3.3V" H 9415 1623 50  0000 C CNN
 F 2 "" H 9400 1450 50  0001 C CNN
@@
 P 8400 2100
 AR Path="/5EA12D94" Ref="#PWR?"  Part="1"
-AR Path="/5E9F954D/5EA12D94" Ref="#PWR?"  Part="1"
-F 0 "#PWR?" H 8400 1850 50  0001 C CNN
+AR Path="/5E9F954D/5EA12D94" Ref="#PWR0118"  Part="1"
+F 0 "#PWR0118" H 8400 1850 50  0001 C CNN
 F 1 "GND" H 8405 1927 50  0000 C CNN
 F 2 "" H 8400 2100 50  0001 C CNN
@@
 P 8400 1900
 AR Path="/5EA12D8E" Ref="SW?"  Part="1"
-AR Path="/5E9F954D/5EA12D8E" Ref="SW?"  Part="1"
-F 0 "SW?" V 8446 1852 50  0000 R CNN
+AR Path="/5E9F954D/5EA12D8E" Ref="SW1"  Part="1"
+F 0 "SW1" V 8446 1852 50  0000 R CNN
 F 1 "SW_Push" V 8355 1852 50  0000 R CNN
 F 2 "" H 8400 2100 50  0001 C CNN
@@
 P 8750 2000
 AR Path="/5EA12D86" Ref="#PWR?"  Part="1"
-AR Path="/5E9F954D/5EA12D86" Ref="#PWR?"  Part="1"
-F 0 "#PWR?" H 8750 1750 50  0001 C CNN
+AR Path="/5E9F954D/5EA12D86" Ref="#PWR0119"  Part="1"
+F 0 "#PWR0119" H 8750 1750 50  0001 C CNN
 F 1 "GND" H 8755 1827 50  0000 C CNN
 F 2 "" H 8750 2000 50  0001 C CNN
@@
 P 8750 1750
 AR Path="/5EA12D7C" Ref="C?"  Part="1"
-AR Path="/5E9F954D/5EA12D7C" Ref="C?"  Part="1"
-F 0 "C?" H 8865 1796 50  0000 L CNN
+AR Path="/5E9F954D/5EA12D7C" Ref="C6"  Part="1"
+F 0 "C6" H 8865 1796 50  0000 L CNN
 F 1 "0.1uF" H 8865 1705 50  0000 L CNN
 F 2 "" H 8788 1600 50  0001 C CNN
@@
 P 9100 1600
 AR Path="/5EA12D76" Ref="R?"  Part="1"
-AR Path="/5E9F954D/5EA12D76" Ref="R?"  Part="1"
-F 0 "R?" V 8893 1600 50  0000 C CNN
+AR Path="/5E9F954D/5EA12D76" Ref="R6"  Part="1"
+F 0 "R6" V 8893 1600 50  0000 C CNN
 F 1 "10k" V 8984 1600 50  0000 C CNN
 F 2 "" V 9030 1600 50  0001 C CNN

Commit message: Add files via upload
Parts:
- C2, C3, C4, C5, C6: footprint (none) -> Capacitor_SMD:C_0603_1608Metric_Pad1.05x0.95mm_HandSolder
- J3: footprint (none) -> Connector_USB:USB_A_Molex_105057_Vertical
- J4: footprint (none) -> Connector_PinSocket_1.27mm:PinSocket_2x10_P1.27mm_Vertical
- L1, L2, L3: footprint (none) -> Inductor_SMD:L_2010_5025Metric
- R4, R5, R6, R7: footprint (none) -> Resistor_SMD:R_0201_0603Metric
Changed lines of the file:
@@
 F 0 "J3" H 1957 2317 50  0000 C CNN
 F 1 "USB_A" H 1957 2226 50  0000 C CNN
-F 2 "" H 2050 1800 50  0001 C CNN
+F 2 "Connector_USB:USB_A_Molex_105057_Vertical" H 2050 1800 50  0001 C CNN
 F 3 " ~" H 2050 1800 50  0001 C CNN
 	1    1900 1850
@@
 F 0 "L1" V 3190 1950 50  0000 C CNN
 F 1 "L" V 3099 1950 50  0000 C CNN
-F 2 "" H 3000 1950 50  0001 C CNN
+F 2 "Inductor_SMD:L_2010_5025Metric" H 3000 1950 50  0001 C CNN
 F 3 "~" H 3000 1950 50  0001 C CNN
 	1    3000 1950
@@
 F 0 "L2" V 3290 1850 50  0000 C CNN
 F 1 "L" V 3199 1850 50  0000 C CNN
-F 2 "" H 3100 1850 50  0001 C CNN
+F 2 "Inductor_SMD:L_2010_5025Metric" H 3100 1850 50  0001 C CNN
 F 3 "~" H 3100 1850 50  0001 C CNN
 	1    3100 1850
@@
 F 0 "R5" V 3393 1850 50  0000 C CNN
 F 1 "R" V 3484 1850 50  0000 C CNN
-F 2 "" V 3530 1850 50  0001 C CNN
+F 2 "Resistor_SMD:R_0201_0603Metric" V 3530 1850 50  0001 C CNN
 F 3 "~" H 3600 1850 50  0001 C CNN
 	1    3600 1850
@@
 F 0 "R4" V 3243 1950 50  0000 C CNN
 F 1 "R" V 3334 1950 50  0000 C CNN
-F 2 "" V 3380 1950 50  0001 C CNN
+F 2 "Resistor_SMD:R_0201_0603Metric" V 3380 1950 50  0001 C CNN
 F 3 "~" H 3450 1950 50  0001 C CNN
 	1    3450 1950
@@
 F 0 "C2" H 3015 1246 50  0000 L CNN
 F 1 "C" H 3015 1155 50  0000 L CNN
-F 2 "" H 2938 1050 50  0001 C CNN
+F 2 "Capacitor_SMD:C_0603_1608Metric_Pad1.05x0.95mm_HandSolder" H 2938 1050 50  0001 C CNN
 F 3 "~" H 2900 1200 50  0001 C CNN
 	1    2900 1200
@@
 F 0 "C3" H 3365 1246 50  0000 L CNN
 F 1 "C" H 3365 1155 50  0000 L CNN
-F 2 "" H 3288 1050 50  0001 C CNN
+F 2 "Capacitor_SMD:C_0603_1608Metric_Pad1.05x0.95mm_HandSolder" H 3288 1050 50  0001 C CNN
 F 3 "~" H 3250 1200 50  0001 C CNN
 	1    3250 1200
@@
 F 0 "L3" V 3840 950 50  0000 C CNN
 F 1 "L" V 3749 950 50  0000 C CNN
-F 2 "" H 3650 950 50  0001 C CNN
+F 2 "Inductor_SMD:L_2010_5025Metric" H 3650 950 50  0001 C CNN
 F 3 "~" H 3650 950 50  0001 C CNN
 	1    3650 950
@@
 F 0 "R7" V 9793 4600 50  0001 C CNN
 F 1 "510" V 9885 4600 50  0000 C CNN
-F 2 "" V 9930 4600 50  0001 C CNN
+F 2 "Resistor_SMD:R_0201_0603Metric" V 9930 4600 50  0001 C CNN
 F 3 "~" H 10000 4600 50  0001 C CNN
 	1    10000 4600
@@
 F 0 "C4" H 3515 4046 50  0000 L CNN
 F 1 "0.1uF" H 3515 3955 50  0000 L CNN
-F 2 "" H 3438 3850 50  0001 C CNN
+F 2 "Capacitor_SMD:C_0603_1608Metric_Pad1.05x0.95mm_HandSolder" H 3438 3850 50  0001 C CNN
 F 3 "~" H 3400 4000 50  0001 C CNN
 	1    3400 4000
@@
 F 0 "C5" H 3915 4046 50  0000 L CNN
 F 1 "0.1uF" H 3915 3955 50  0000 L CNN
-F 2 "" H 3838 3850 50  0001 C CNN
+F 2 "Capacitor_SMD:C_0603_1608Metric_Pad1.05x0.95mm_HandSolder" H 3838 3850 50  0001 C CNN
 F 3 "~" H 3800 4000 50  0001 C CNN
 	1    3800 4000
@@
 F 0 "J4" H 8071 4846 50  0000 R CNN
 F 1 "Conn_ARM_JTAG_SWD_20" H 8071 4755 50  0000 R CNN
-F 2 "" H 9050 3750 50  0001 L TNN
+F 2 "Connector_PinSocket_1.27mm:PinSocket_2x10_P1.27mm_Vertical" H 9050 3750 50  0001 L TNN
 F 3 "http://infocenter.arm.com/help/topic/com.arm.doc.dui0499b/DUI0499B_system_design_reference.pdf" V 8250 3550 50  0001 C CNN
 	1    8600 4800
@@
 F 0 "C6" H 8865 1796 50  0000 L CNN
 F 1 "0.1uF" H 8865 1705 50  0000 L CNN
-F 2 "" H 8788 1600 50  0001 C CNN
+F 2 "Capacitor_SMD:C_0603_1608Metric_Pad1.05x0.95mm_HandSolder" H 8788 1600 50  0001 C CNN
 F 3 "~" H 8750 1750 50  0001 C CNN
 	1    8750 1750
@@
 F 0 "R6" V 8893 1600 50  0000 C CNN
 F 1 "10k" V 8984 1600 50  0000 C CNN
-F 2 "" V 9030 1600 50  0001 C CNN
+F 2 "Resistor_SMD:R_0201_0603Metric" V 9030 1600 50  0001 C CNN
 F 3 "~" H 9100 1600 50  0001 C CNN
 	1    9100 1600

Commit message: Add files via upload
Parts:
- added C43: 0.1uF, Capacitor_SMD:C_0603_1608Metric_Pad1.05x0.95mm_HandSolder, symbol Device:C
Connections:
- net GND: now also C43.2; no longer J3.5 (Shield)
- new net: C43.1, J3.5 (Shield)
Changed lines of the file:
@@
 	1    0    0    -1
 $EndComp
-Wire Wire Line
-	1900 2450 1900 2350
-Wire Wire Line
-	1800 2250 1800 2350
-Wire Wire Line
-	1800 2350 1900 2350
-Connection ~ 1900 2350
-Wire Wire Line
-	1900 2350 1900 2250
 $Comp
 L power:GND #PWR?
@@
 Text Notes 7000 3050 0    50   ~ 0
 RESET
+Wire Wire Line
+	1900 2250 1900 2450
+$Comp
+L Device:C C43
+U 1 1 5EB1B686
+P 1650 2550
+F 0 "C43" H 1450 2650 50  0000 L CNN
+F 1 "0.1uF" H 1400 2450 50  0000 L CNN
+F 2 "Capacitor_SMD:C_0603_1608Metric_Pad1.05x0.95mm_HandSolder" H 1688 2400 50  0001 C CNN
+F 3 "~" H 1650 2550 50  0001 C CNN
+	1    1650 2550
+	1    0    0    -1
+$EndComp
+$Comp
+L power:GND #PWR0170
+U 1 1 5EB1E40A
+P 1650 2800
+F 0 "#PWR0170" H 1650 2550 50  0001 C CNN
+F 1 "GND" H 1655 2627 50  0000 C CNN
+F 2 "" H 1650 2800 50  0001 C CNN
+F 3 "" H 1650 2800 50  0001 C CNN
+	1    1650 2800
+	1    0    0    -1
+$EndComp
+Wire Wire Line
+	1800 2250 1800 2350
+Wire Wire Line
+	1800 2350 1650 2350
+Wire Wire Line
+	1650 2350 1650 2400
+Wire Wire Line
+	1650 2700 1650 2800
 $EndSCHEMATC

Commit message: Add files via upload
Parts:
- SW1: footprint (none) -> Button_Switch_SMD:SW_DIP_SPSTx05_Slide_6.7x14.26mm_W6.73mm_P2.54mm_LowProfile_JPin
Changed lines of the file:
@@
 F 0 "SW1" V 8446 1852 50  0000 R CNN
 F 1 "SW_Push" V 8355 1852 50  0000 R CNN
-F 2 "" H 8400 2100 50  0001 C CNN
+F 2 "Button_Switch_SMD:SW_DIP_SPSTx05_Slide_6.7x14.26mm_W6.73mm_P2.54mm_LowProfile_JPin" H 8400 2100 50  0001 C CNN
 F 3 "~" H 8400 2100 50  0001 C CNN
 	1    8400 1900

Commit message: Add files via upload
Parts:
- SW1: footprint Button_Switch_SMD:SW_DIP_SPSTx05_Slide_6.7x14.26mm_W6.73mm_P2.54mm_LowProfile_JPin -> Button_Switch_SMD:SW_DIP_SPSTx01_Slide_6.7x4.1mm_W6.73mm_P2.54mm_LowProfile_JPin
Connections:
- net +3V3 renamed +3V8
Changed lines of the file:
@@
 Wire Wire Line
 	3800 3600 3800 3800
-$Comp
-L power:+3.3V #PWR0113
-U 1 1 5E9C8B2C
-P 3800 3600
-F 0 "#PWR0113" H 3800 3450 50  0001 C CNN
-F 1 "+3.3V" H 3815 3773 50  0000 C CNN
-F 2 "" H 3800 3600 50  0001 C CNN
-F 3 "" H 3800 3600 50  0001 C CNN
-	1    3800 3600
-	1    0    0    -1
-$EndComp
 Wire Wire Line
 	2400 5150 2200 5150
@@
 	1    0    0    -1
 $EndComp
-$Comp
-L power:+3.3V #PWR?
-U 1 1 5EA20F4E
-P 8600 3700
-AR Path="/5E9DF408/5EA20F4E" Ref="#PWR?"  Part="1"
-AR Path="/5E9F954D/5EA20F4E" Ref="#PWR0116"  Part="1"
-F 0 "#PWR0116" H 8600 3550 50  0001 C CNN
-F 1 "+3.3V" H 8615 3873 50  0000 C CNN
-F 2 "" H 8600 3700 50  0001 C CNN
-F 3 "" H 8600 3700 50  0001 C CNN
-	1    8600 3700
-	1    0    0    -1
-$EndComp
 Wire Wire Line
 	9400 1450 9400 1600
-$Comp
-L power:+3.3V #PWR0117
-U 1 1 5E9CA689
-P 9400 1450
-F 0 "#PWR0117" H 9400 1300 50  0001 C CNN
-F 1 "+3.3V" H 9415 1623 50  0000 C CNN
-F 2 "" H 9400 1450 50  0001 C CNN
-F 3 "" H 9400 1450 50  0001 C CNN
-	1    9400 1450
-	1    0    0    -1
-$EndComp
 Text Label 8150 1600 2    50   ~ 0
 RST_P
@@
 F 0 "SW1" V 8446 1852 50  0000 R CNN
 F 1 "SW_Push" V 8355 1852 50  0000 R CNN
-F 2 "Button_Switch_SMD:SW_DIP_SPSTx05_Slide_6.7x14.26mm_W6.73mm_P2.54mm_LowProfile_JPin" H 8400 2100 50  0001 C CNN
+F 2 "Button_Switch_SMD:SW_DIP_SPSTx01_Slide_6.7x4.1mm_W6.73mm_P2.54mm_LowProfile_JPin" H 8400 2100 50  0001 C CNN
 F 3 "~" H 8400 2100 50  0001 C CNN
 	1    8400 1900
@@
 Wire Wire Line
 	1650 2700 1650 2800
+$Comp
+L power:+3V8 #PWR0113
+U 1 1 5EB689CB
+P 9400 1450
+F 0 "#PWR0113" H 9400 1300 50  0001 C CNN
+F 1 "+3V8" H 9415 1623 50  0000 C CNN
+F 2 "" H 9400 1450 50  0001 C CNN
+F 3 "" H 9400 1450 50  0001 C CNN
+	1    9400 1450
+	1    0    0    -1
+$EndComp
+$Comp
+L power:+3V8 #PWR0116
+U 1 1 5EB6AB0F
+P 8600 3700
+F 0 "#PWR0116" H 8600 3550 50  0001 C CNN
+F 1 "+3V8" H 8615 3873 50  0000 C CNN
+F 2 "" H 8600 3700 50  0001 C CNN
+F 3 "" H 8600 3700 50  0001 C CNN
+	1    8600 3700
+	1    0    0    -1
+$EndComp
+$Comp
+L power:+3V8 #PWR0117
+U 1 1 5EB6AF97
+P 3800 3600
+F 0 "#PWR0117" H 3800 3450 50  0001 C CNN
+F 1 "+3V8" H 3815 3773 50  0000 C CNN
+F 2 "" H 3800 3600 50  0001 C CNN
+F 3 "" H 3800 3600 50  0001 C CNN
+	1    3800 3600
+	1    0    0    -1
+$EndComp
 $EndSCHEMATC
