File: proyecto/Puente H.sch (KiCad schematic (older format))
At the start: 3 parts

Commit message: Add files via upload
Parts:
- removed U?: L293D, Package_DIP:DIP-16_W7.62mm, symbol Driver_Motor:L293D
- added C?: C, symbol Device:C
- added R? (x3): 10K, symbol Device:R
- added U?: DRV8848, Package_SO:TSSOP-16-1EP_4.4x5mm_P0.65mm, symbol Driver_Motor:DRV8848
Connections:
- net labels added: +3.3V
- net labels removed: 3.3v, 5v, PH_EN34
- wire segments 24 -> 32
Changed lines of the file:
@@
 $Descr A4 11693 8268
 encoding utf-8
-Sheet 3 5
+Sheet 3 7
 Title ""
 Date ""
@@
 Comment4 ""
 $EndDescr
-$Comp
-L Driver_Motor:L293D U?
-U 1 1 5EA1B20C
-P 5400 3400
-AR Path="/5EA1B20C" Ref="U?"  Part="1"
-AR Path="/5EA16FA2/5EA1B20C" Ref="U?"  Part="1"
-F 0 "U?" H 5006 4581 50  0000 C CNN
-F 1 "L293D" H 5006 4490 50  0000 C CNN
-F 2 "Package_DIP:DIP-16_W7.62mm" H 5650 2650 50  0001 L CNN
-F 3 "http://www.ti.com/lit/ds/symlink/l293.pdf" H 5100 4100 50  0001 C CNN
-	1    5400 3400
-	1    0    0    -1
-$EndComp
-Wire Wire Line
-	6100 2800 5900 2800
-Wire Wire Line
-	6100 3000 5900 3000
-Wire Wire Line
-	5900 3400 6100 3400
-Wire Wire Line
-	6100 3600 5900 3600
-Connection ~ 5500 4400
-Wire Wire Line
-	5600 4400 5500 4400
-Wire Wire Line
-	5600 4200 5600 4400
-Connection ~ 5400 4400
-Wire Wire Line
-	5500 4400 5400 4400
-Wire Wire Line
-	5500 4200 5500 4400
-Wire Wire Line
-	5300 4400 5400 4400
-Connection ~ 5300 4400
-Wire Wire Line
-	5300 4200 5300 4400
-Wire Wire Line
-	5200 4400 5300 4400
-Wire Wire Line
-	5200 4200 5200 4400
-$Comp
-L power:GND #PWR?
-U 1 1 5EA1B221
-P 5400 4400
-AR Path="/5EA1B221" Ref="#PWR?"  Part="1"
-AR Path="/5EA16FA2/5EA1B221" Ref="#PWR?"  Part="1"
-F 0 "#PWR?" H 5400 4150 50  0001 C CNN
-F 1 "GND" H 5405 4227 50  0000 C CNN
-F 2 "" H 5400 4400 50  0001 C CNN
-F 3 "" H 5400 4400 50  0001 C CNN
-	1    5400 4400
-	1    0    0    -1
-$EndComp
-Text GLabel 6100 3600 2    50   Input ~ 0
-M2-
-Text GLabel 6100 3400 2    50   Input ~ 0
-M2+
-Text GLabel 6100 3000 2    50   Input ~ 0
-M1-
-Text GLabel 6100 2800 2    50   Input ~ 0
-M1+
-Wire Wire Line
-	4750 3800 4900 3800
-Wire Wire Line
-	4900 3600 4750 3600
-Wire Wire Line
-	4750 3400 4900 3400
-Wire Wire Line
-	4900 3200 4750 3200
-Wire Wire Line
-	4750 3000 4900 3000
-Wire Wire Line
-	4900 2800 4750 2800
 $Comp
 L Connector_Generic:Conn_01x02 J?
@@
 	1    0    0    -1
 $EndComp
-Text GLabel 6900 2850 0    50   Input ~ 0
-M1+
-Text GLabel 6900 2950 0    50   Input ~ 0
-M1-
 Wire Wire Line
 	7050 2850 6900 2850
@@
 	1    0    0    -1
 $EndComp
-Text GLabel 6900 3350 0    50   Input ~ 0
+Wire Wire Line
+	7050 3350 6900 3350
+Wire Wire Line
+	6900 3450 7050 3450
+Text Label 6900 2850 0    50   ~ 0
+M1+
+Text Label 6900 2950 0    50   ~ 0
+M1-
+Text Label 6900 3350 0    50   ~ 0
 M2+
-Text GLabel 6900 3450 0    50   Input ~ 0
+Text Label 6900 3450 0    50   ~ 0
 M2-
-Wire Wire Line
-	7050 3350 6900 3350
-Wire Wire Line
-	6900 3450 7050 3450
-Text HLabel 4750 2800 0    50   Input ~ 0
+$Comp
+L Driver_Motor:DRV8848 U?
+U 1 1 5E9F03B2
+P 4200 3550
+F 0 "U?" H 4200 4331 50  0000 C CNN
+F 1 "DRV8848" H 4200 4240 50  0000 C CNN
+F 2 "Package_SO:TSSOP-16-1EP_4.4x5mm_P0.65mm" H 4200 2850 50  0001 C CNN
+F 3 "http://www.ti.com/lit/ds/symlink/drv8848.pdf" H 3050 4900 50  0001 C CNN
+	1    4200 3550
+	1    0    0    -1
+$EndComp
+Text Label 5100 3350 2    50   ~ 0
+M1+
+Text Label 5100 3750 2    50   ~ 0
+M2+
+$Comp
+L power:GND #PWR?
+U 1 1 5E9F40C3
+P 5550 3550
+F 0 "#PWR?" H 5550 3300 50  0001 C CNN
+F 1 "GND" V 5555 3422 50  0000 R CNN
+F 2 "" H 5550 3550 50  0001 C CNN
+F 3 "" H 5550 3550 50  0001 C CNN
+	1    5550 3550
+	0    -1   -1   0
+$EndComp
+Wire Wire Line
+	3350 3350 3600 3350
+Wire Wire Line
+	3600 3550 3350 3550
+Wire Wire Line
+	3600 3650 3350 3650
+Wire Wire Line
+	3350 3850 3600 3850
+Wire Wire Line
+	3600 3950 3350 3950
+Wire Wire Line
+	5100 3350 4800 3350
+Wire Wire Line
+	4800 3750 5100 3750
+$Comp
+L power:GND #PWR?
+U 1 1 5E9FC71B
+P 4200 4400
+F 0 "#PWR?" H 4200 4150 50  0001 C CNN
+F 1 "GND" H 4205 4227 50  0000 C CNN
+F 2 "" H 4200 4400 50  0001 C CNN
+F 3 "" H 4200 4400 50  0001 C CNN
+	1    4200 4400
+	1    0    0    -1
+$EndComp
+Wire Wire Line
+	4200 4150 4200 4300
+Wire Wire Line
+	5100 3850 4800 3850
+$Comp
+L power:GND #PWR?
+U 1 1 5E9F49EA
+P 5550 3950
+F 0 "#PWR?" H 5550 3700 50  0001 C CNN
+F 1 "GND" V 5555 3822 50  0000 R CNN
+F 2 "" H 5550 3950 50  0001 C CNN
+F 3 "" H 5550 3950 50  0001 C CNN
+	1    5550 3950
+	0    -1   -1   0
+$EndComp
+Text Label 5100 3850 2    50   ~ 0
+M2-
+$Comp
+L Device:R R?
+U 1 1 5E9FF7D6
+P 5300 3550
+F 0 "R?" V 5093 3550 50  0000 C CNN
+F 1 "10K" V 5184 3550 50  0000 C CNN
+F 2 "" V 5230 3550 50  0001 C CNN
+F 3 "~" H 5300 3550 50  0001 C CNN
+	1    5300 3550
+	0    1    1    0
+$EndComp
+Wire Wire Line
+	4800 3450 5100 3450
+Text Label 5100 3450 2    50   ~ 0
+M1-
+$Comp
+L Device:R R?
+U 1 1 5EA01869
+P 5300 3950
+F 0 "R?" V 5093 3950 50  0000 C CNN
+F 1 "10K" V 5184 3950 50  0000 C CNN
+F 2 "" V 5230 3950 50  0001 C CNN
+F 3 "~" H 5300 3950 50  0001 C CNN
+	1    5300 3950
+	0    1    1    0
+$EndComp
+Wire Wire Line
+	5550 3550 5450 3550
+Wire Wire Line
+	5150 3550 4800 3550
+Wire Wire Line
+	5150 3950 4800 3950
+Wire Wire Line
+	5550 3950 5450 3950
+$Comp
+L Device:R R?
+U 1 1 5EA175D5
+P 2200 3400
+F 0 "R?" H 2270 3446 50  0000 L CNN
+F 1 "10K" H 2270 3355 50  0000 L CNN
+F 2 "" V 2130 3400 50  0001 C CNN
+F 3 "~" H 2200 3400 50  0001 C CNN
+	1    2200 3400
+	1    0    0    -1
+$EndComp
+$Comp
+L power:+3.3V #PWR?
+U 1 1 5EA12F42
+P 2200 2950
+F 0 "#PWR?" H 2200 2800 50  0001 C CNN
+F 1 "+3.3V" H 2215 3123 50  0000 C CNN
+F 2 "" H 2200 2950 50  0001 C CNN
+F 3 "" H 2200 2950 50  0001 C CNN
+	1    2200 2950
+	1    0    0    -1
+$EndComp
+$Comp
+L power:GND #PWR?
+U 1 1 5EA0F0CB
+P 2200 4150
+F 0 "#PWR?" H 2200 3900 50  0001 C CNN
+F 1 "GND" H 2205 3977 50  0000 C CNN
+F 2 "" H 2200 4150 50  0001 C CNN
+F 3 "" H 2200 4150 50  0001 C CNN
+	1    2200 4150
+	1    0    0    -1
+$EndComp
+$Comp
+L Device:C C?
+U 1 1 5EA0E86B
+P 2200 3850
+F 0 "C?" H 2315 3896 50  0000 L CNN
+F 1 "C" H 2315 3805 50  0000 L CNN
+F 2 "" H 2238 3700 50  0001 C CNN
+F 3 "~" H 2200 3850 50  0001 C CNN
+	1    2200 3850
+	1    0    0    -1
+$EndComp
+Text HLabel 3350 3350 0    50   Input ~ 0
+PH_EN12
+Text HLabel 3350 3950 0    50   Input ~ 0
+PH_4A
+Text HLabel 3350 3850 0    50   Input ~ 0
+PH_3A
+Text HLabel 3350 3650 0    50   Input ~ 0
+PH_2A
+Text HLabel 3350 3550 0    50   Input ~ 0
 PH_1A
-Text HLabel 4750 3000 0    50   Input ~ 0
-PH_2A
-Text HLabel 4750 3200 0    50   Input ~ 0
-PH_EN12
-Text HLabel 4750 3400 0    50   Input ~ 0
-PH_3A
-Text HLabel 4750 3600 0    50   Input ~ 0
-PH_4A
-Text HLabel 4750 3800 0    50   Input ~ 0
-PH_EN34
-Text HLabel 5300 2250 1    50   Input ~ 0
-3.3v
-Text HLabel 5500 2250 1    50   Input ~ 0
-5v
-Wire Wire Line
-	5500 2250 5500 2400
-Wire Wire Line
-	5300 2400 5300 2250
+Wire Wire Line
+	2200 4150 2200 4000
+Wire Wire Line
+	2200 3700 2200 3650
+Wire Wire Line
+	2200 2950 2200 3150
+Wire Wire Line
+	3600 3150 2200 3150
+Connection ~ 2200 3150
+Wire Wire Line
+	2200 3150 2200 3250
+Wire Wire Line
+	3600 3250 2700 3250
+Wire Wire Line
+	2700 3250 2700 3650
+Wire Wire Line
+	2700 3650 2200 3650
+Connection ~ 2200 3650
+Wire Wire Line
+	2200 3650 2200 3550
+$Comp
+L power:+3.3V #PWR?
+U 1 1 5EA2378A
+P 5250 2900
+F 0 "#PWR?" H 5250 2750 50  0001 C CNN
+F 1 "+3.3V" H 5265 3073 50  0000 C CNN
+F 2 "" H 5250 2900 50  0001 C CNN
+F 3 "" H 5250 2900 50  0001 C CNN
+	1    5250 2900
+	1    0    0    -1
+$EndComp
+Wire Wire Line
+	4800 3150 5250 3150
+Wire Wire Line
+	5250 3150 5250 2900
+Wire Wire Line
+	4300 4150 4300 4300
+Wire Wire Line
+	4300 4300 4200 4300
+Connection ~ 4200 4300
+Wire Wire Line
+	4200 4300 4200 4400
 $EndSCHEMATC

Commit message: Add files via upload
Connections:
- net +3V3 renamed +5V
Changed lines of the file:
@@
-$EndComp
-$Comp
-L power:+3.3V #PWR?
-U 1 1 5EA12F42
-P 2200 2950
-F 0 "#PWR?" H 2200 2800 50  0001 C CNN
-F 1 "+3.3V" H 2215 3123 50  0000 C CNN
-F 2 "" H 2200 2950 50  0001 C CNN
-F 3 "" H 2200 2950 50  0001 C CNN
-	1    2200 2950
-	1    0    0    -1
 $EndComp
 $Comp
@@
 	2200 3700 2200 3650
 Wire Wire Line
-	2200 2950 2200 3150
-Wire Wire Line
 	3600 3150 2200 3150
 Connection ~ 2200 3150
@@
 Wire Wire Line
 	2200 3650 2200 3550
-$Comp
-L power:+3.3V #PWR?
-U 1 1 5EA2378A
-P 5250 2900
-F 0 "#PWR?" H 5250 2750 50  0001 C CNN
-F 1 "+3.3V" H 5265 3073 50  0000 C CNN
-F 2 "" H 5250 2900 50  0001 C CNN
-F 3 "" H 5250 2900 50  0001 C CNN
-	1    5250 2900
-	1    0    0    -1
-$EndComp
 Wire Wire Line
 	4800 3150 5250 3150
-Wire Wire Line
-	5250 3150 5250 2900
 Wire Wire Line
 	4300 4150 4300 4300
@@
 Wire Wire Line
 	4200 4300 4200 4400
+$Comp
+L power:+5V #PWR?
+U 1 1 5E9F1326
+P 2200 2800
+F 0 "#PWR?" H 2200 2650 50  0001 C CNN
+F 1 "+5V" H 2215 2973 50  0000 C CNN
+F 2 "" H 2200 2800 50  0001 C CNN
+F 3 "" H 2200 2800 50  0001 C CNN
+	1    2200 2800
+	1    0    0    -1
+$EndComp
+$Comp
+L power:+5V #PWR?
+U 1 1 5E9F1ADD
+P 5250 2850
+F 0 "#PWR?" H 5250 2700 50  0001 C CNN
+F 1 "+5V" H 5265 3023 50  0000 C CNN
+F 2 "" H 5250 2850 50  0001 C CNN
+F 3 "" H 5250 2850 50  0001 C CNN
+	1    5250 2850
+	1    0    0    -1
+$EndComp
+Wire Wire Line
+	5250 2850 5250 3150
+Wire Wire Line
+	2200 2800 2200 3150
 $EndSCHEMATC

Commit message: Add files via upload
Connections:
- net +5V: no longer R?.1, U?.11 (VREF)
- new net +3V3: R?.1, U?.11 (VREF)
Other:
- moved on the sheet: C?, J?, R?, U?

Commit message: Add files via upload
Other:
- note added: "CONECTORES MOTORES"
- note added: "PUENTE H"
- moved on the sheet: C?, J?, R?, U?

Commit message: Add files via upload
Parts:
- removed J?: M1, symbol Connector_Generic:Conn_01x02
- removed J?: M2, symbol Connector_Generic:Conn_01x02
- added J1, J2: Conn_01x03, symbol Connector_Generic:Conn_01x03
- gave numbers to parts that had none: 5
Connections:
- net +5V: now also J1.1 (Pin_1), J2.1 (Pin_1)
- net M1+: now also J1.2 (Pin_2)
- net M1-: now also J1.3 (Pin_3)
- net M2+: now also J2.2 (Pin_2)
- net M2-: now also J2.3 (Pin_3)
Changed lines of the file:
@@
 Comment4 ""
 $EndDescr
-$Comp
-L Connector_Generic:Conn_01x02 J?
-U 1 1 5EA1B237
-P 8850 2950
-AR Path="/5EA1B237" Ref="J?"  Part="1"
-AR Path="/5EA16FA2/5EA1B237" Ref="J?"  Part="1"
-F 0 "J?" H 8930 2942 50  0000 L CNN
-F 1 "M1" H 8930 2851 50  0000 L CNN
-F 2 "" H 8850 2950 50  0001 C CNN
-F 3 "~" H 8850 2950 50  0001 C CNN
-	1    8850 2950
-	1    0    0    -1
-$EndComp
-Wire Wire Line
-	8650 2950 8500 2950
-Wire Wire Line
-	8500 3050 8650 3050
-$Comp
-L Connector_Generic:Conn_01x02 J?
-U 1 1 5EA1B241
-P 8850 3650
-AR Path="/5EA1B241" Ref="J?"  Part="1"
-AR Path="/5EA16FA2/5EA1B241" Ref="J?"  Part="1"
-F 0 "J?" H 8930 3642 50  0000 L CNN
-F 1 "M2" H 8930 3551 50  0000 L CNN
-F 2 "" H 8850 3650 50  0001 C CNN
-F 3 "~" H 8850 3650 50  0001 C CNN
-	1    8850 3650
-	1    0    0    -1
-$EndComp
-Wire Wire Line
-	8650 3650 8500 3650
-Wire Wire Line
-	8500 3750 8650 3750
-Text Label 8500 2950 0    50   ~ 0
+Wire Wire Line
+	9350 3000 9200 3000
+Wire Wire Line
+	9200 3100 9350 3100
+Wire Wire Line
+	9350 3700 9200 3700
+Wire Wire Line
+	9200 3800 9350 3800
+Text Label 9200 3000 0    50   ~ 0
 M1+
-Text Label 8500 3050 0    50   ~ 0
+Text Label 9200 3100 0    50   ~ 0
 M1-
-Text Label 8500 3650 0    50   ~ 0
+Text Label 9200 3700 0    50   ~ 0
 M2+
-Text Label 8500 3750 0    50   ~ 0
+Text Label 9200 3800 0    50   ~ 0
 M2-
 $Comp
-L Driver_Motor:DRV8848 U?
+L Driver_Motor:DRV8848 U1
 U 1 1 5E9F03B2
 P 4250 3850
-F 0 "U?" H 4250 4631 50  0000 C CNN
+F 0 "U1" H 4250 4631 50  0000 C CNN
 F 1 "DRV8848" H 4250 4540 50  0000 C CNN
 F 2 "Package_SO:TSSOP-16-1EP_4.4x5mm_P0.65mm" H 4250 3150 50  0001 C CNN
@@
 M2+
 $Comp
-L power:GND #PWR?
+L power:GND #PWR0101
 U 1 1 5E9F40C3
 P 5600 3850
-F 0 "#PWR?" H 5600 3600 50  0001 C CNN
+F 0 "#PWR0101" H 5600 3600 50  0001 C CNN
 F 1 "GND" V 5605 3722 50  0000 R CNN
 F 2 "" H 5600 3850 50  0001 C CNN
@@
 	4850 4050 5150 4050
 $Comp
-L power:GND #PWR?
+L power:GND #PWR0102
 U 1 1 5E9FC71B
 P 4250 4700
-F 0 "#PWR?" H 4250 4450 50  0001 C CNN
+F 0 "#PWR0102" H 4250 4450 50  0001 C CNN
 F 1 "GND" H 4255 4527 50  0000 C CNN
 F 2 "" H 4250 4700 50  0001 C CNN
@@
 	5150 4150 4850 4150
 $Comp
-L power:GND #PWR?
+L power:GND #PWR0103
 U 1 1 5E9F49EA
 P 5600 4250
-F 0 "#PWR?" H 5600 4000 50  0001 C CNN
+F 0 "#PWR0103" H 5600 4000 50  0001 C CNN
 F 1 "GND" V 5605 4122 50  0000 R CNN
 F 2 "" H 5600 4250 50  0001 C CNN
@@
 M2-
 $Comp
-L Device:R R?
+L Device:R R2
 U 1 1 5E9FF7D6
 P 5350 3850
-F 0 "R?" V 5143 3850 50  0000 C CNN
+F 0 "R2" V 5143 3850 50  0000 C CNN
 F 1 "10K" V 5234 3850 50  0000 C CNN
 F 2 "" V 5280 3850 50  0001 C CNN
@@
 M1-
 $Comp
-L Device:R R?
+L Device:R R3
 U 1 1 5EA01869
 P 5350 4250
-F 0 "R?" V 5143 4250 50  0000 C CNN
+F 0 "R3" V 5143 4250 50  0000 C CNN
 F 1 "10K" V 5234 4250 50  0000 C CNN
 F 2 "" V 5280 4250 50  0001 C CNN
@@
 	5600 4250 5500 4250
 $Comp
-L Device:R R?
+L Device:R R1
 U 1 1 5EA175D5
 P 2250 3700
-F 0 "R?" H 2320 3746 50  0000 L CNN
+F 0 "R1" H 2320 3746 50  0000 L CNN
 F 1 "10K" H 2320 3655 50  0000 L CNN
 F 2 "" V 2180 3700 50  0001 C CNN
@@
 $EndComp
 $Comp
-L power:GND #PWR?
+L power:GND #PWR0104
 U 1 1 5EA0F0CB
 P 2250 4450
-F 0 "#PWR?" H 2250 4200 50  0001 C CNN
+F 0 "#PWR0104" H 2250 4200 50  0001 C CNN
 F 1 "GND" H 2255 4277 50  0000 C CNN
 F 2 "" H 2250 4450 50  0001 C CNN
@@
 $EndComp
 $Comp
-L Device:C C?
+L Device:C C1
 U 1 1 5EA0E86B
 P 2250 4150
-F 0 "C?" H 2365 4196 50  0000 L CNN
+F 0 "C1" H 2365 4196 50  0000 L CNN
 F 1 "C" H 2365 4105 50  0000 L CNN
 F 2 "" H 2288 4000 50  0001 C CNN
@@
 	4250 4600 4250 4700
 $Comp
-L power:+3.3V #PWR?
+L power:+3.3V #PWR0105
 U 1 1 5E9FAB94
 P 2250 3200
-F 0 "#PWR?" H 2250 3050 50  0001 C CNN
+F 0 "#PWR0105" H 2250 3050 50  0001 C CNN
 F 1 "+3.3V" H 2265 3373 50  0000 C CNN
 F 2 "" H 2250 3200 50  0001 C CNN
@@
 Connection ~ 2250 3450
 $Comp
-L power:+5V #PWR?
+L power:+5V #PWR0106
 U 1 1 5E9FCF22
 P 5300 3200
-F 0 "#PWR?" H 5300 3050 50  0001 C CNN
+F 0 "#PWR0106" H 5300 3050 50  0001 C CNN
 F 1 "+5V" H 5315 3373 50  0000 C CNN
 F 2 "" H 5300 3200 50  0001 C CNN
@@
 Text Notes 500  7750 0    50   ~ 0
 PUENTE H
+$Comp
+L Connector_Generic:Conn_01x03 J1
+U 1 1 5EBA02CF
+P 9550 3000
+F 0 "J1" H 9630 3042 50  0000 L CNN
+F 1 "Conn_01x03" H 9630 2951 50  0000 L CNN
+F 2 "" H 9550 3000 50  0001 C CNN
+F 3 "~" H 9550 3000 50  0001 C CNN
+	1    9550 3000
+	1    0    0    -1
+$EndComp
+$Comp
+L Connector_Generic:Conn_01x03 J2
+U 1 1 5EBA0E92
+P 9550 3700
+F 0 "J2" H 9630 3742 50  0000 L CNN
+F 1 "Conn_01x03" H 9630 3651 50  0000 L CNN
+F 2 "" H 9550 3700 50  0001 C CNN
+F 3 "~" H 9550 3700 50  0001 C CNN
+	1    9550 3700
+	1    0    0    -1
+$EndComp
+$Comp
+L power:+5V #PWR?
+U 1 1 5EBA2E7B
+P 9050 3600
+F 0 "#PWR?" H 9050 3450 50  0001 C CNN
+F 1 "+5V" V 9065 3728 50  0000 L CNN
+F 2 "" H 9050 3600 50  0001 C CNN
+F 3 "" H 9050 3600 50  0001 C CNN
+	1    9050 3600
+	0    -1   -1   0
+$EndComp
+Wire Wire Line
+	9050 3600 9350 3600
+$Comp
+L power:+5V #PWR?
+U 1 1 5EBA4FE6
+P 9050 2900
+F 0 "#PWR?" H 9050 2750 50  0001 C CNN
+F 1 "+5V" V 9065 3028 50  0000 L CNN
+F 2 "" H 9050 2900 50  0001 C CNN
+F 3 "" H 9050 2900 50  0001 C CNN
+	1    9050 2900
+	0    -1   -1   0
+$EndComp
+Wire Wire Line
+	9350 2900 9050 2900
 $EndSCHEMATC

Commit message: Add files via upload
Parts:
- C1: footprint (none) -> Capacitor_SMD:C_0603_1608Metric_Pad1.05x0.95mm_HandSolder
- J1, J2: footprint (none) -> Connector_JST:JST_EH_B3B-EH-A_1x03_P2.50mm_Vertical
- R1, R2, R3: footprint (none) -> Resistor_SMD:R_0201_0603Metric
Changed lines of the file:
@@
 F 0 "R2" V 5143 3850 50  0000 C CNN
 F 1 "10K" V 5234 3850 50  0000 C CNN
-F 2 "" V 5280 3850 50  0001 C CNN
+F 2 "Resistor_SMD:R_0201_0603Metric" V 5280 3850 50  0001 C CNN
 F 3 "~" H 5350 3850 50  0001 C CNN
 	1    5350 3850
@@
 F 0 "R3" V 5143 4250 50  0000 C CNN
 F 1 "10K" V 5234 4250 50  0000 C CNN
-F 2 "" V 5280 4250 50  0001 C CNN
+F 2 "Resistor_SMD:R_0201_0603Metric" V 5280 4250 50  0001 C CNN
 F 3 "~" H 5350 4250 50  0001 C CNN
 	1    5350 4250
@@
 F 0 "R1" H 2320 3746 50  0000 L CNN
 F 1 "10K" H 2320 3655 50  0000 L CNN
-F 2 "" V 2180 3700 50  0001 C CNN
+F 2 "Resistor_SMD:R_0201_0603Metric" V 2180 3700 50  0001 C CNN
 F 3 "~" H 2250 3700 50  0001 C CNN
 	1    2250 3700
@@
 F 0 "C1" H 2365 4196 50  0000 L CNN
 F 1 "C" H 2365 4105 50  0000 L CNN
-F 2 "" H 2288 4000 50  0001 C CNN
+F 2 "Capacitor_SMD:C_0603_1608Metric_Pad1.05x0.95mm_HandSolder" H 2288 4000 50  0001 C CNN
 F 3 "~" H 2250 4150 50  0001 C CNN
 	1    2250 4150
@@
 F 0 "J1" H 9630 3042 50  0000 L CNN
 F 1 "Conn_01x03" H 9630 2951 50  0000 L CNN
-F 2 "" H 9550 3000 50  0001 C CNN
+F 2 "Connector_JST:JST_EH_B3B-EH-A_1x03_P2.50mm_Vertical" H 9550 3000 50  0001 C CNN
 F 3 "~" H 9550 3000 50  0001 C CNN
 	1    9550 3000
@@
 F 0 "J2" H 9630 3742 50  0000 L CNN
 F 1 "Conn_01x03" H 9630 3651 50  0000 L CNN
-F 2 "" H 9550 3700 50  0001 C CNN
+F 2 "Connector_JST:JST_EH_B3B-EH-A_1x03_P2.50mm_Vertical" H 9550 3700 50  0001 C CNN
 F 3 "~" H 9550 3700 50  0001 C CNN
 	1    9550 3700
@@
 $EndComp
 $Comp
-L power:+5V #PWR?
+L power:+5V #PWR0122
 U 1 1 5EBA2E7B
 P 9050 3600
-F 0 "#PWR?" H 9050 3450 50  0001 C CNN
+F 0 "#PWR0122" H 9050 3450 50  0001 C CNN
 F 1 "+5V" V 9065 3728 50  0000 L CNN
 F 2 "" H 9050 3600 50  0001 C CNN
@@
 	9050 3600 9350 3600
 $Comp
-L power:+5V #PWR?
+L power:+5V #PWR0128
 U 1 1 5EBA4FE6
 P 9050 2900
-F 0 "#PWR?" H 9050 2750 50  0001 C CNN
+F 0 "#PWR0128" H 9050 2750 50  0001 C CNN
 F 1 "+5V" V 9065 3028 50  0000 L CNN
 F 2 "" H 9050 2900 50  0001 C CNN

Commit message: Add files via upload
Connections:
- net +3V3 renamed +3V8
Changed lines of the file:
@@
 Wire Wire Line
 	4250 4600 4250 4700
-$Comp
-L power:+3.3V #PWR0105
-U 1 1 5E9FAB94
-P 2250 3200
-F 0 "#PWR0105" H 2250 3050 50  0001 C CNN
-F 1 "+3.3V" H 2265 3373 50  0000 C CNN
-F 2 "" H 2250 3200 50  0001 C CNN
-F 3 "" H 2250 3200 50  0001 C CNN
-	1    2250 3200
-	1    0    0    -1
-$EndComp
 Wire Wire Line
 	2250 3200 2250 3450
@@
 Wire Wire Line
 	9350 2900 9050 2900
+$Comp
+L power:+3V8 #PWR0105
+U 1 1 5EB6C7F3
+P 2250 3200
+F 0 "#PWR0105" H 2250 3050 50  0001 C CNN
+F 1 "+3V8" H 2265 3373 50  0000 C CNN
+F 2 "" H 2250 3200 50  0001 C CNN
+F 3 "" H 2250 3200 50  0001 C CNN
+	1    2250 3200
+	1    0    0    -1
+$EndComp
 $EndSCHEMATC
