File: proyecto/Puente H.sch (KiCad schematic (older format))
At the start: 7 parts, among them J1 Conn_01x03, J2 Conn_01x03, U1 DRV8848

Commit message: Add files via upload
Parts:
- J1, J2: footprint Connector_JST:JST_EH_B3B-EH-A_1x03_P2.50mm_Vertical -> Connector_PinHeader_1.00mm:PinHeader_1x03_P1.00mm_Horizontal
- R1, R2, R3: footprint Resistor_SMD:R_0201_0603Metric -> Resistor_SMD:R_0603_1608Metric_Pad1.05x0.95mm_HandSolder
Changed lines of the file:
@@
 F 0 "R2" V 5143 3850 50  0000 C CNN
 F 1 "10K" V 5234 3850 50  0000 C CNN
-F 2 "Resistor_SMD:R_0201_0603Metric" V 5280 3850 50  0001 C CNN
+F 2 "Resistor_SMD:R_0603_1608Metric_Pad1.05x0.95mm_HandSolder" V 5280 3850 50  0001 C CNN
 F 3 "~" H 5350 3850 50  0001 C CNN
 	1    5350 3850
@@
 F 0 "R3" V 5143 4250 50  0000 C CNN
 F 1 "10K" V 5234 4250 50  0000 C CNN
-F 2 "Resistor_SMD:R_0201_0603Metric" V 5280 4250 50  0001 C CNN
+F 2 "Resistor_SMD:R_0603_1608Metric_Pad1.05x0.95mm_HandSolder" V 5280 4250 50  0001 C CNN
 F 3 "~" H 5350 4250 50  0001 C CNN
 	1    5350 4250
@@
 F 0 "R1" H 2320 3746 50  0000 L CNN
 F 1 "10K" H 2320 3655 50  0000 L CNN
-F 2 "Resistor_SMD:R_0201_0603Metric" V 2180 3700 50  0001 C CNN
+F 2 "Resistor_SMD:R_0603_1608Metric_Pad1.05x0.95mm_HandSolder" V 2180 3700 50  0001 C CNN
 F 3 "~" H 2250 3700 50  0001 C CNN
 	1    2250 3700
@@
 F 0 "J1" H 9630 3042 50  0000 L CNN
 F 1 "Conn_01x03" H 9630 2951 50  0000 L CNN
-F 2 "Connector_JST:JST_EH_B3B-EH-A_1x03_P2.50mm_Vertical" H 9550 3000 50  0001 C CNN
+F 2 "Connector_PinHeader_1.00mm:PinHeader_1x03_P1.00mm_Horizontal" H 9550 3000 50  0001 C CNN
 F 3 "~" H 9550 3000 50  0001 C CNN
 	1    9550 3000
@@
 F 0 "J2" H 9630 3742 50  0000 L CNN
 F 1 "Conn_01x03" H 9630 3651 50  0000 L CNN
-F 2 "Connector_JST:JST_EH_B3B-EH-A_1x03_P2.50mm_Vertical" H 9550 3700 50  0001 C CNN
+F 2 "Connector_PinHeader_1.00mm:PinHeader_1x03_P1.00mm_Horizontal" H 9550 3700 50  0001 C CNN
 F 3 "~" H 9550 3700 50  0001 C CNN
 	1    9550 3700
