File: proyecto/camara.sch (KiCad schematic (older format))
At the start: 16 parts

Commit message: Add files via upload
Parts:
- added J?: Conn_ARM_JTAG_SWD_20, symbol Connector:Conn_ARM_JTAG_SWD_20
- added R?: 510, symbol Device:R
Connections:
- net labels added: +3V3, +5VD, GNDA, SRST3, TCK3, TD03, TD13, TMS3, TRST3
- net labels removed: +3.3V, +5V
- wire segments 53 -> 72
Other:
- moved on the sheet: C?, D?, J?, L?, R?, SW?, U?

Commit message: Add files via upload
Other:
- note added: "JTAG"
- note added: "PROCESADOR"
- note added: "RESET"
- note added: "USB"
- moved on the sheet: C?, D?, J?, L?, R?, SW?, U?

Commit message: Add files via upload
Parts:
- gave numbers to parts that had none: 18
Changed lines of the file:
@@
 AR Path="/5EA368A5" Ref="R?"  Part="1"
 AR Path="/5E9F954D/5EA368A5" Ref="R?"  Part="1"
-AR Path="/5E9DF2DA/5EA368A5" Ref="R?"  Part="1"
-F 0 "R?" V 8993 5100 50  0000 C CNN
+AR Path="/5E9DF2DA/5EA368A5" Ref="R14"  Part="1"
+F 0 "R14" V 8993 5100 50  0000 C CNN
 F 1 "10k" V 9084 5100 50  0000 C CNN
 F 2 "" V 9130 5100 50  0001 C CNN
@@
 AR Path="/5EA368AB" Ref="C?"  Part="1"
 AR Path="/5E9F954D/5EA368AB" Ref="C?"  Part="1"
-AR Path="/5E9DF2DA/5EA368AB" Ref="C?"  Part="1"
-F 0 "C?" H 8965 5296 50  0000 L CNN
+AR Path="/5E9DF2DA/5EA368AB" Ref="C19"  Part="1"
+F 0 "C19" H 8965 5296 50  0000 L CNN
 F 1 "0.1uF" H 8965 5205 50  0000 L CNN
 F 2 "" H 8888 5100 50  0001 C CNN
@@
 AR Path="/5EA368BC" Ref="SW?"  Part="1"
 AR Path="/5E9F954D/5EA368BC" Ref="SW?"  Part="1"
-AR Path="/5E9DF2DA/5EA368BC" Ref="SW?"  Part="1"
-F 0 "SW?" V 8546 5352 50  0000 R CNN
+AR Path="/5E9DF2DA/5EA368BC" Ref="SW2"  Part="1"
+F 0 "SW2" V 8546 5352 50  0000 R CNN
 F 1 "SW_Push" V 8455 5352 50  0000 R CNN
 F 2 "" H 8500 5600 50  0001 C CNN
@@
 AR Path="/5EA3ADB9" Ref="D?"  Part="1"
 AR Path="/5E9F954D/5EA3ADB9" Ref="D?"  Part="1"
-AR Path="/5E9DF2DA/5EA3ADB9" Ref="D?"  Part="1"
-F 0 "D?" H 3105 2496 50  0000 L CNN
+AR Path="/5E9DF2DA/5EA3ADB9" Ref="D5"  Part="1"
+F 0 "D5" H 3105 2496 50  0000 L CNN
 F 1 "SP0502BAHT" H 3105 2405 50  0000 L CNN
 F 2 "Package_TO_SOT_SMD:SOT-23" H 3125 2400 50  0001 L CNN
@@
 AR Path="/5EA3ADBF" Ref="J?"  Part="1"
 AR Path="/5E9F954D/5EA3ADBF" Ref="J?"  Part="1"
-AR Path="/5E9DF2DA/5EA3ADBF" Ref="J?"  Part="1"
-F 0 "J?" H 2207 2517 50  0000 C CNN
+AR Path="/5E9DF2DA/5EA3ADBF" Ref="J6"  Part="1"
+F 0 "J6" H 2207 2517 50  0000 C CNN
 F 1 "USB_A" H 2207 2426 50  0000 C CNN
 F 2 "" H 2300 2000 50  0001 C CNN
@@
 AR Path="/5EA3ADD1" Ref="L?"  Part="1"
 AR Path="/5E9F954D/5EA3ADD1" Ref="L?"  Part="1"
-AR Path="/5E9DF2DA/5EA3ADD1" Ref="L?"  Part="1"
-F 0 "L?" V 3440 2150 50  0000 C CNN
+AR Path="/5E9DF2DA/5EA3ADD1" Ref="L5"  Part="1"
+F 0 "L5" V 3440 2150 50  0000 C CNN
 F 1 "L" V 3349 2150 50  0000 C CNN
 F 2 "" H 3250 2150 50  0001 C CNN
@@
 AR Path="/5EA3ADD7" Ref="L?"  Part="1"
 AR Path="/5E9F954D/5EA3ADD7" Ref="L?"  Part="1"
-AR Path="/5E9DF2DA/5EA3ADD7" Ref="L?"  Part="1"
-F 0 "L?" V 3540 2050 50  0000 C CNN
+AR Path="/5E9DF2DA/5EA3ADD7" Ref="L6"  Part="1"
+F 0 "L6" V 3540 2050 50  0000 C CNN
 F 1 "L" V 3449 2050 50  0000 C CNN
 F 2 "" H 3350 2050 50  0001 C CNN
@@
 AR Path="/5EA3ADDD" Ref="R?"  Part="1"
 AR Path="/5E9F954D/5EA3ADDD" Ref="R?"  Part="1"
-AR Path="/5E9DF2DA/5EA3ADDD" Ref="R?"  Part="1"
-F 0 "R?" V 3643 2050 50  0000 C CNN
+AR Path="/5E9DF2DA/5EA3ADDD" Ref="R13"  Part="1"
+F 0 "R13" V 3643 2050 50  0000 C CNN
 F 1 "R" V 3734 2050 50  0000 C CNN
 F 2 "" V 3780 2050 50  0001 C CNN
@@
 AR Path="/5EA3ADE3" Ref="R?"  Part="1"
 AR Path="/5E9F954D/5EA3ADE3" Ref="R?"  Part="1"
-AR Path="/5E9DF2DA/5EA3ADE3" Ref="R?"  Part="1"
-F 0 "R?" V 3493 2150 50  0000 C CNN
+AR Path="/5E9DF2DA/5EA3ADE3" Ref="R12"  Part="1"
+F 0 "R12" V 3493 2150 50  0000 C CNN
 F 1 "R" V 3584 2150 50  0000 C CNN
 F 2 "" V 3630 2150 50  0001 C CNN
@@
 AR Path="/5EA3ADF5" Ref="D?"  Part="1"
 AR Path="/5E9F954D/5EA3ADF5" Ref="D?"  Part="1"
-AR Path="/5E9DF2DA/5EA3ADF5" Ref="D?"  Part="1"
-F 0 "D?" V 2704 1479 50  0000 L CNN
+AR Path="/5E9DF2DA/5EA3ADF5" Ref="D4"  Part="1"
+F 0 "D4" V 2704 1479 50  0000 L CNN
 F 1 "1N47xxA" V 2795 1479 50  0000 L CNN
 F 2 "Diode_THT:D_DO-41_SOD81_P10.16mm_Horizontal" H 2750 1225 50  0001 C CNN
@@
 AR Path="/5EA3ADFB" Ref="C?"  Part="1"
 AR Path="/5E9F954D/5EA3ADFB" Ref="C?"  Part="1"
-AR Path="/5E9DF2DA/5EA3ADFB" Ref="C?"  Part="1"
-F 0 "C?" H 3265 1446 50  0000 L CNN
+AR Path="/5E9DF2DA/5EA3ADFB" Ref="C15"  Part="1"
+F 0 "C15" H 3265 1446 50  0000 L CNN
 F 1 "C" H 3265 1355 50  0000 L CNN
 F 2 "" H 3188 1250 50  0001 C CNN
@@
 AR Path="/5EA3AE01" Ref="C?"  Part="1"
 AR Path="/5E9F954D/5EA3AE01" Ref="C?"  Part="1"
-AR Path="/5E9DF2DA/5EA3AE01" Ref="C?"  Part="1"
-F 0 "C?" H 3615 1446 50  0000 L CNN
+AR Path="/5E9DF2DA/5EA3AE01" Ref="C16"  Part="1"
+F 0 "C16" H 3615 1446 50  0000 L CNN
 F 1 "C" H 3615 1355 50  0000 L CNN
 F 2 "" H 3538 1250 50  0001 C CNN
@@
 AR Path="/5EA3AE07" Ref="#PWR?"  Part="1"
 AR Path="/5E9F954D/5EA3AE07" Ref="#PWR?"  Part="1"
-AR Path="/5E9DF2DA/5EA3AE07" Ref="#PWR?"  Part="1"
-F 0 "#PWR?" H 3000 1500 50  0001 C CNN
+AR Path="/5E9DF2DA/5EA3AE07" Ref="#PWR0129"  Part="1"
+F 0 "#PWR0129" H 3000 1500 50  0001 C CNN
 F 1 "GND" H 3005 1577 50  0000 C CNN
 F 2 "" H 3000 1750 50  0001 C CNN
@@
 AR Path="/5EA3AE12" Ref="L?"  Part="1"
 AR Path="/5E9F954D/5EA3AE12" Ref="L?"  Part="1"
-AR Path="/5E9DF2DA/5EA3AE12" Ref="L?"  Part="1"
-F 0 "L?" V 4090 1150 50  0000 C CNN
+AR Path="/5E9DF2DA/5EA3AE12" Ref="L7"  Part="1"
+F 0 "L7" V 4090 1150 50  0000 C CNN
 F 1 "L" V 3999 1150 50  0000 C CNN
 F 2 "" H 3900 1150 50  0001 C CNN
@@
 	4250 1000 4250 1150
 $Comp
-L power:+3V3 #PWR?
+L power:+3V3 #PWR0130
 U 1 1 5EA60D1B
 P 9500 4950
-F 0 "#PWR?" H 9500 4800 50  0001 C CNN
+F 0 "#PWR0130" H 9500 4800 50  0001 C CNN
 F 1 "+3V3" H 9515 5123 50  0000 C CNN
 F 2 "" H 9500 4950 50  0001 C CNN
@@
 $EndComp
 $Comp
-L power:+5VD #PWR?
+L power:+5VD #PWR0131
 U 1 1 5EA613B3
 P 4250 1000
-F 0 "#PWR?" H 4250 850 50  0001 C CNN
+F 0 "#PWR0131" H 4250 850 50  0001 C CNN
 F 1 "+5VD" H 4265 1173 50  0000 C CNN
 F 2 "" H 4250 1000 50  0001 C CNN
@@
 $EndComp
 $Comp
-L power:GNDA #PWR?
+L power:GNDA #PWR0132
 U 1 1 5EA61C2C
 P 2900 2800
-F 0 "#PWR?" H 2900 2550 50  0001 C CNN
+F 0 "#PWR0132" H 2900 2550 50  0001 C CNN
 F 1 "GNDA" H 2905 2627 50  0000 C CNN
 F 2 "" H 2900 2800 50  0001 C CNN
@@
 $EndComp
 $Comp
-L power:GNDA #PWR?
+L power:GNDA #PWR0133
 U 1 1 5EA63529
 P 2150 2650
-F 0 "#PWR?" H 2150 2400 50  0001 C CNN
+F 0 "#PWR0133" H 2150 2400 50  0001 C CNN
 F 1 "GNDA" H 2155 2477 50  0000 C CNN
 F 2 "" H 2150 2650 50  0001 C CNN
@@
 $EndComp
 $Comp
-L power:GNDA #PWR?
+L power:GNDA #PWR0134
 U 1 1 5EA65F71
 P 8500 5600
-F 0 "#PWR?" H 8500 5350 50  0001 C CNN
+F 0 "#PWR0134" H 8500 5350 50  0001 C CNN
 F 1 "GNDA" H 8505 5427 50  0000 C CNN
 F 2 "" H 8500 5600 50  0001 C CNN
@@
 $EndComp
 $Comp
-L power:GNDA #PWR?
+L power:GNDA #PWR0135
 U 1 1 5EA6646F
 P 8850 5500
-F 0 "#PWR?" H 8850 5250 50  0001 C CNN
+F 0 "#PWR0135" H 8850 5250 50  0001 C CNN
 F 1 "GNDA" H 8855 5327 50  0000 C CNN
 F 2 "" H 8850 5500 50  0001 C CNN
@@
 P 8600 2100
 AR Path="/5E9DF408/5EA69339" Ref="J?"  Part="1"
-AR Path="/5E9DF2DA/5EA69339" Ref="J?"  Part="1"
-F 0 "J?" H 8071 2146 50  0000 R CNN
+AR Path="/5E9DF2DA/5EA69339" Ref="J7"  Part="1"
+F 0 "J7" H 8071 2146 50  0000 R CNN
 F 1 "Conn_ARM_JTAG_SWD_20" H 8071 2055 50  0000 R CNN
 F 2 "" H 9050 1050 50  0001 L TNN
@@
 P 9950 1900
 AR Path="/5E9DF408/5EA6935F" Ref="#PWR?"  Part="1"
-AR Path="/5E9DF2DA/5EA6935F" Ref="#PWR?"  Part="1"
-F 0 "#PWR?" H 9950 1650 50  0001 C CNN
+AR Path="/5E9DF2DA/5EA6935F" Ref="#PWR0136"  Part="1"
+F 0 "#PWR0136" H 9950 1650 50  0001 C CNN
 F 1 "GND" V 9955 1772 50  0000 R CNN
 F 2 "" H 9950 1900 50  0001 C CNN
@@
 P 9700 1900
 AR Path="/5E9DF408/5EA69365" Ref="R?"  Part="1"
-AR Path="/5E9DF2DA/5EA69365" Ref="R?"  Part="1"
-F 0 "R?" V 9493 1900 50  0001 C CNN
+AR Path="/5E9DF2DA/5EA69365" Ref="R15"  Part="1"
+F 0 "R15" V 9493 1900 50  0001 C CNN
 F 1 "510" V 9585 1900 50  0000 C CNN
 F 2 "" V 9630 1900 50  0001 C CNN
@@
 $EndComp
 $Comp
-L power:GNDA #PWR?
+L power:GNDA #PWR0137
 U 1 1 5EA65BD2
 P 3750 4450
-F 0 "#PWR?" H 3750 4200 50  0001 C CNN
+F 0 "#PWR0137" H 3750 4200 50  0001 C CNN
 F 1 "GNDA" H 3755 4277 50  0000 C CNN
 F 2 "" H 3750 4450 50  0001 C CNN
@@
 $EndComp
 $Comp
-L power:GNDA #PWR?
+L power:GNDA #PWR0138
 U 1 1 5EA63E3E
 P 3600 7000
-F 0 "#PWR?" H 3600 6750 50  0001 C CNN
+F 0 "#PWR0138" H 3600 6750 50  0001 C CNN
 F 1 "GNDA" H 3605 6827 50  0000 C CNN
 F 2 "" H 3600 7000 50  0001 C CNN
@@
 $EndComp
 $Comp
-L power:+3V3 #PWR?
+L power:+3V3 #PWR0139
 U 1 1 5EA6068B
 P 4000 3850
-F 0 "#PWR?" H 4000 3700 50  0001 C CNN
+F 0 "#PWR0139" H 4000 3700 50  0001 C CNN
 F 1 "+3V3" H 4015 4023 50  0000 C CNN
 F 2 "" H 4000 3850 50  0001 C CNN
@@
 AR Path="/5EA3688F" Ref="C?"  Part="1"
 AR Path="/5E9F954D/5EA3688F" Ref="C?"  Part="1"
-AR Path="/5E9DF2DA/5EA3688F" Ref="C?"  Part="1"
-F 0 "C?" H 3715 4296 50  0000 L CNN
+AR Path="/5E9DF2DA/5EA3688F" Ref="C17"  Part="1"
+F 0 "C17" H 3715 4296 50  0000 L CNN
 F 1 "0.1uF" H 3715 4205 50  0000 L CNN
 F 2 "" H 3638 4100 50  0001 C CNN
@@
 AR Path="/5EA36889" Ref="C?"  Part="1"
 AR Path="/5E9F954D/5EA36889" Ref="C?"  Part="1"
-AR Path="/5E9DF2DA/5EA36889" Ref="C?"  Part="1"
-F 0 "C?" H 4115 4296 50  0000 L CNN
+AR Path="/5E9DF2DA/5EA36889" Ref="C18"  Part="1"
+F 0 "C18" H 4115 4296 50  0000 L CNN
 F 1 "0.1uF" H 4115 4205 50  0000 L CNN
 F 2 "" H 4038 4100 50  0001 C CNN
@@
 AR Path="/5EA36883" Ref="U?"  Part="1"
 AR Path="/5E9F954D/5EA36883" Ref="U?"  Part="1"
-AR Path="/5E9DF2DA/5EA36883" Ref="U?"  Part="1"
-F 0 "U?" H 3300 4511 50  0000 C CNN
+AR Path="/5E9DF2DA/5EA36883" Ref="U6"  Part="1"
+F 0 "U6" H 3300 4511 50  0000 C CNN
 F 1 "Omega2+" H 3300 4420 50  0000 C CNN
 F 2 "Module:Onion_Omega2+" H 3300 4300 50  0001 C CNN
@@
 	4100 5100 4000 5100
 $Comp
-L power:GNDA #PWR?
+L power:GNDA #PWR0140
 U 1 1 5EA8F42E
 P 8500 3000
-F 0 "#PWR?" H 8500 2750 50  0001 C CNN
+F 0 "#PWR0140" H 8500 2750 50  0001 C CNN
 F 1 "GNDA" H 8505 2827 50  0000 C CNN
 F 2 "" H 8500 3000 50  0001 C CNN
@@
 $EndComp
 $Comp
-L power:+3V3 #PWR?
+L power:+3V3 #PWR0141
 U 1 1 5EA9158C
 P 8600 1000
-F 0 "#PWR?" H 8600 850 50  0001 C CNN
+F 0 "#PWR0141" H 8600 850 50  0001 C CNN
 F 1 "+3V3" H 8615 1173 50  0000 C CNN
 F 2 "" H 8600 1000 50  0001 C CNN

Commit message: Add files via upload
Parts:
- C15, C16, C17, C18, C19: footprint (none) -> Capacitor_SMD:C_0603_1608Metric_Pad1.05x0.95mm_HandSolder
- J6: footprint (none) -> Connector_USB:USB_A_Molex_105057_Vertical
- J7: footprint (none) -> Connector_PinSocket_1.27mm:PinSocket_2x10_P1.27mm_Vertical
- L5, L6, L7: footprint (none) -> Inductor_SMD:L_2010_5025Metric
- R12, R13, R14, R15: footprint (none) -> Resistor_SMD:R_0201_0603Metric
Changed lines of the file:
@@
 F 0 "R14" V 8993 5100 50  0000 C CNN
 F 1 "10k" V 9084 5100 50  0000 C CNN
-F 2 "" V 9130 5100 50  0001 C CNN
+F 2 "Resistor_SMD:R_0201_0603Metric" V 9130 5100 50  0001 C CNN
 F 3 "~" H 9200 5100 50  0001 C CNN
 	1    9200 5100
@@
 F 0 "C19" H 8965 5296 50  0000 L CNN
 F 1 "0.1uF" H 8965 5205 50  0000 L CNN
-F 2 "" H 8888 5100 50  0001 C CNN
+F 2 "Capacitor_SMD:C_0603_1608Metric_Pad1.05x0.95mm_HandSolder" H 8888 5100 50  0001 C CNN
 F 3 "~" H 8850 5250 50  0001 C CNN
 	1    8850 5250
@@
 F 0 "J6" H 2207 2517 50  0000 C CNN
 F 1 "USB_A" H 2207 2426 50  0000 C CNN
-F 2 "" H 2300 2000 50  0001 C CNN
+F 2 "Connector_USB:USB_A_Molex_105057_Vertical" H 2300 2000 50  0001 C CNN
 F 3 " ~" H 2300 2000 50  0001 C CNN
 	1    2150 2050
@@
 F 0 "L5" V 3440 2150 50  0000 C CNN
 F 1 "L" V 3349 2150 50  0000 C CNN
-F 2 "" H 3250 2150 50  0001 C CNN
+F 2 "Inductor_SMD:L_2010_5025Metric" H 3250 2150 50  0001 C CNN
 F 3 "~" H 3250 2150 50  0001 C CNN
 	1    3250 2150
@@
 F 0 "L6" V 3540 2050 50  0000 C CNN
 F 1 "L" V 3449 2050 50  0000 C CNN
-F 2 "" H 3350 2050 50  0001 C CNN
+F 2 "Inductor_SMD:L_2010_5025Metric" H 3350 2050 50  0001 C CNN
 F 3 "~" H 3350 2050 50  0001 C CNN
 	1    3350 2050
@@
 F 0 "R13" V 3643 2050 50  0000 C CNN
 F 1 "R" V 3734 2050 50  0000 C CNN
-F 2 "" V 3780 2050 50  0001 C CNN
+F 2 "Resistor_SMD:R_0201_0603Metric" V 3780 2050 50  0001 C CNN
 F 3 "~" H 3850 2050 50  0001 C CNN
 	1    3850 2050
@@
 F 0 "R12" V 3493 2150 50  0000 C CNN
 F 1 "R" V 3584 2150 50  0000 C CNN
-F 2 "" V 3630 2150 50  0001 C CNN
+F 2 "Resistor_SMD:R_0201_0603Metric" V 3630 2150 50  0001 C CNN
 F 3 "~" H 3700 2150 50  0001 C CNN
 	1    3700 2150
@@
 F 0 "C15" H 3265 1446 50  0000 L CNN
 F 1 "C" H 3265 1355 50  0000 L CNN
-F 2 "" H 3188 1250 50  0001 C CNN
+F 2 "Capacitor_SMD:C_0603_1608Metric_Pad1.05x0.95mm_HandSolder" H 3188 1250 50  0001 C CNN
 F 3 "~" H 3150 1400 50  0001 C CNN
 	1    3150 1400
@@
 F 0 "C16" H 3615 1446 50  0000 L CNN
 F 1 "C" H 3615 1355 50  0000 L CNN
-F 2 "" H 3538 1250 50  0001 C CNN
+F 2 "Capacitor_SMD:C_0603_1608Metric_Pad1.05x0.95mm_HandSolder" H 3538 1250 50  0001 C CNN
 F 3 "~" H 3500 1400 50  0001 C CNN
 	1    3500 1400
@@
 F 0 "L7" V 4090 1150 50  0000 C CNN
 F 1 "L" V 3999 1150 50  0000 C CNN
-F 2 "" H 3900 1150 50  0001 C CNN
+F 2 "Inductor_SMD:L_2010_5025Metric" H 3900 1150 50  0001 C CNN
 F 3 "~" H 3900 1150 50  0001 C CNN
 	1    3900 1150
@@
 F 0 "J7" H 8071 2146 50  0000 R CNN
 F 1 "Conn_ARM_JTAG_SWD_20" H 8071 2055 50  0000 R CNN
-F 2 "" H 9050 1050 50  0001 L TNN
+F 2 "Connector_PinSocket_1.27mm:PinSocket_2x10_P1.27mm_Vertical" H 9050 1050 50  0001 L TNN
 F 3 "http://infocenter.arm.com/help/topic/com.arm.doc.dui0499b/DUI0499B_system_design_reference.pdf" V 8250 850 50  0001 C CNN
 	1    8600 2100
@@
 F 0 "R15" V 9493 1900 50  0001 C CNN
 F 1 "510" V 9585 1900 50  0000 C CNN
-F 2 "" V 9630 1900 50  0001 C CNN
+F 2 "Resistor_SMD:R_0201_0603Metric" V 9630 1900 50  0001 C CNN
 F 3 "~" H 9700 1900 50  0001 C CNN
 	1    9700 1900
@@
 F 0 "C17" H 3715 4296 50  0000 L CNN
 F 1 "0.1uF" H 3715 4205 50  0000 L CNN
-F 2 "" H 3638 4100 50  0001 C CNN
+F 2 "Capacitor_SMD:C_0603_1608Metric_Pad1.05x0.95mm_HandSolder" H 3638 4100 50  0001 C CNN
 F 3 "~" H 3600 4250 50  0001 C CNN
 	1    3600 4250
@@
 F 0 "C18" H 4115 4296 50  0000 L CNN
 F 1 "0.1uF" H 4115 4205 50  0000 L CNN
-F 2 "" H 4038 4100 50  0001 C CNN
+F 2 "Capacitor_SMD:C_0603_1608Metric_Pad1.05x0.95mm_HandSolder" H 4038 4100 50  0001 C CNN
 F 3 "~" H 4000 4250 50  0001 C CNN
 	1    4000 4250

Commit message: Add files via upload
Parts:
- SW2: footprint (none) -> Button_Switch_SMD:SW_DIP_SPSTx05_Slide_6.7x14.26mm_W6.73mm_P2.54mm_LowProfile_JPin
Changed lines of the file:
@@
 F 0 "SW2" V 8546 5352 50  0000 R CNN
 F 1 "SW_Push" V 8455 5352 50  0000 R CNN
-F 2 "" H 8500 5600 50  0001 C CNN
+F 2 "Button_Switch_SMD:SW_DIP_SPSTx05_Slide_6.7x14.26mm_W6.73mm_P2.54mm_LowProfile_JPin" H 8500 5600 50  0001 C CNN
 F 3 "~" H 8500 5600 50  0001 C CNN
 	1    8500 5400

Commit message: Add files via upload
Parts:
- SW2: footprint Button_Switch_SMD:SW_DIP_SPSTx05_Slide_6.7x14.26mm_W6.73mm_P2.54mm_LowProfile_JPin -> Button_Switch_SMD:SW_DIP_SPSTx01_Slide_6.7x4.1mm_W6.73mm_P2.54mm_LowProfile_JPin
Connections:
- net labels added: +3V0
- net labels removed: +3V3, GND
- wire segments 72 -> 73
Changed lines of the file:
@@
 F 0 "SW2" V 8546 5352 50  0000 R CNN
 F 1 "SW_Push" V 8455 5352 50  0000 R CNN
-F 2 "Button_Switch_SMD:SW_DIP_SPSTx05_Slide_6.7x14.26mm_W6.73mm_P2.54mm_LowProfile_JPin" H 8500 5600 50  0001 C CNN
+F 2 "Button_Switch_SMD:SW_DIP_SPSTx01_Slide_6.7x4.1mm_W6.73mm_P2.54mm_LowProfile_JPin" H 8500 5600 50  0001 C CNN
 F 3 "~" H 8500 5600 50  0001 C CNN
 	1    8500 5400
@@
 Wire Wire Line
 	2900 2800 2900 2650
-$Comp
-L Device:L L?
-U 1 1 5EA3ADD1
-P 3250 2150
-AR Path="/5EA3ADD1" Ref="L?"  Part="1"
-AR Path="/5E9F954D/5EA3ADD1" Ref="L?"  Part="1"
-AR Path="/5E9DF2DA/5EA3ADD1" Ref="L5"  Part="1"
-F 0 "L5" V 3440 2150 50  0000 C CNN
-F 1 "L" V 3349 2150 50  0000 C CNN
-F 2 "Inductor_SMD:L_2010_5025Metric" H 3250 2150 50  0001 C CNN
-F 3 "~" H 3250 2150 50  0001 C CNN
-	1    3250 2150
-	0    -1   -1   0
-$EndComp
 $Comp
 L Device:L L?
@@
 	3550 2150 3400 2150
 Wire Wire Line
-	3100 2150 2800 2150
-Wire Wire Line
 	2800 2250 2800 2150
-Connection ~ 2800 2150
 Wire Wire Line
 	2800 2150 2450 2150
 Wire Wire Line
-	3200 2050 3000 2050
-Wire Wire Line
 	3000 2250 3000 2050
-Connection ~ 3000 2050
 Wire Wire Line
 	3000 2050 2450 2050
@@
 	1    0    0    -1
 $EndComp
-$Comp
-L power:GND #PWR?
-U 1 1 5EA3AE07
-P 3000 1750
-AR Path="/5EA3AE07" Ref="#PWR?"  Part="1"
-AR Path="/5E9F954D/5EA3AE07" Ref="#PWR?"  Part="1"
-AR Path="/5E9DF2DA/5EA3AE07" Ref="#PWR0129"  Part="1"
-F 0 "#PWR0129" H 3000 1500 50  0001 C CNN
-F 1 "GND" H 3005 1577 50  0000 C CNN
-F 2 "" H 3000 1750 50  0001 C CNN
-F 3 "" H 3000 1750 50  0001 C CNN
-	1    3000 1750
-	1    0    0    -1
-$EndComp
 Wire Wire Line
 	3500 1550 3500 1650
 Wire Wire Line
-	3500 1650 3150 1650
-Wire Wire Line
 	2750 1550 2750 1650
-Wire Wire Line
-	3150 1550 3150 1650
-Connection ~ 3150 1650
 $Comp
 L Device:L L?
@@
 Wire Wire Line
 	3000 1750 3000 1650
-Connection ~ 3000 1650
-Wire Wire Line
-	3000 1650 3150 1650
 Wire Wire Line
 	3750 1150 3500 1150
@@
 Wire Wire Line
 	4250 1000 4250 1150
-$Comp
-L power:+3V3 #PWR0130
-U 1 1 5EA60D1B
-P 9500 4950
-F 0 "#PWR0130" H 9500 4800 50  0001 C CNN
-F 1 "+3V3" H 9515 5123 50  0000 C CNN
-F 2 "" H 9500 4950 50  0001 C CNN
-F 3 "" H 9500 4950 50  0001 C CNN
-	1    9500 4950
-	1    0    0    -1
-$EndComp
 $Comp
 L power:+5VD #PWR0131
@@
 Wire Wire Line
 	9200 1900 9550 1900
-Wire Wire Line
-	9950 1900 9850 1900
-$Comp
-L power:GND #PWR?
-U 1 1 5EA6935F
-P 9950 1900
-AR Path="/5E9DF408/5EA6935F" Ref="#PWR?"  Part="1"
-AR Path="/5E9DF2DA/5EA6935F" Ref="#PWR0136"  Part="1"
-F 0 "#PWR0136" H 9950 1650 50  0001 C CNN
-F 1 "GND" V 9955 1772 50  0000 R CNN
-F 2 "" H 9950 1900 50  0001 C CNN
-F 3 "" H 9950 1900 50  0001 C CNN
-	1    9950 1900
-	0    -1   -1   0
-$EndComp
 $Comp
 L Device:R R?
@@
 	1    0    0    -1
 $EndComp
-$Comp
-L power:+3V3 #PWR0139
-U 1 1 5EA6068B
-P 4000 3850
-F 0 "#PWR0139" H 4000 3700 50  0001 C CNN
-F 1 "+3V3" H 4015 4023 50  0000 C CNN
-F 2 "" H 4000 3850 50  0001 C CNN
-F 3 "" H 4000 3850 50  0001 C CNN
-	1    4000 3850
-	1    0    0    -1
-$EndComp
 Connection ~ 4000 4050
 Wire Wire Line
@@
 F 3 "" H 8500 3000 50  0001 C CNN
 	1    8500 3000
-	1    0    0    -1
-$EndComp
-$Comp
-L power:+3V3 #PWR0141
-U 1 1 5EA9158C
-P 8600 1000
-F 0 "#PWR0141" H 8600 850 50  0001 C CNN
-F 1 "+3V3" H 8615 1173 50  0000 C CNN
-F 2 "" H 8600 1000 50  0001 C CNN
-F 3 "" H 8600 1000 50  0001 C CNN
-	1    8600 1000
 	1    0    0    -1
 $EndComp
@@
 Text Notes 500  3500 0    50   ~ 0
 USB
+$Comp
+L power:GNDA #PWR0129
+U 1 1 5EB4B7ED
+P 3000 1750
+F 0 "#PWR0129" H 3000 1500 50  0001 C CNN
+F 1 "GNDA" H 3005 1577 50  0000 C CNN
+F 2 "" H 3000 1750 50  0001 C CNN
+F 3 "" H 3000 1750 50  0001 C CNN
+	1    3000 1750
+	1    0    0    -1
+$EndComp
+$Comp
+L power:GNDA #PWR0136
+U 1 1 5EB4EF5F
+P 10150 2050
+F 0 "#PWR0136" H 10150 1800 50  0001 C CNN
+F 1 "GNDA" H 10155 1877 50  0000 C CNN
+F 2 "" H 10150 2050 50  0001 C CNN
+F 3 "" H 10150 2050 50  0001 C CNN
+	1    10150 2050
+	1    0    0    -1
+$EndComp
+Wire Wire Line
+	9850 1900 10150 1900
+Wire Wire Line
+	10150 1900 10150 2050
+Connection ~ 3000 1650
+Connection ~ 3000 2050
+Connection ~ 2800 2150
+Wire Wire Line
+	3000 1650 3150 1650
+Wire Wire Line
+	3150 1550 3150 1650
+Wire Wire Line
+	3200 2050 3000 2050
+Wire Wire Line
+	3100 2150 2800 2150
+$Comp
+L Device:L L?
+U 1 1 5EA3ADD1
+P 3250 2150
+AR Path="/5EA3ADD1" Ref="L?"  Part="1"
+AR Path="/5E9F954D/5EA3ADD1" Ref="L?"  Part="1"
+AR Path="/5E9DF2DA/5EA3ADD1" Ref="L5"  Part="1"
+F 0 "L5" V 3440 2150 50  0000 C CNN
+F 1 "L" V 3349 2150 50  0000 C CNN
+F 2 "Inductor_SMD:L_2010_5025Metric" H 3250 2150 50  0001 C CNN
+F 3 "~" H 3250 2150 50  0001 C CNN
+	1    3250 2150
+	0    -1   -1   0
+$EndComp
+Connection ~ 3150 1650
+Wire Wire Line
+	3150 1650 3500 1650
+$Comp
+L power:+3V0 #PWR0130
+U 1 1 5EB5B908
+P 4000 3850
+F 0 "#PWR0130" H 4000 3700 50  0001 C CNN
+F 1 "+3V0" H 4015 4023 50  0000 C CNN
+F 2 "" H 4000 3850 50  0001 C CNN
+F 3 "" H 4000 3850 50  0001 C CNN
+	1    4000 3850
+	1    0    0    -1
+$EndComp
+$Comp
+L power:+3V0 #PWR0139
+U 1 1 5EB5BF1C
+P 9500 4950
+F 0 "#PWR0139" H 9500 4800 50  0001 C CNN
+F 1 "+3V0" H 9515 5123 50  0000 C CNN
+F 2 "" H 9500 4950 50  0001 C CNN
+F 3 "" H 9500 4950 50  0001 C CNN
+	1    9500 4950
+	1    0    0    -1
+$EndComp
+$Comp
+L power:+3V0 #PWR0141
+U 1 1 5EB5C40F
+P 8600 1000
+F 0 "#PWR0141" H 8600 850 50  0001 C CNN
+F 1 "+3V0" H 8615 1173 50  0000 C CNN
+F 2 "" H 8600 1000 50  0001 C CNN
+F 3 "" H 8600 1000 50  0001 C CNN
+	1    8600 1000
+	1    0    0    -1
+$EndComp
 $EndSCHEMATC

Commit message: Add files via upload
Parts:
- removed C18: 0.1uF, Capacitor_SMD:C_0603_1608Metric_Pad1.05x0.95mm_HandSolder, symbol Device:C
- removed J7: Conn_ARM_JTAG_SWD_20, Connector_PinSocket_1.27mm:PinSocket_2x10_P1.27mm_Vertical, symbol Connector:Conn_ARM_JTAG_SWD_20
- added C33, C35: 0.1uF, Capacitor_SMD:C_0603_1608Metric_Pad1.05x0.95mm_HandSolder, symbol Device:C
- added J7: AVR-JTAG-10, Connector_PinSocket_2.54mm:PinSocket_1x10_P2.54mm_Vertical, symbol Connector:AVR-JTAG-10
- L5, L6, L7: footprint Inductor_SMD:L_2010_5025Metric -> Inductor_SMD:L_2010_5025Metric_Pad1.52x2.65mm_HandSolder
- R12, R13, R14, R15: footprint Resistor_SMD:R_0201_0603Metric -> Resistor_SMD:R_0603_1608Metric_Pad1.05x0.95mm_HandSolder
Connections:
- wire segments 73 -> 75
