File: proyecto/proyecto.kicad_pcb (KiCad board)
At the start: 2 copper layers, 109 parts, among them J1 Conn_01x03, J2 Conn_01x03, J3 USB_A, J4 Conn_ARM_JTAG_SWD_20, J5 USB_B_Mini, J6 USB_A, J7 Conn_ARM_JTAG_SWD_20, J8 USB_B_Mini, J9 Conn_ARM_JTAG_SWD_20, Q1 Q_PMOS_DSG, Q2 Q_PMOS_DSG, SW1 SW_Push, SW2 SW_Push, SW3 SW_Push, U1 DRV8848, U10 STM32L052C6Tx, U11 LM1117-5.0, U12 LM1117-5.0, U2 Omega2+, U3 MCP73811T-435I-OT, U4 LM1117-3.3, U5 TPS61200DRC, U6 Omega2+, U7 LM1117-3.3, U8 MCP73811T-435I-OT, U9 TPS61200DRC, Y1 24M

Commit message: Add files via upload
Parts:
- Q1, Q2: footprint Diode_SMD:D_0805_2012Metric -> Package_TO_SOT_SMD:SOT-23
- SW2: moved to B.Cu
- moved R22 137.4 mm to (113.5, 89.4), turned to 180 degrees
- moved C20 124.3 mm to (91.8, 158.2)
- moved J9 117.9 mm to (109.7, 83.3)
- moved R20 117.3 mm to (135.4, 91.2)
- moved C36 117.1 mm to (140.6, 96.8)
- moved U9 116.1 mm to (100.3, 177.8), turned to 90 degrees
- moved U10 114.1 mm to (121.2, 86.6), turned to 180 degrees
- moved R21 111.7 mm to (138.2, 94.5)
- moved C40 110.5 mm to (89.2, 167.1)
- moved R19 108.7 mm to (94.8, 170.7)
- moved Y1 107.2 mm to (136.1, 83.6)
- moved C32 106.8 mm to (123.1, 100.6)
- moved C30 106.6 mm to (145.9, 94.2)
- moved R17 106.5 mm to (83.8, 167.3)
- moved C28 105.6 mm to (138.9, 99.3)
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Connections:
- U10 pad 25: /Microcontrolador/TCK1 -> /Microcontrolador/TD11
- U10 pad 27: /Microcontrolador/TD01 -> /Microcontrolador/TCK1
- U10 pad 28: /Microcontrolador/TD11 -> /Microcontrolador/TD01
Routing:
- net GND: track 0.00 -> 570.0 mm
- net +3V0: track 0.00 -> 259.1 mm
- net +3V8: track 0.00 -> 180.3 mm
- net GNDA: track 0.00 -> 147.8 mm
- net +5VP: track 0.00 -> 118.1 mm
- net +5VL: track 0.00 -> 101.2 mm
- net Net-(C15-Pad1): track 0.00 -> 75.7 mm
- net +5V: track 0.00 -> 69.8 mm
- net Net-(C2-Pad1): track 0.00 -> 59.8 mm
- net Net-(C20-Pad1): track 0.00 -> 45.0 mm
- net Net-(D5-Pad2): track 0.00 -> 44.5 mm
- net Net-(D5-Pad1): track 0.00 -> 43.1 mm
- net Net-(BT2-Pad1): track 0.00 -> 42.2 mm
- net Net-(C25-Pad1): track 0.00 -> 39.2 mm
- net +5VD: track 0.00 -> 38.3 mm
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
Commit message: Add files via upload
Parts:
- C10, C11, C14, C28, C29, C30, C32, C33, C35, C37, C4, C5, C8, J7, R11: moved to B.Cu
- SW2: moved to F.Cu
- moved U4 134.5 mm to (47.3, 31.9), turned to 90 degrees
- moved C37 128.2 mm to (50.6, 43.4)
- moved C33 123.6 mm to (42.3, 48.0), turned to 180 degrees
- moved C4 123.3 mm to (46.5, 47.9)
- moved C10 122.8 mm to (46.5, 38.8), turned to 0 degrees
- moved C11 120.8 mm to (46.5, 41.2)
- moved C5 120.2 mm to (42.4, 38.9), turned to 180 degrees
- moved C29 119.6 mm to (46.5, 45.8)
- moved C35 119.5 mm to (46.5, 43.6)
- moved C8 117.7 mm to (50.7, 41.1), turned to 180 degrees
- moved C30 115.3 mm to (42.3, 43.6), turned to 180 degrees
- moved C28 112.6 mm to (42.4, 41.3), turned to 180 degrees
- moved R11 111.4 mm to (51.1, 45.4), turned to 180 degrees
- moved C39 106.2 mm to (54.2, 35.1), turned to 180 degrees
- moved C38 102.8 mm to (54.0, 32.8), turned to 180 degrees
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Connections:
- net /Microcontrolador/PH_EN34 renamed Net-(U10-Pad31)
- U10 pad 11: /Microcontrolador/PH_1A -> Net-(U10-Pad11)
- U10 pad 12: /Microcontrolador/PH_2A -> Net-(U10-Pad12)
- U10 pad 13: /Microcontrolador/PH_EN12 -> Net-(U10-Pad13)
- U10 pad 29: /Microcontrolador/PH_3A -> Net-(U10-Pad29)
- U10 pad 30: /Microcontrolador/PH_4A -> Net-(U10-Pad30)
- U10 pad 34: Net-(U10-Pad34) -> /Microcontrolador/PH_EN12
- U10 pad 37: Net-(U10-Pad37) -> /Microcontrolador/PH_1A
- U10 pad 38: Net-(U10-Pad38) -> /Microcontrolador/PH_2A
- U10 pad 39: Net-(U10-Pad39) -> /Microcontrolador/PH_4A
- U10 pad 40: Net-(U10-Pad40) -> /Microcontrolador/PH_3A
Routing:
- net +3V0: track 259.1 -> 0.00 mm
- net GND: track 570.0 -> 353.2 mm, vias 0 -> 12
- net GNDA: track 147.8 -> 0.00 mm
- net +5VP: track 118.1 -> 0.00 mm
- net +5V: track 69.8 -> 134.1 mm
- net Net-(C15-Pad1): track 75.7 -> 13.3 mm
- net +3V8: track 180.3 -> 119.7 mm, vias 0 -> 4
- net Net-(C20-Pad1): track 45.0 -> 0.00 mm
- net /Procesador/TD02: track 0.00 -> 44.3 mm
- net +5VL: track 101.2 -> 144.0 mm, vias 0 -> 3
- net Net-(BT2-Pad1): track 42.2 -> 0.00 mm
- net Net-(C2-Pad1): track 59.8 -> 19.2 mm
- net /Procesador/TD12: track 0.00 -> 40.1 mm
- net Net-(C25-Pad1): track 39.2 -> 0.00 mm
- net +5VD: track 38.3 -> 0.00 mm
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Other:
- net class Dig added: clearance 0.1, trace_width 0.25, via_dia 0.8, via_drill 0.4

Commit message: Add files via upload
Parts:
- removed BT1: Battery_Cell_1, Battery:Battery_Panasonic_CR3032-VCN_Vertical_CircularHoles
- removed BT2: Battery_Cell_2, Battery:Battery_Panasonic_CR3032-VCN_Vertical_CircularHoles
- added J10: Conn_01x02, Connector_PinHeader_1.00mm:PinHeader_1x02_P1.00mm_Horizontal, F.Cu at (110.0, 163.3)
- added R23: 100, Resistor_SMD:R_0603_1608Metric_Pad1.05x0.95mm_HandSolder, F.Cu at (102.1, 48.8)
- added R24: 100, Resistor_SMD:R_0603_1608Metric_Pad1.05x0.95mm_HandSolder, F.Cu at (102.0, 44.5)
- added R25: 100, Resistor_SMD:R_0603_1608Metric_Pad1.05x0.95mm_HandSolder, F.Cu at (102.0, 46.7)
- added R26: 100, Resistor_SMD:R_0603_1608Metric_Pad1.05x0.95mm_HandSolder, F.Cu at (95.0, 63.8)
- C10, C11, C14, C28, C29, C30, C37, C4, C5, C8: moved to F.Cu
- C32, C33, C35: value 0.1uM -> 0.1uF; moved to F.Cu
- J1, J2: footprint Connector_JST:JST_EH_B3B-EH-A_1x03_P2.50mm_Vertical -> Connector_PinHeader_1.00mm:PinHeader_1x03_P1.00mm_Horizontal
- J4: value Conn_ARM_JTAG_SWD_20 -> AVR-JTAG-10; footprint Connector_PinSocket_1.27mm:PinSocket_2x10_P1.27mm_Vertical -> Connector_PinSocket_2.54mm:PinSocket_1x10_P2.54mm_Vertical
- J7: value Conn_ARM_JTAG_SWD_20 -> AVR-JTAG-10; footprint Connector_PinSocket_1.27mm:PinSocket_2x10_P1.27mm_Vertical -> Connector_PinSocket_2.54mm:PinSocket_1x10_P2.54mm_Vertical; moved to F.Cu
- J9: value Conn_ARM_JTAG_SWD_20 -> Conn_01x02; footprint Connector_PinSocket_1.27mm:PinSocket_2x10_P1.27mm_Vertical -> Connector_PinHeader_1.00mm:PinHeader_1x02_P1.00mm_Horizontal
- L1, L2, L3, L4, L5, L6, L7, L8: footprint Inductor_SMD:L_2010_5025Metric -> Inductor_SMD:L_2010_5025Metric_Pad1.52x2.65mm_HandSolder
- R1, R10, R12, R13, R14, R15, R16, R17, R18, R19, R2, R20, R21, R3, R4, R5, R6, R7, R8, R9: footprint Resistor_SMD:R_0201_0603Metric -> Resistor_SMD:R_0603_1608Metric_Pad1.05x0.95mm_HandSolder
- R11: footprint Resistor_SMD:R_0201_0603Metric -> Resistor_SMD:R_0603_1608Metric_Pad1.05x0.95mm_HandSolder; moved to F.Cu
- R22: value 510 -> 100; footprint Resistor_SMD:R_0201_0603Metric -> Resistor_SMD:R_0603_1608Metric_Pad1.05x0.95mm_HandSolder
- Y1: footprint Crystal:Crystal_HC35-U -> Crystal:Crystal_HC49-U_Horizontal
- moved U4 125.3 mm to (171.4, 48.8), turned to 0 degrees
- moved C18 117.9 mm to (113.8, 38.7), turned to 270 degrees
- moved C10 116.4 mm to (162.6, 48.0), turned to 180 degrees
- moved C11 116.1 mm to (162.6, 45.5), turned to 180 degrees
- moved R11 114.7 mm to (165.4, 54.9), turned to 0 degrees
- moved U11 113.4 mm to (171.4, 39.1)
- moved C8 112.3 mm to (162.6, 50.8)
- moved C37 112.0 mm to (162.6, 41.4)
- moved C38 108.7 mm to (162.7, 36.6)
- moved C39 108.5 mm to (162.6, 39.1)
- moved SW2 101.8 mm to (141.0, 163.1), turned to 180 degrees
- moved C35 96.1 mm to (95.2, 126.4), turned to 270 degrees
- moved C5 95.6 mm to (137.2, 51.1), turned to 0 degrees
- moved C14 94.4 mm to (141.0, 66.0)
- moved C4 90.9 mm to (137.2, 53.1)
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Connections:
- C18 pad 1: +3V0 -> +3V8
- C18 pad 2: GNDA -> GND
- C33 pad 1: +3V8 -> +3V0
- C33 pad 2: GND -> GNDA
- C35 pad 1: +3V8 -> +3V0
- C35 pad 2: GND -> GNDA
- C9 pad 1: Net-(BT1-Pad1) -> Net-(C9-Pad1)
- J4 pad 1: +3V8 -> /Procesador/TCK2
- J4 pad 10: GND -> Net-(J4-Pad10)
- J4 pad 2: +3V8 -> Net-(J4-Pad10)
- J4 pad 3: /Procesador/TRST2 -> /Procesador/TD02
- J4 pad 4: GND -> +3V8
- J4 pad 5: /Procesador/TD12 -> /Procesador/TMS2
- J4 pad 6: GND -> /Procesador/SRST2
- J4 pad 7: /Procesador/TMS2 -> +3V8
- J4 pad 8: GND -> /Procesador/TRST2
- J4 pad 9: /Procesador/TCK2 -> /Procesador/TD12
- J7 pad 1: +3V0 -> /camara/TCK3
- J7 pad 10: GNDA -> Net-(J7-Pad10)
- J7 pad 2: +3V0 -> Net-(J7-Pad10)
- J7 pad 3: /camara/TRST3 -> /camara/TD03
- J7 pad 4: GNDA -> +3V0
- J7 pad 5: /camara/TD13 -> /camara/TMS3
- J7 pad 6: GNDA -> /camara/SRST3
- J7 pad 7: /camara/TMS3 -> +3V0
- J7 pad 8: GNDA -> /camara/TRST3
- J7 pad 9: /camara/TCK3 -> /camara/TD13
- J9 pad 1: +3V8 -> Net-(C9-Pad1)
- J9 pad 2: +3V8 -> GND
- Q1 pad 2: Net-(BT1-Pad1) -> Net-(C9-Pad1)
- R15 pad 2: Net-(J7-Pad11) -> Net-(J7-Pad10)
- R22 pad 1: GND -> Net-(R22-Pad1)
- R22 pad 2: Net-(J9-Pad11) -> /Microcontrolador/MISO
- R7 pad 2: Net-(J4-Pad11) -> Net-(J4-Pad10)
- U10 pad 24: Net-(U10-Pad24) -> +3V8
- U2 pad 10: /Microcontrolador/MISO -> Net-(R22-Pad1)
- U2 pad 11: /Microcontrolador/MOSI -> Net-(R23-Pad1)
- U2 pad 12: /Microcontrolador/SCLK -> Net-(R24-Pad1)
- U2 pad 13: /Microcontrolador/CS1 -> Net-(R25-Pad1)
- U2 pad 16: /Procesador/RST_P -> Net-(R26-Pad2)
- U3 pad 3: Net-(BT1-Pad1) -> Net-(C9-Pad1)
Routing:
- net GND: track 353.2 -> 0.00 mm, vias 12 -> 0
- net +5VL: track 144.0 -> 0.00 mm, vias 3 -> 0
- net +5V: track 134.1 -> 0.00 mm
- net +3V8: track 119.7 -> 0.00 mm, vias 4 -> 0
- net /Microcontrolador/USART_1: track 0.00 -> 100.3 mm
- net /Microcontrolador/USART_2: track 0.00 -> 95.8 mm
- net /camara/RST_P2: track 0.00 -> 60.3 mm
- net /camara/TD13: track 0.00 -> 48.8 mm, vias 0 -> 2
- net /camara/TD03: track 0.00 -> 44.6 mm, vias 0 -> 2
- net /Microcontrolador/SRST1: track 40.5 -> 0.00 mm
- net Net-(C25-Pad1): track 0.00 -> 38.2 mm
- net Net-(BT1-Pad1): track 38.2 -> 0.00 mm
- net Net-(C20-Pad1): track 0.00 -> 37.8 mm
- net /camara/TCK3: track 0.00 -> 35.4 mm
- net /camara/TMS3: track 0.00 -> 33.8 mm, vias 0 -> 2
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Other:
- rule via_min_drill: 0.3 -> 0.4
- rule via_min_size: 0.4 -> 0.8

Commit message: Add files via upload
Parts:
- D1, D3, D4: footprint Diode_THT:D_DO-41_SOD81_P10.16mm_Horizontal -> Diode_THT:D_DO-41_SOD81_P5.08mm_Vertical_AnodeUp
- SW1, SW2, SW3: footprint Button_Switch_SMD:SW_DIP_SPSTx01_Slide_6.7x4.1mm_W6.73mm_P2.54mm_LowProfile_JPin -> Button_Switch_SMD:SW_Push_1P1T_NO_6x6mm_H9.5mm
- Y1: footprint Crystal:Crystal_HC49-U_Horizontal -> Crystal:Crystal_HC49-U_Vertical
- moved J3 5.84 mm to (147.3, 34.8)
- moved J2 4.83 mm to (66.8, 47.5)
- moved J5 4.83 mm to (176.8, 63.2)
- moved Y1 4.32 mm to (76.5, 74.7)
- moved J1 2.69 mm to (66.8, 41.1), turned to 180 degrees
- moved SW1 1.52 mm to (96.8, 58.2)
- moved C38 0.51 mm to (162.7, 37.1)
- moved C39 0.51 mm to (162.6, 39.6)
- moved U11 0.51 mm to (171.4, 39.6)
- moved C37 0.51 mm to (162.6, 41.9)
- moved D3 0.36 mm to (160.5, 57.7)
Routing:
- net Net-(C7-Pad1): track 43.3 -> 53.9 mm
- net /Procesador/RST_P: track 8.96 -> 15.5 mm
- net Net-(D2-Pad1): track 19.7 -> 25.8 mm
- net Net-(C2-Pad1): track 38.0 -> 44.1 mm
- net /Microcontrolador/RST_M: track 32.2 -> 38.1 mm
- net Net-(C43-Pad1): track 23.6 -> 29.5 mm
- net Net-(D2-Pad2): track 10.4 -> 16.2 mm
- net Net-(C44-Pad1): track 15.7 -> 20.5 mm
- net /Puente H/M2+: track 6.16 -> 10.9 mm
- net /Puente H/M2-: track 6.28 -> 11.0 mm
- net Net-(C31-Pad2): track 30.9 -> 35.2 mm
- net Net-(C34-Pad2): track 35.3 -> 39.6 mm
- net /Puente H/M1-: track 8.76 -> 11.7 mm
- net /Puente H/M1+: track 8.63 -> 10.8 mm, vias 0 -> 1
- net Net-(C7-Pad2): track 24.0 -> 26.0 mm
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
Commit message: Add files via upload
Parts:
- moved J9 41.3 mm to (176.3, 75.7), turned to 0 degrees
- moved Q1 24.4 mm to (163.6, 73.9), turned to 0 degrees
- moved U3 20.3 mm to (163.6, 68.3), turned to 0 degrees
- moved C44 5.59 mm to (170.6, 69.3)
Routing:
- net Net-(C7-Pad1): track 53.9 -> 21.8 mm
- net Net-(C9-Pad1): track 18.5 -> 40.8 mm
- net Net-(R8-Pad1): track 7.50 -> 22.4 mm
- net Net-(C12-Pad1): track 35.2 -> 44.5 mm, vias 2 -> 4
- net Net-(C44-Pad1): track 20.5 -> 14.9 mm

Commit message: Add files via upload
Parts:
- removed C18, C32, C33, C35: 0.1uF, Capacitor_SMD:C_0603_1608Metric_Pad1.05x0.95mm_HandSolder
- removed J4, J7: AVR-JTAG-10, Connector_PinSocket_2.54mm:PinSocket_1x10_P2.54mm_Vertical
- removed R15: 510, Resistor_SMD:R_0603_1608Metric_Pad1.05x0.95mm_HandSolder
- added D7: LED, Diode_SMD:D_0805_2012Metric_Pad1.15x1.40mm_HandSolder, F.Cu at (98.0, 51.8)
- added FL1: BLM18SG121TN1D, Resistor_SMD:R_0603_1608Metric_Pad1.05x0.95mm_HandSolder, F.Cu at (75.6, 34.0)
- added FL2: BLM18SG121TN1D, Resistor_SMD:R_0603_1608Metric_Pad1.05x0.95mm_HandSolder, F.Cu at (166.9, 34.3)
- added FL3: BLM18SG121TN1D, Resistor_SMD:R_0603_1608Metric_Pad1.05x0.95mm_HandSolder, F.Cu at (70.6, 69.6)
- added FL4: BLM18SG121TN1D, Resistor_SMD:R_0603_1608Metric_Pad1.05x0.95mm_HandSolder, F.Cu at (166.0, 77.7)
- added FL5: BLM18SG121TN1D, Resistor_SMD:R_0603_1608Metric_Pad1.05x0.95mm_HandSolder, F.Cu at (79.0, 168.3)
- added FL6: BLM18SG121TN1D, Resistor_SMD:R_0603_1608Metric_Pad1.05x0.95mm_HandSolder, F.Cu at (88.9, 121.9)
- added FL7: BLM18SG121TN1D, Resistor_SMD:R_0603_1608Metric_Pad1.05x0.95mm_HandSolder, F.Cu at (137.0, 172.7)
- added FL8: BLM18SG121TN1D, Resistor_SMD:R_0603_1608Metric_Pad1.05x0.95mm_HandSolder, F.Cu at (137.2, 121.9)
- added H1: MountingHole_Pad, MountingHole:MountingHole_2.5mm_Pad, F.Cu at (69.6, 34.0)
- added H2: MountingHole_Pad, MountingHole:MountingHole_2.5mm_Pad, F.Cu at (173.5, 34.3)
- added H3: MountingHole_Pad, MountingHole:MountingHole_2.5mm_Pad, F.Cu at (70.6, 75.7)
- added H4: MountingHole_Pad, MountingHole:MountingHole_2.5mm_Pad, F.Cu at (172.5, 76.2)
- added H5: MountingHole_Pad, MountingHole:MountingHole_2.5mm_Pad, F.Cu at (82.8, 172.7)
- added H6: MountingHole_Pad, MountingHole:MountingHole_2.5mm_Pad, F.Cu at (82.5, 122.2)
- added H7: MountingHole_Pad, MountingHole:MountingHole_2.5mm_Pad, F.Cu at (142.7, 173.0)
- added H8: MountingHole_Pad, MountingHole:MountingHole_2.5mm_Pad, F.Cu at (143.5, 122.4)
- R7: value 510 -> R
- moved J9 35.1 mm to (141.2, 78.0), turned to 180 degrees
- moved R7 28.5 mm to (100.8, 51.9), turned to 270 degrees
- moved R26 11.6 mm to (104.6, 70.2), turned to 90 degrees
- moved C5 9.22 mm to (136.0, 41.9)
- moved C4 8.96 mm to (136.0, 44.2)
- moved U2 8.70 mm to (107.4, 42.4)
- moved C6 8.29 mm to (102.4, 70.1), turned to 90 degrees
- moved J10 7.64 mm to (117.1, 166.1)
- moved R2 7.41 mm to (81.5, 38.9), turned to 180 degrees
- moved U12 7.15 mm to (142.0, 130.6)
- moved U7 7.15 mm to (142.2, 141.0)
- moved R19 6.75 mm to (136.1, 149.0)
- moved R6 6.43 mm to (100.1, 70.1), turned to 270 degrees
- moved C21 6.14 mm to (134.0, 142.7)
- moved C22 6.14 mm to (134.1, 138.4)
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Connections:
- R7 pad 1: GND -> Net-(D7-Pad1)
- R7 pad 2: Net-(J4-Pad10) -> GND
- U10 pad 25: /Microcontrolador/TD11 -> /Procesador/TCK1
- U2 pad 19: /Procesador/TD02 -> /Microcontrolador/TCK1
- U2 pad 2: /Procesador/TRST2 -> /Microcontrolador/TRST1
- U2 pad 20: /Procesador/TD12 -> /Microcontrolador/TD01
- U2 pad 5: /Procesador/SRST2 -> /Microcontrolador/SRST1
- U2 pad 6: /Procesador/TCK2 -> /Procesador/TCK1
- U2 pad 7: /Procesador/TMS2 -> /Microcontrolador/TMS1
- U6 pad 19: /camara/TD03 -> Net-(U6-Pad19)
- U6 pad 2: /camara/TRST3 -> Net-(U6-Pad2)
- U6 pad 20: /camara/TD13 -> Net-(U6-Pad20)
- U6 pad 5: /camara/SRST3 -> Net-(U6-Pad5)
- U6 pad 6: /camara/TCK3 -> Net-(U6-Pad6)
- U6 pad 7: /camara/TMS3 -> Net-(U6-Pad7)
Routing:
- net +3V8: track 0.00 -> 182.1 mm, vias 0 -> 10
- net +5V: track 0.00 -> 166.9 mm, vias 0 -> 3
- net +3V0: track 0.00 -> 85.3 mm, vias 0 -> 2
- net +5VL: track 0.00 -> 67.6 mm, vias 0 -> 4
- net +5VP: track 0.00 -> 58.9 mm, vias 0 -> 5
- net /Microcontrolador/TCK1: track 0.00 -> 55.7 mm
- net /Microcontrolador/TD01: track 0.00 -> 55.0 mm
- net /Procesador/TD12: track 50.1 -> 0.00 mm, vias 2 -> 0
- net /camara/TD13: track 48.8 -> 0.00 mm, vias 2 -> 0
- net /Procesador/TD02: track 45.8 -> 0.00 mm
- net /camara/TD03: track 44.6 -> 0.00 mm, vias 2 -> 0
- net +5VD: track 0.00 -> 40.3 mm, vias 0 -> 2
- net /Procesador/TCK2: track 39.6 -> 0.00 mm, vias 2 -> 0
- net /camara/TCK3: track 35.4 -> 0.00 mm
- net /Procesador/TMS2: track 34.4 -> 0.00 mm
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- added copper zone on B.Cu, net GND
- added copper zone on F.Cu, net GND
- added copper zone on B.Cu, net GNDA
- added copper zone on F.Cu, net GNDA
