File: proyecto/proyecto.sch (KiCad schematic (older format))
At the start: 34 parts, among them SW1 SW_Push, SW2 SW_Push

Commit message: Add files via upload
Parts:
- removed C1, C3: 10uF, symbol Device:C
- removed C10, C11, C12, C13, C8, C9: 0.1uM, symbol Device:C
- removed C14, C15, C2, C6, C7: 0.1uF, symbol Device:C
- removed C4, C5: C, symbol Device:C
- removed D?: SP0502BAHT, Package_TO_SOT_SMD:SOT-23, symbol Power_Protection:SP0502BAHT
- removed D?: 1N47xxA, Diode_THT:D_DO-41_SOD81_P10.16mm_Horizontal, symbol Diode:1N47xxA
- removed J?: USB_A, symbol Connector:USB_A
- removed J?: M1, symbol Connector_Generic:Conn_01x02
- removed J?: M2, symbol Connector_Generic:Conn_01x02
- removed L1, L2, L3: L, symbol Device:L
- removed R1, R2: R, symbol Device:R
- removed R3, R4: 10k, symbol Device:R
- removed R5: 10K, symbol Device:R
- removed SW1, SW2: SW_Push, symbol Switch:SW_Push
- removed U?: Omega2+, Module:Onion_Omega2+, symbol MCU_Module:Omega2+
- removed U?: STM32L052C6Tx, Package_QFP:LQFP-48_7x7mm_P0.5mm, symbol MCU_ST_STM32L0:STM32L052C6Tx
- removed U?: L293D, Package_DIP:DIP-16_W7.62mm, symbol Driver_Motor:L293D
- removed U?: LM1117-3.3, symbol Regulator_Linear:LM1117-3.3

Commit message: Add files via upload
Changed lines of the file:
@@
 $Descr A4 11693 8268
 encoding utf-8
-Sheet 1 5
+Sheet 1 7
 Title ""
 Date ""
@@
 $EndDescr
 $Sheet
-S 5950 3400 1050 2000
+S 5950 3400 1050 2600
 U 5E9DF408
 F0 "Microcontrolador" 50
@@
 F8 "PH_4A" I R 7000 4450 50
 F9 "PH_EN34" I R 7000 4550 50
-F10 "3.3v" I L 5950 3800 50
-F11 "MOSI" I L 5950 4800 50
-F12 "CS1" I L 5950 5000 50
-F13 "SCLK" I L 5950 4900 50
-F14 "MISO" I L 5950 4700 50
+F10 "MOSI" I L 5950 4800 50
+F11 "CS1" I L 5950 5000 50
+F12 "SCLK" I L 5950 4900 50
+F13 "MISO" I L 5950 4700 50
+F14 "TRST" I L 5950 5200 50
+F15 "SRST" I L 5950 5300 50
+F16 "TCK" I L 5950 5400 50
+F17 "TMS" I L 5950 5500 50
+F18 "TD0" I L 5950 5600 50
+F19 "TD1" I L 5950 5700 50
 $EndSheet
 $Sheet
@@
 F6 "PH_4A" I L 8000 4450 50
 F7 "PH_EN34" I L 8000 4550 50
-F8 "3.3v" I L 8000 3800 50
-F9 "5v" I L 8000 3600 50
-$EndSheet
-$Sheet
-S 1950 1500 1000 1500
-U 5E9BC166
-F0 "Alimentacion" 50
-F1 "Alimentacion.sch" 50
-F2 "3.3v" I R 2950 2550 50
-F3 "5v" I R 2950 2100 50
 $EndSheet
 Wire Wire Line
@@
 Wire Wire Line
 	5050 4400 5950 4400
-Wire Wire Line
-	7000 4050 8000 4050
 Wire Wire Line
 	8000 4150 7000 4150
@@
 Wire Wire Line
 	8000 4550 7000 4550
-Wire Wire Line
-	7500 2550 5650 2550
-Wire Wire Line
-	7500 2550 7500 3800
-Wire Wire Line
-	8000 3800 7500 3800
-Wire Wire Line
-	8000 3600 7750 3600
-Wire Wire Line
-	7750 3600 7750 2100
-Wire Wire Line
-	5950 3800 5650 3800
-Wire Wire Line
-	5650 3800 5650 2550
-Connection ~ 5650 2550
-Wire Wire Line
-	7750 2100 3650 2100
-Wire Wire Line
-	5650 2550 3350 2550
 $Sheet
-S 4000 3400 1050 2000
+S 4000 3400 1050 2600
 U 5E9F954D
 F0 "Procesador" 50
@@
 F2 "USART_1" I R 5050 4300 50
 F3 "USART_2" I R 5050 4400 50
-F4 "3.3v" I L 4000 3800 50
-F5 "5v" I L 4000 3600 50
-F6 "MISO" I R 5050 4700 50
-F7 "MOSI" I R 5050 4800 50
-F8 "SCLK" I R 5050 4900 50
-F9 "CS1" I R 5050 5000 50
+F4 "MISO" I R 5050 4700 50
+F5 "MOSI" I R 5050 4800 50
+F6 "SCLK" I R 5050 4900 50
+F7 "CS1" I R 5050 5000 50
+F8 "TRST" I R 5050 5200 50
+F9 "SRST" I R 5050 5300 50
+F10 "TCK" I R 5050 5400 50
+F11 "TMS" I R 5050 5500 50
+F12 "TD0" I R 5050 5600 50
+F13 "TD1" I R 5050 5700 50
 $EndSheet
-Wire Wire Line
-	4000 3800 3350 3800
-Wire Wire Line
-	3350 3800 3350 2550
-Connection ~ 3350 2550
-Wire Wire Line
-	3350 2550 2950 2550
-Wire Wire Line
-	4000 3600 3650 3600
-Wire Wire Line
-	3650 3600 3650 2100
-Connection ~ 3650 2100
-Wire Wire Line
-	3650 2100 2950 2100
 Wire Wire Line
 	5050 4700 5950 4700
@@
 Wire Wire Line
 	5950 5000 5050 5000
+$Sheet
+S 1950 4500 1000 1500
+U 5E9BC166
+F0 "Alimentacion" 50
+F1 "Alimentacion.sch" 50
+$EndSheet
+Wire Wire Line
+	5050 5200 5950 5200
+Wire Wire Line
+	5950 5300 5050 5300
+Wire Wire Line
+	5050 5400 5950 5400
+Wire Wire Line
+	5950 5500 5050 5500
+Wire Wire Line
+	5950 5700 5050 5700
+Wire Wire Line
+	5050 5600 5950 5600
+Wire Wire Line
+	7000 4050 8000 4050
+$Sheet
+S 5200 1150 1050 1000
+U 5E9DF2DA
+F0 "camara" 50
+F1 "camara.sch" 50
+$EndSheet
+$Sheet
+S 2900 950  1000 1500
+U 5EA3D59C
+F0 "Alimentacion_camara" 50
+F1 "Alimentacion_camara.sch" 50
+$EndSheet
 $EndSCHEMATC

Commit message: Add files via upload
Changed lines of the file:
@@
 $EndSheet
 $Sheet
-S 2900 950  1000 1500
+S 2200 1200 1000 1500
 U 5EA3D59C
 F0 "Alimentacion_camara" 50

Commit message: Add files via upload
Changed lines of the file:
@@
 $EndDescr
-$Sheet
-S 5950 3400 1050 2600
-U 5E9DF408
-F0 "Microcontrolador" 50
-F1 "Microcontrolador.sch" 50
-F2 "USART_1" I L 5950 4300 50
-F3 "USART_2" I L 5950 4400 50
-F4 "PH_1A" I R 7000 4050 50
-F5 "PH_2A" I R 7000 4150 50
-F6 "PH_EN12" I R 7000 4250 50
-F7 "PH_3A" I R 7000 4350 50
-F8 "PH_4A" I R 7000 4450 50
-F9 "PH_EN34" I R 7000 4550 50
-F10 "MOSI" I L 5950 4800 50
-F11 "CS1" I L 5950 5000 50
-F12 "SCLK" I L 5950 4900 50
-F13 "MISO" I L 5950 4700 50
-F14 "TRST" I L 5950 5200 50
-F15 "SRST" I L 5950 5300 50
-F16 "TCK" I L 5950 5400 50
-F17 "TMS" I L 5950 5500 50
-F18 "TD0" I L 5950 5600 50
-F19 "TD1" I L 5950 5700 50
-$EndSheet
 $Sheet
 S 8000 3450 1000 1950
@@
 F6 "SCLK" I R 5050 4900 50
 F7 "CS1" I R 5050 5000 50
-F8 "TRST" I R 5050 5200 50
-F9 "SRST" I R 5050 5300 50
-F10 "TCK" I R 5050 5400 50
-F11 "TMS" I R 5050 5500 50
-F12 "TD0" I R 5050 5600 50
-F13 "TD1" I R 5050 5700 50
 $EndSheet
 Wire Wire Line
@@
 $EndSheet
 Wire Wire Line
-	5050 5200 5950 5200
-Wire Wire Line
-	5950 5300 5050 5300
-Wire Wire Line
-	5050 5400 5950 5400
-Wire Wire Line
-	5950 5500 5050 5500
-Wire Wire Line
-	5950 5700 5050 5700
-Wire Wire Line
-	5050 5600 5950 5600
-Wire Wire Line
 	7000 4050 8000 4050
 $Sheet
@@
 F1 "Alimentacion_camara.sch" 50
 $EndSheet
+$Sheet
+S 5950 3400 1050 2600
+U 5E9DF408
+F0 "Microcontrolador" 50
+F1 "Microcontrolador.sch" 50
+F2 "USART_1" I L 5950 4300 50
+F3 "USART_2" I L 5950 4400 50
+F4 "PH_1A" I R 7000 4050 50
+F5 "PH_2A" I R 7000 4150 50
+F6 "PH_EN12" I R 7000 4250 50
+F7 "PH_3A" I R 7000 4350 50
+F8 "PH_4A" I R 7000 4450 50
+F9 "PH_EN34" I R 7000 4550 50
+F10 "MOSI" I L 5950 4800 50
+F11 "CS1" I L 5950 5000 50
+F12 "SCLK" I L 5950 4900 50
+F13 "MISO" I L 5950 4700 50
+$EndSheet
 $EndSCHEMATC

Commit message: Add files via upload
Other:
- note added: "PLACA CARRO"
- note added: "PLACA CÁMARA"
Changed lines of the file:
@@
 $EndDescr
 $Sheet
-S 8000 3450 1000 1950
+S 7450 4000 1000 1950
 U 5EA16FA2
 F0 "Puente H" 50
 F1 "Puente H.sch" 50
-F2 "PH_1A" I L 8000 4050 50
-F3 "PH_2A" I L 8000 4150 50
-F4 "PH_EN12" I L 8000 4250 50
-F5 "PH_3A" I L 8000 4350 50
-F6 "PH_4A" I L 8000 4450 50
-F7 "PH_EN34" I L 8000 4550 50
+F2 "PH_1A" I L 7450 4600 50
+F3 "PH_2A" I L 7450 4700 50
+F4 "PH_EN12" I L 7450 4800 50
+F5 "PH_3A" I L 7450 4900 50
+F6 "PH_4A" I L 7450 5000 50
+F7 "PH_EN34" I L 7450 5100 50
 $EndSheet
 Wire Wire Line
-	5050 4300 5950 4300
+	4500 4850 5400 4850
 Wire Wire Line
-	5050 4400 5950 4400
+	4500 4950 5400 4950
 Wire Wire Line
-	8000 4150 7000 4150
+	7450 4700 6450 4700
 Wire Wire Line
-	7000 4250 8000 4250
+	6450 4800 7450 4800
 Wire Wire Line
-	8000 4350 7000 4350
+	7450 4900 6450 4900
 Wire Wire Line
-	7000 4450 8000 4450
+	6450 5000 7450 5000
 Wire Wire Line
-	8000 4550 7000 4550
+	7450 5100 6450 5100
 $Sheet
-S 4000 3400 1050 2600
+S 3450 3950 1050 2600
 U 5E9F954D
 F0 "Procesador" 50
 F1 "Procesador.sch" 50
-F2 "USART_1" I R 5050 4300 50
-F3 "USART_2" I R 5050 4400 50
-F4 "MISO" I R 5050 4700 50
-F5 "MOSI" I R 5050 4800 50
-F6 "SCLK" I R 5050 4900 50
-F7 "CS1" I R 5050 5000 50
+F2 "USART_1" I R 4500 4850 50
+F3 "USART_2" I R 4500 4950 50
+F4 "MISO" I R 4500 5250 50
+F5 "MOSI" I R 4500 5350 50
+F6 "SCLK" I R 4500 5450 50
+F7 "CS1" I R 4500 5550 50
 $EndSheet
 Wire Wire Line
-	5050 4700 5950 4700
+	4500 5250 5400 5250
 Wire Wire Line
-	5950 4800 5050 4800
+	5400 5350 4500 5350
 Wire Wire Line
-	5050 4900 5950 4900
+	4500 5450 5400 5450
 Wire Wire Line
-	5950 5000 5050 5000
+	5400 5550 4500 5550
 $Sheet
-S 1950 4500 1000 1500
+S 1400 5050 1000 1500
 U 5E9BC166
 F0 "Alimentacion" 50
@@
 $EndSheet
 Wire Wire Line
-	7000 4050 8000 4050
+	6450 4600 7450 4600
 $Sheet
-S 5200 1150 1050 1000
+S 5400 1150 1050 1000
 U 5E9DF2DA
 F0 "camara" 50
@@
 $EndSheet
 $Sheet
-S 2200 1200 1000 1500
+S 3150 1050 1000 1500
 U 5EA3D59C
 F0 "Alimentacion_camara" 50
@@
 $EndSheet
 $Sheet
-S 5950 3400 1050 2600
+S 5400 3950 1050 2600
 U 5E9DF408
 F0 "Microcontrolador" 50
 F1 "Microcontrolador.sch" 50
-F2 "USART_1" I L 5950 4300 50
-F3 "USART_2" I L 5950 4400 50
-F4 "PH_1A" I R 7000 4050 50
-F5 "PH_2A" I R 7000 4150 50
-F6 "PH_EN12" I R 7000 4250 50
-F7 "PH_3A" I R 7000 4350 50
-F8 "PH_4A" I R 7000 4450 50
-F9 "PH_EN34" I R 7000 4550 50
-F10 "MOSI" I L 5950 4800 50
-F11 "CS1" I L 5950 5000 50
-F12 "SCLK" I L 5950 4900 50
-F13 "MISO" I L 5950 4700 50
+F2 "USART_1" I L 5400 4850 50
+F3 "USART_2" I L 5400 4950 50
+F4 "PH_1A" I R 6450 4600 50
+F5 "PH_2A" I R 6450 4700 50
+F6 "PH_EN12" I R 6450 4800 50
+F7 "PH_3A" I R 6450 4900 50
+F8 "PH_4A" I R 6450 5000 50
+F9 "PH_EN34" I R 6450 5100 50
+F10 "MOSI" I L 5400 5350 50
+F11 "CS1" I L 5400 5550 50
+F12 "SCLK" I L 5400 5450 50
+F13 "MISO" I L 5400 5250 50
 $EndSheet
+Wire Notes Line
+	11250 3400 450  3400
+Text Notes 550  3350 0    50   ~ 0
+PLACA CÁMARA
+Text Notes 550  7750 0    50   ~ 0
+PLACA CARRO
 $EndSCHEMATC

Commit message: Add files via upload
Changed lines of the file:
@@
 Wire Wire Line
 	7450 5100 6450 5100
-$Sheet
-S 3450 3950 1050 2600
-U 5E9F954D
-F0 "Procesador" 50
-F1 "Procesador.sch" 50
-F2 "USART_1" I R 4500 4850 50
-F3 "USART_2" I R 4500 4950 50
-F4 "MISO" I R 4500 5250 50
-F5 "MOSI" I R 4500 5350 50
-F6 "SCLK" I R 4500 5450 50
-F7 "CS1" I R 4500 5550 50
-$EndSheet
 Wire Wire Line
 	4500 5250 5400 5250
@@
 F1 "Alimentacion_camara.sch" 50
 $EndSheet
+Wire Notes Line
+	11250 3400 450  3400
+Text Notes 550  3350 0    50   ~ 0
+PLACA CÁMARA
+Text Notes 550  7750 0    50   ~ 0
+PLACA CARRO
+$Sheet
+S 3450 3950 1050 2600
+U 5E9F954D
+F0 "Procesador" 50
+F1 "Procesador.sch" 50
+F2 "USART_1" I R 4500 4850 50
+F3 "USART_2" I R 4500 4950 50
+F4 "MISO" I R 4500 5250 50
+F5 "MOSI" I R 4500 5350 50
+F6 "SCLK" I R 4500 5450 50
+F7 "CS1" I R 4500 5550 50
+F8 "TRST1" I R 4500 5800 50
+F9 "SRST1" I R 4500 5900 50
+F10 "TCK1" I R 4500 6000 50
+F11 "TMS1" I R 4500 6100 50
+F12 "TD01" I R 4500 6200 50
+F13 "TDI1" I R 4500 6300 50
+$EndSheet
 $Sheet
 S 5400 3950 1050 2600
@@
 F12 "SCLK" I L 5400 5450 50
 F13 "MISO" I L 5400 5250 50
+F14 "TRST1" I L 5400 5800 50
+F15 "SRST1" I L 5400 5900 50
+F16 "TDI1" I L 5400 6000 50
+F17 "TMS1" I L 5400 6100 50
+F18 "TCK1" I L 5400 6200 50
+F19 "TD01" I L 5400 6300 50
 $EndSheet
-Wire Notes Line
-	11250 3400 450  3400
-Text Notes 550  3350 0    50   ~ 0
-PLACA CÁMARA
-Text Notes 550  7750 0    50   ~ 0
-PLACA CARRO
+Wire Wire Line
+	5400 5800 4500 5800
+Wire Wire Line
+	4500 5900 5400 5900
+Wire Wire Line
+	5400 6000 4500 6000
+Wire Wire Line
+	4500 6100 5400 6100
+Wire Wire Line
+	5400 6200 4500 6200
+Wire Wire Line
+	4500 6300 5400 6300
 $EndSCHEMATC
